File: Hardware/SPU2/SPU2.sch (KiCad schematic (older format))
At the start: 71 parts, among them U1 74LS86, U10 74LS08, U11 74LS173, U12 74LS173, U2 74LS86, U3 74LS245, U4 74LS283, U5 74LS283, U6 4077, U7 4077, U8 74LS02, U9 4068

Commit message: im tired
Parts:
- added C? (x3): CP, symbol Device:CP
- added D? (x44): LED, symbol Device:LED
- added Q?: BC547, Package_TO_SOT_THT:TO-92_Inline, symbol Transistor_BJT:BC547
- added R? (x45): R, symbol Device:R
- added U? (x5): 74LS245, symbol 74xx:74LS245
- added U?: 74HCT574, symbol 74xx:74HCT574
- added U? (x6): 74LS173, symbol 74xx:74LS173
- added U? (x2): 74LS189, symbol custom:74LS189
- gave numbers to parts that had none: 41
Connections:
- net +5V: now also C?.1, C?.1, C?.1, R?.1, U?.1 (A->B), U?.1 (A->B), U?.1 (A->B), U?.1 (A->B), U?.1 (A->B), U?.16 (VCC), U?.16 (VCC), U?.16 (VCC), U?.16 (VCC), U?.16 (VCC), U?.16 (VCC), U?.16 (VCC), U?.16 (VCC), U?.20 (VCC), U?.20 (VCC), U?.20 (VCC), U?.20 (VCC), U?.20 (VCC); no longer U13.1 (~MR), U14.1 (~MR), U15.1 (~MR)
- net CLK: now also U?.7 (Cp), U?.7 (Cp), U?.7 (Cp), U?.7 (Cp), U?.7 (Cp), U?.7 (Cp)
- net D0: now also U?.18 (B0)
- net D1: now also U?.17 (B1)
- net D2: now also U?.16 (B2)
- net D3: now also U?.15 (B3)
- net D4: now also U?.14 (B4)
- net D5: now also U?.13 (B5)
- net D6: now also U?.12 (B6)
- net D7: now also U?.11 (B7)
- net GND: now also C?.2, C?.2, C?.2, D?.1 (K), D?.1 (K), D?.1 (K), D?.1 (K), D?.1 (K), D?.1 (K), D?.1 (K), D?.1 (K), D?.1 (K), D?.1 (K), D?.1 (K), D?.1 (K), D?.1 (K), D?.1 (K), D?.1 (K), D?.1 (K), D?.1 (K), D?.1 (K), D?.1 (K), D?.1 (K), D?.1 (K), D?.1 (K), D?.1 (K), D?.1 (K), D?.1 (K), D?.1 (K), D?.1 (K), D?.1 (K), D?.1 (K), D?.1 (K), D?.1 (K), D?.1 (K), D?.1 (K), D?.1 (K), D?.1 (K), D?.1 (K), D?.1 (K), D?.1 (K), D?.1 (K), D?.1 (K), D?.1 (K), D?.1 (K), D?.1 (K), D?.1 (K), Q?.3 (E), U?.1 (Oe1), U?.1 (Oe1), U?.1 (Oe1), U?.1 (Oe1), U?.1 (Oe1), U?.1 (Oe1), U?.10 (GND), U?.10 (GND), U?.10 (GND), U?.10 (GND), U?.10 (GND), U?.15 (Mr), U?.15 (Mr), U?.15 (Mr), U?.15 (Mr), U?.15 (Mr), U?.15 (Mr), U?.2 (Oe2), U?.2 (Oe2), U?.2 (Oe2), U?.2 (Oe2), U?.2 (Oe2), U?.2 (Oe2), U?.2 (~CS), U?.2 (~CS), U?.6 (A4), U?.6 (A4), U?.7 (A5), U?.7 (A5), U?.8 (A6), U?.8 (A6), U?.8 (GND), U?.8 (GND), U?.8 (GND), U?.8 (GND), U?.8 (GND), U?.8 (GND), U?.8 (GND), U?.8 (GND), U?.9 (A7), U?.9 (A7)
- net PC3: now reaches U13.11 (Q3)
- net PC3: now also R?.2, U?.2 (A0)
- net PC2: now reaches U13.12 (Q2)
- net PC2: now also R?.2, U?.3 (A1)
- net PC1: now reaches U13.13 (Q1)
- net PC1: now also R?.2, U?.4 (A2)
- net PC0: now reaches U13.14 (Q0)
- net PC0: now also R?.2, U?.5 (A3)
- net ADDR0: now reaches U13.3 (D0)
- net ADDR0: now also U?.14 (D0), U?.14 (D0), U?.15 (B3), U?.15 (B3)
- net ADDR1: now reaches U13.4 (D1)
- net ADDR1: now also U?.13 (D1), U?.13 (D1), U?.16 (B2), U?.16 (B2)
- net ADDR2: now reaches U13.5 (D2)
- net ADDR2: now also U?.12 (D2), U?.12 (D2), U?.17 (B1), U?.17 (B1)
- net ADDR3: now reaches U13.6 (D3)
- net ADDR3: now also U?.11 (D3), U?.11 (D3), U?.18 (B0), U?.18 (B0)
- net ~J: now reaches U13.9 (~PE)
- net ~J: now also U14.9 (~PE), U15.9 (~PE)
- net PC7: now reaches U14.11 (Q3)
- net PC7: now also R?.2, U?.6 (A4)
- net PC6: now reaches U14.12 (Q2)
- net PC6: now also R?.2, U?.7 (A5)
- net PC5: now reaches U14.13 (Q1)
- net PC5: now also R?.2, U?.8 (A6)
- net PC4: now reaches U14.14 (Q0)
- net PC4: now also R?.2, U?.9 (A7)
- net ADDR4: now reaches U14.3 (D0)
- net ADDR4: now also U?.11 (B7), U?.11 (B7), U?.14 (D0), U?.14 (D0)
- net ADDR5: now reaches U14.4 (D1)
- net ADDR5: now also U?.12 (B6), U?.12 (B6), U?.13 (D1), U?.13 (D1)
- net ADDR6: now reaches U14.5 (D2)
- net ADDR6: now also U?.12 (D2), U?.12 (D2), U?.13 (B5), U?.13 (B5)
- net ADDR7: now reaches U14.6 (D3)
- net ADDR7: now also U?.11 (D3), U?.11 (D3), U?.14 (B4), U?.14 (B4)
- net PC11: now reaches U15.11 (Q3)
- net PC11: now also Q?.2 (B), R?.2, U?.2 (A0)
- net PC10: now reaches U15.12 (Q2)
- net PC10: now also R?.2, U?.3 (A1)
- net PC9: now reaches U15.13 (Q1)
- net PC9: now also R?.2, U?.4 (A2)
- net PC8: now reaches U15.14 (Q0)
- net PC8: now also R?.2, U?.5 (A3)
- net ADDR8: now reaches U15.3 (D0)
- net ADDR8: now also U?.14 (D0), U?.14 (D0), U?.15 (B3), U?.15 (B3)
- net ADDR9: now reaches U15.4 (D1)
- net ADDR9: now also U?.13 (D1), U?.13 (D1), U?.16 (B2), U?.16 (B2)
- net ADDR10: now reaches U15.5 (D2)
- net ADDR10: now also U?.12 (D2), U?.12 (D2), U?.17 (B1), U?.17 (B1)
- net ADDR11: now reaches U15.6 (D3)
- net ADDR11: now also U?.11 (D3), U?.11 (D3), U?.18 (B0), U?.18 (B0)
- new net: Q?.1 (C), R?.2, U13.1 (~MR), U14.1 (~MR), U15.1 (~MR)
- new net: D?.2 (A), R?.1 (x44)
- new net: R?.2, U?.11 (~O3), U?.5 (A3)
- new net: R?.2, U?.2 (A0), U?.5 (~O0)
- new net: R?.2, U?.3 (A1), U?.7 (~O1)
- new net: R?.2, U?.4 (A2), U?.9 (~O2)
- new net: R?.2, U?.11 (~O3), U?.9 (A7)
- new net: R?.2, U?.5 (~O0), U?.6 (A4)
- new net: R?.2, U?.7 (A5), U?.7 (~O1)
- new net: R?.2, U?.8 (A6), U?.9 (~O2)
- new net BJAB0: R?.2, U?.3 (Q0), U?.5 (A3)
- new net BJAB1: R?.2, U?.4 (A2), U?.4 (Q1)
- new net BJAB10: R?.2, U?.3 (A1), U?.5 (Q2)
- new net BJAB11: R?.2, U?.2 (A0), U?.6 (Q3)
- new net BJAB2: R?.2, U?.3 (A1), U?.5 (Q2)
- new net BJAB3: R?.2, U?.2 (A0), U?.6 (Q3)
- new net BJAB4: R?.2, U?.3 (Q0), U?.9 (A7)
- new net BJAB5: R?.2, U?.4 (Q1), U?.8 (A6)
- new net BJAB6: R?.2, U?.5 (Q2), U?.7 (A5)
- new net BJAB7: R?.2, U?.6 (A4), U?.6 (Q3)
- new net BJAB8: R?.2, U?.3 (Q0), U?.5 (A3)
- new net BJAB9: R?.2, U?.4 (A2), U?.4 (Q1)
- new net MEMADDR0: R?.2, U?.1 (A0), U?.1 (A0), U?.3 (Q0)
- new net MEMADDR1: R?.2, U?.15 (A1), U?.15 (A1), U?.4 (Q1)
- new net MEMADDR10: R?.2, U?.5 (Q2)
- new net MEMADDR11: R?.2, U?.6 (Q3)
- new net MEMADDR2: R?.2, U?.14 (A2), U?.14 (A2), U?.5 (Q2)
- new net MEMADDR3: R?.2, U?.13 (A3), U?.13 (A3), U?.6 (Q3)
- new net MEMADDR4: R?.2, U?.3 (Q0)
- new net MEMADDR5: R?.2, U?.4 (Q1)
- new net MEMADDR6: R?.2, U?.5 (Q2)
- new net MEMADDR7: R?.2, U?.6 (Q3)
- new net MEMADDR8: R?.2, U?.3 (Q0)
- new net MEMADDR9: R?.2, U?.4 (Q1)
- new net ~JI: U?.10 (E2), U?.10 (E2), U?.10 (E2), U?.9 (E1), U?.9 (E1), U?.9 (E1)
- new net ~JO: U?.19 (CE), U?.19 (CE)
- new net ~MC: U?.10 (E2), U?.10 (E2), U?.10 (E2), U?.9 (E1), U?.9 (E1), U?.9 (E1)
- new net ~PO: U?.19 (CE), U?.19 (CE)
- new net ~RAMI: U?.3 (~WE), U?.3 (~WE)
- new net ~RAMO: U?.19 (CE)
- no-connect marks 2 -> 11
Other:
- note added: "ACHTUNG! \nEIGENTLICH 74FCT2574T\n=> geliches pinout"
- note added: "PROGRAM COUNTER (LEDs)\n"
- note added: "PROGRAM COUNTER (output control)\n"
- note added: "RAM\n\n"
- note added: "REGISTER JUMP (output control)\n\n\n"
- note added: "REGISTER JUMP\n\n\n"
- note added: "REGISTER MEMORY ADDRESS\n\n\n"

Commit message: *yawns*
Parts:
- removed U?: 74LS245, symbol 74xx:74LS245
- added D? (x52): LED, symbol Device:LED
- added R? (x52): R, symbol Device:R
- added U29: 74LS540, symbol 74xx:74LS540
- added U30, U31: 28c16, symbol custom:28c16
- added U? (x3): 74LS245, symbol 74xx:74LS245
- added U? (x2): 74HCT574, symbol 74xx:74HCT574
- added U? (x5): 74LS08, symbol 74xx:74LS08
- added U?: 74LS161, symbol 74xx:74LS161
- gave numbers to parts that had none: 106
Connections:
- net +5V: now also R62.2, R63.2, R64.2, R65.2, R66.2, R67.2, R68.2, R69.2, U29.20 (VCC), U30.21 (~WE), U30.24 (VCC), U31.21 (~WE), U31.24 (VCC), U?.1 (A->B), U?.1 (A->B), U?.1 (A->B), U?.14 (VCC), U?.20 (VCC), U?.20 (VCC), U?.20 (VCC), U?.20 (VCC), U?.20 (VCC)
- net ADDR0: now also R?.2, U30.8 (A0), U31.8 (A0), U?.18 (B0)
- net ADDR1: now also R?.2, U30.7 (A1), U31.7 (A1), U?.17 (B1)
- net ADDR10: now also R?.2, U30.19 (A10), U31.19 (A10), U?.16 (B2)
- net ADDR11: now also R?.2, U?.15 (B3)
- net ADDR2: now also R?.2, U30.6 (A2), U31.6 (A2), U?.16 (B2)
- net ADDR3: now also R?.2, U30.5 (A3), U31.5 (A3), U?.15 (B3)
- net ADDR4: now also R?.2, U30.4 (A4), U31.4 (A4), U?.14 (B4)
- net ADDR5: now also R?.2, U30.3 (A5), U31.3 (A5), U?.13 (B5)
- net ADDR6: now also R?.2, U30.2 (A6), U31.2 (A6), U?.12 (B6)
- net ADDR7: now also R?.2, U30.1 (A7), U31.1 (A7), U?.11 (B7)
- net ADDR8: now also R?.2, U30.23 (A8), U31.23 (A8), U?.18 (B0)
- net ADDR9: now also R?.2, U30.22 (A9), U31.22 (A9), U?.17 (B1)
- net CLK: now also U?.1, U?.4
- net D0: now also R?.2, U29.18 (Y0), U?.18 (B0)
- net D1: now also R?.2, U29.17 (Y1), U?.17 (B1)
- net D2: now also R?.2, U29.16 (Y2), U?.16 (B2)
- net D3: now also R?.2, U29.15 (Y3), U?.15 (B3)
- net D4: now also R?.2, U29.14 (Y4), U?.14 (B4)
- net D5: now also R?.2, U29.13 (Y5), U?.13 (B5)
- net D6: now also R?.2, U29.12 (Y6), U?.12 (B6)
- net D7: now also R?.2, U29.11 (Y7), U?.11 (B7)
- net GND: now also D?.1 (K), D?.1 (K), D?.1 (K), D?.1 (K), D?.1 (K), D?.1 (K), D?.1 (K), D?.1 (K), D?.1 (K), D?.1 (K), D?.1 (K), D?.1 (K), D?.1 (K), D?.1 (K), D?.1 (K), D?.1 (K), D?.1 (K), D?.1 (K), D?.1 (K), D?.1 (K), D?.1 (K), D?.1 (K), D?.1 (K), D?.1 (K), D?.1 (K), D?.1 (K), D?.1 (K), D?.1 (K), D?.1 (K), D?.1 (K), D?.1 (K), D?.1 (K), D?.1 (K), D?.1 (K), D?.1 (K), D?.1 (K), D?.1 (K), D?.1 (K), D?.1 (K), D?.1 (K), D?.1 (K), D?.1 (K), D?.1 (K), D?.1 (K), D?.1 (K), D?.1 (K), D?.1 (K), D?.1 (K), D?.1 (K), D?.1 (K), D?.1 (K), D?.1 (K), U29.10 (GND), U30.12 (GND), U30.18 (~CE), U30.20 (~OE), U31.12 (GND), U31.18 (~CE), U31.20 (~OE), U?.1 (OE), U?.1 (OE), U?.10, U?.10 (GND), U?.10 (GND), U?.10 (GND), U?.10 (GND), U?.10 (GND), U?.12, U?.13, U?.7 (GND), U?.9; no longer D61.1 (K), D62.1 (K), D63.1 (K), D64.1 (K), D65.1 (K), D66.1 (K), D67.1 (K), D68.1 (K)
- net ~RAMO: now also U29.1 (G1), U29.19 (G2)
- net at U26.11 (~O3): now also D65.1 (K), U29.5 (A3); no longer R65.2
- net at U26.5 (~O0): now also D68.1 (K), U29.2 (A0); no longer R62.2
- net at U26.7 (~O1): now also D67.1 (K), U29.3 (A1); no longer R63.2
- net at U26.9 (~O2): now also D66.1 (K), U29.4 (A2); no longer R64.2
- net at U27.11 (~O3): now also D61.1 (K), U29.9 (A7); no longer R69.2
- net at U27.5 (~O0): now also D64.1 (K), U29.6 (A4); no longer R66.2
- net at U27.7 (~O1): now also D63.1 (K), U29.7 (A5); no longer R67.2
- net at U27.9 (~O2): now also D62.1 (K), U29.8 (A6); no longer R68.2
- new net: D?.2 (A), R?.1 (x52)
- new net: U?.11 (Cp), U?.3
- new net: U?.11 (Cp), U?.6
- new net ARG0: R?.2, U?.19 (Q0)
- new net ARG1: R?.2, U?.18 (Q1)
- new net ARG10: R?.2, U?.17 (Q2)
- new net ARG11: R?.2, U?.16 (Q3)
- new net ARG2: R?.2, U?.17 (Q2)
- new net ARG3: R?.2, U?.16 (Q3)
- new net ARG4: R?.2, U?.15 (Q4)
- new net ARG5: R?.2, U?.14 (Q5)
- new net ARG6: R?.2, U?.13 (Q6)
- new net ARG7: R?.2, U?.12 (Q7)
- new net ARG8: R?.2, U?.19 (Q0)
- new net ARG9: R?.2, U?.18 (Q1)
- new net II: U?.2, U?.5
- new net OP0: R?.2, U?.15 (Q4)
- new net OP1: R?.2, U?.14 (Q5)
- new net OP2: R?.2, U?.13 (Q6)
- new net OP3: R?.2, U?.12 (Q7)
- new net ROM0: R?.2, U31.9 (I/O0), U?.2 (A0), U?.2 (A0), U?.2 (D0)
- new net ROM1: R?.2, U31.10 (I/O1), U?.3 (A1), U?.3 (A1), U?.3 (D1)
- new net ROM10: R?.2, U30.11 (I/O2), U?.4 (A2), U?.4 (D2)
- new net ROM11: R?.2, U30.13 (I/O3), U?.5 (A3), U?.5 (D3)
- new net ROM12: R?.2, U30.14 (I/O4), U?.6 (A4), U?.6 (D4)
- new net ROM13: R?.2, U30.15 (I/O5), U?.7 (A5), U?.7 (D5)
- new net ROM14: R?.2, U30.16 (I/O6), U?.8 (A6), U?.8 (D6)
- new net ROM15: R?.2, U30.17 (I/O7), U?.9 (A7), U?.9 (D7)
- new net ROM2: R?.2, U31.11 (I/O2), U?.4 (A2), U?.4 (A2), U?.4 (D2)
- new net ROM3: R?.2, U31.13 (I/O3), U?.5 (A3), U?.5 (A3), U?.5 (D3)
- new net ROM4: R?.2, U31.14 (I/O4), U?.6 (A4), U?.6 (A4), U?.6 (D4)
- new net ROM5: R?.2, U31.15 (I/O5), U?.7 (A5), U?.7 (A5), U?.7 (D5)
- new net ROM6: R?.2, U31.16 (I/O6), U?.8 (A6), U?.8 (A6), U?.8 (D6)
- new net ROM7: R?.2, U31.17 (I/O7), U?.9 (A7), U?.9 (A7), U?.9 (D7)
- new net ROM8: R?.2, U30.9 (I/O0), U?.2 (A0), U?.2 (D0)
- new net ROM9: R?.2, U30.10 (I/O1), U?.3 (A1), U?.3 (D1)
- new net ~ROMAO: U?.19 (CE), U?.19 (CE)
- new net ~ROMDO: U?.19 (CE)
- no-connect marks 11 -> 17
Other:
- note added: "ACHTUNG! \nEIGENTLICH 74FCT2574T\n=> gleiches pinout"
- note added: "BUS LEDs"
- note added: "INSTRUCTION REGISTER (LEDs)\n\n\n"
- note added: "INSTRUCTION REGISTER\n\n"
- note added: "ROM (LEDs)\n\n"
- note added: "ROM (output control)\n"
- note added: "ROM\n"
- note removed: "ACHTUNG! \nEIGENTLICH 74FCT2574T\n=> geliches pinout"
- moved on the sheet: D61, D62, D63, D64, D65, D66, D67, D68, Q1, R37, R62, R63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

Commit message: started making uINST
Parts:
- added U? (x3): INTEL2716, symbol custom:INTEL2716
- U9: symbol 4xxx_IEEE_:4068 -> SPU2-rescue:4068-4xxx_IEEE_
- gave numbers to parts that had none: 111
Connections:
- net +5V: now also U40.1 (~MR), U40.10 (CET), U40.16 (VCC), U40.7 (CEP), U?.21 (VPP), U?.21 (VPP), U?.21 (VPP), U?.24 (VCC), U?.24 (VCC), U?.24 (VCC)
- net CE: now also U?.9 (O0)
- net D0: now also U26.4 (D0)
- net D1: now also U26.6 (D1)
- net D2: now also U26.10 (D2)
- net D3: now also U26.12 (D3)
- net D4: now also U27.4 (D0)
- net D5: now also U27.6 (D1)
- net D6: now also U27.10 (D2)
- net D7: now also U27.12 (D3)
- net GND: now also U40.3 (D0), U40.4 (D1), U40.5 (D2), U40.6 (D3), U40.8 (GND), U?.12 (GND), U?.12 (GND), U?.12 (GND), U?.18 (~CE), U?.18 (~CE), U?.18 (~CE), U?.20 (~OE), U?.20 (~OE), U?.20 (~OE)
- net II: now also U?.13 (O3)
- net OP0: now also U?.8 (A0), U?.8 (A0), U?.8 (A0)
- net OP1: now also U?.7 (A1), U?.7 (A1), U?.7 (A1)
- net OP2: now also U?.6 (A2), U?.6 (A2), U?.6 (A2)
- net OP3: now also U?.5 (A3), U?.5 (A3), U?.5 (A3)
- net SU: now also U?.17 (O7)
- net carry: now also U?.22 (A9), U?.22 (A9), U?.22 (A9)
- net at U40.11 (Q3): now also U?.1 (A7), U?.1 (A7), U?.1 (A7)
- net at U40.12 (Q2): now also U?.2 (A6), U?.2 (A6), U?.2 (A6)
- net at U40.13 (Q1): now also U?.3 (A5), U?.3 (A5), U?.3 (A5)
- net at U40.14 (Q0): now also U?.4 (A4), U?.4 (A4), U?.4 (A4)
- net ~clk: now reaches U40.2 (CP)
- net at U40.9 (~PE): now also U?.17 (O7)
- new net AI: U?.13 (O3)
- new net AO: U?.14 (O4)
- new net BI: U?.10 (O1)
- new net BO: U?.11 (O2)
- new net EO: U?.9 (O0)
- new net EXT: U?.13 (O3)
- new net GFXI: U?.17 (O7)
- new net HLT: U?.16 (O6)
- new net J: U?.10 (O1)
- new net JI: U?.9 (O0)
- new net JO: U?.10 (O1)
- new net MC: U?.15 (O5)
- new net PO: U?.11 (O2)
- new net RAMI: U?.15 (O5)
- new net RAMO: U?.16 (O6)
- new net ROMAO: U?.11 (O2)
- new net ROMDO: U?.14 (O4)
- new net eql: U?.19 (A10), U?.19 (A10), U?.19 (A10)
- new net zero: U?.23 (A8), U?.23 (A8), U?.23 (A8)
- no-connect marks 17 -> 18
Other:
- moved on the sheet: U40
