File: Hardware/SPU2/SPU2.sch (KiCad schematic (older format))
At the start: 294 parts, among them Q1 BC547, U1 74LS86, U10 74LS08, U11 74LS173, U12 74LS173, U13 74LS161, U14 74LS161, U15 74LS161, U16 74LS173, U17 74LS173, U18 74HCT574, U19 74LS173, U2 74LS86, U20 74LS173, U21 74LS173, U22 74LS173, U23 74LS173, U24 74LS173, U25 74LS245, U26 74LS189, U27 74LS189, U28 74LS245, U29 74LS540, U3 74LS245, U30 28c16, U31 28c16, U32 74LS245, U33 74LS245, U34 74LS245, U35 74LS245, U36 74LS245, U37 74LS08, U38 74HCT574, U39 74HCT574, U4 74LS283, U40 74LS161, U5 74LS283, U6 4077, U7 4077, U8 74LS02, U9 4068

Commit message: finished uINST in schematic
Parts:
- added U? (x6): 74LS245, symbol 74xx:74LS245
Connections:
- net labels added: GFX, GFX0, GFX1, GFX2, GFX3
- wire segments 1579 -> 1681
- no-connect marks 18 -> 30
Other:
- note added: "MICRO-INSTRUCTION MANAGER"
- moved on the sheet: U40, U?

Commit message: finished schematic
Parts:
- removed U18: 74HCT574, symbol 74xx:74HCT574
- added C10, C12, C13, C15: C, symbol Device:C
- added C11, C14, C16, C17, C18, C19, C20: CP, symbol Device:CP
- added D121, D122, D123, D124, D125, D126, D127, D128, D129, D130, D131, D132, D133, D134, D135, D136, D137, D138, D139, D140, D141, D142, D143, D144, D145, D146, D147, D148, D149, D150, D151, D152, D153, D154, D155, D156, D157, D158, D159, D160, D161, D162, D163, D164, D165, D166, D167, D168, D169, D170, D171, D172, D173, D174, D175, D176, D177, D178, D179, D180, D181, D182, D183, D184, D185, D186, D187, D188, D189, D190, D191, D192, D193, D194, D195, D196, D197, D198, D199, D200, D201, D202, D203, D204, D205, D206, D207, D208, D209, D210, D211, D212, D213, D214, D215, D216, D217, D218, D219, D220, D221, D222, D223, D224, D225, D226, D227, D228, D229, D230, D231, D232, D233, D234, D235, D236, D237, D238, D239, D240, D241, D242, D243, D244, D245, D246, D247, D248, D249: LED, symbol Device:LED
- added F1: Fuse, symbol Device:Fuse
- added J1: Conn_02x01_Row_Letter_First, symbol Connector_Generic:Conn_02x01_Row_Letter_First
- added J2: Conn_02x13_Counter_Clockwise, symbol Connector_Generic:Conn_02x13_Counter_Clockwise
- added J3: Conn_01x02, symbol Connector_Generic:Conn_01x02
- added Q2, Q3, Q4: BC547, Package_TO_SOT_THT:TO-92_Inline, symbol Transistor_BJT:BC547
- added R122, R123, R124, R125, R126, R127, R128, R129, R130, R131, R132, R133, R134, R135, R136, R137, R138, R139, R140, R141, R142, R143, R144, R145, R146, R147, R148, R149, R150, R151, R152, R153, R154, R155, R156, R157, R158, R159, R160, R161, R162, R163, R164, R165, R166, R167, R168, R169, R170, R171, R172, R173, R174, R175, R176, R177, R178, R179, R180, R181, R182, R183, R184, R185, R186, R187, R188, R189, R190, R191, R192, R193, R194, R195, R196, R197, R198, R199, R200, R201, R202, R203, R204, R205, R206, R207, R208, R209, R210, R211, R212, R213, R214, R215, R216, R217, R218, R219, R220, R221, R222, R223, R224, R225, R226, R227, R228, R229, R230, R231, R232, R233, R234, R235, R236, R237, R238, R239, R240, R241, R242, R243, R244, R245, R246, R247, R248, R249, R250, R251, R252, R253, R254, R255, R256, R257, R258, R259, R260, R261: R, symbol Device:R
- added RV1: R_POT, symbol Device:R_POT
- added SW1: SW_Push, symbol Switch:SW_Push
- added SW2: SW_SPDT, symbol Switch:SW_SPDT
- added U18, U43, U44: NE555, symbol Timer:NE555
- added U41: 74LS04, symbol 74xx:74LS04
- added U42, U62, U64, U65, U66, U67: 74LS08, symbol 74xx:74LS08
- added U45, U46, U47, U48, U49, U50, U51, U52, U53, U54, U55, U56, U57, U58, U59, U60: 74HCT574, symbol 74xx:74HCT574
- added U69: CD4514B, symbol custom:CD4514B
- gave numbers to parts that had none: 9
Connections:
- net labels added: CARRY, GFXC0, GFXC1, GFXC10, GFXC11, GFXC12, GFXC13, GFXC14, GFXC15, GFXC2, GFXC3, GFXC4, GFXC5, GFXC6, GFXC7, GFXC8, GFXC9, GFXCLK, ~AO, ~BO, ~CLK
- net labels removed: AI, AO, BI, BO, EO, J, JI, JO, MC, PO, RAMI, RAMO, ROMAO, ROMDO, carry, eql, zero, ~clk
- wire segments 1681 -> 2519
- no-connect marks 30 -> 37
Other:
- note added: "CLOCK\n"
- note added: "GFX Logic\n"
- note added: "GFX Matrix\n"
- note added: "architecture diagram\n\n"
- note added: "parallel bus interface\n"
- note added: "power supply\n"
- moved on the sheet: D100, D85, D86, D87, D88, D89, D90, D91, D92, D93, D94, D95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

Commit message: mach du mal
Parts:
- removed C1, C16, C18, C19, C2, C3, C4, C5, C6, C7, C8, C9: CP, symbol Device:CP
- added C? (x75): C, symbol Device:C
- added J?: Conn_01x04_Male, symbol Connector:Conn_01x04_Male
Connections:
- wire segments 2519 -> 2513
Other:
- note added: "Aufsteck Clock module \n=> Inverter mit RC Glied"
- note added: "SMA\n"
- moved on the sheet: J1

Commit message: enlarged ram to 2k16 and added support for running code from ram
Parts:
- removed C? (x3): C, symbol Device:C
- removed D61, D62, D63, D64, D65, D66, D67, D68: LED, symbol Device:LED
- removed Q1: BC547, Package_TO_SOT_THT:TO-92_Inline, symbol Transistor_BJT:BC547
- removed R37, R62, R63, R64, R65, R66, R67, R68, R69: R, symbol Device:R
- removed U26, U27: 74LS189, symbol custom:74LS189
- removed U29: 74LS540, symbol 74xx:74LS540
- added C? (x7): C, symbol Device:C
- added D? (x32): LED, symbol Device:LED
- added R? (x32): R, symbol Device:R
- added U? (x2): M84Z02, symbol custom:M84Z02
- added U? (x5): 74LS00, symbol 74xx:74LS00
- added U? (x4): 74LS157, symbol 74xx:74LS157
Connections:
- net labels added: MEM, MEM0, MEM1, MEM10, MEM11, MEM12, MEM13, MEM14, MEM15, MEM2, MEM3, MEM4, MEM5, MEM6, MEM7, MEM8, MEM9, RAMI, RAMOBUS, RAMOBUS0, RAMOBUS1, RAMOBUS10, RAMOBUS11, RAMOBUS12, RAMOBUS13, RAMOBUS14, RAMOBUS15, RAMOBUS2, RAMOBUS3, RAMOBUS4, RAMOBUS5, RAMOBUS6, RAMOBUS7, RAMOBUS8, RAMOBUS9, ~MEMAO, ~MEMDO
- net labels removed: ~AO, ~BO, ~RAMI, ~RAMO, ~ROMAO, ~ROMDO
- wire segments 2513 -> 2687
- no-connect marks 37 -> 49
Other:
- moved on the sheet: C?, D122, D123, D124, D125, D126, D127, D128, D129, D130, D131, D132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

Commit message: upgraded rom to 8k8, ability to hold 4 programs at once
Parts:
- removed C? (x2): C, symbol Device:C
- removed U30, U31: 28c16, symbol custom:28c16
- added C? (x4): C, symbol Device:C
- added R? (x2): R, symbol Device:R
- added SW?: SW_DIP_x02, symbol Switch:SW_DIP_x02
- added U? (x2): 28c16, symbol custom:28c16
- added U? (x2): 28c64, symbol custom:28c64
Connections:
- wire segments 2687 -> 2801
Other:
- note added: "MEM (output control)\n"
- note added: "address space control"
- note added: "altes rom\nNICHT EINBAUEN!"
- note added: "ram leds"
- note added: "übrige nand gates (für ram)"
- note removed: "ROM (output control)\n"
- moved on the sheet: C?

Commit message: updated compiler; minor efficiency improvements in schematic
Parts:
- removed C?: C, symbol Device:C
- removed U70: 74LS245, symbol 74xx:74LS245
- U18, U43, U44: symbol Timer:NE555 -> SPU2-rescue:NE555-Timer
Connections:
- wire segments 2801 -> 2786
- no-connect marks 49 -> 41

Commit message: assigned footprints
Parts:
- removed C? (x2): C, symbol Device:C
- removed U? (x2): 28c16, symbol custom:28c16
- C1, C16, C18, C19, C2, C21, C22, C23, C24, C25, C26, C27, C28, C29, C3, C30, C31, C32, C33, C34, C35, C36, C37, C38, C39, C4, C40, C41, C42, C43, C44, C45, C46, C47, C48, C49, C5, C50, C51, C52, C53, C54, C55, C56, C57, C58, C59, C6, C60, C61, C62, C63, C64, C65, C66, C67, C68, C69, C7, C70, C71, C72, C73, C74, C75, C76, C77, C78, C79, C8, C80, C81, C82, C83, C84, C85, C86, C9: renamed from C?; footprint (none) -> Capacitor_SMD:C_0805_2012Metric_Pad1.15x1.40mm_HandSolder
- C10, C12, C13, C15: footprint (none) -> Capacitor_SMD:C_0805_2012Metric_Pad1.15x1.40mm_HandSolder
- C11, C14, C17, C20: footprint (none) -> Capacitor_Tantalum_SMD:CP_EIA-6032-15_Kemet-U_Pad2.25x2.35mm_HandSolder
- D1, D10, D100, D101, D102, D103, D104, D105, D106, D107, D108, D109, D11, D110, D111, D112, D113, D114, D115, D116, D117, D118, D119, D12, D120, D121, D122, D123, D124, D125, D126, D127, D128, D129, D13, D130, D131, D132, D133, D134, D135, D136, D137, D138, D139, D14, D140, D141, D142, D143, D144, D145, D146, D147, D148, D149, D15, D150, D151, D152, D153, D154, D155, D156, D157, D158, D159, D16, D160, D161, D162, D163, D164, D165, D166, D167, D168, D169, D17, D170, D171, D172, D173, D174, D175, D176, D177, D178, D179, D18, D180, D181, D182, D183, D184, D185, D186, D187, D188, D189, D19, D190, D191, D192, D193, D194, D195, D196, D197, D198, D199, D2, D20, D200, D201, D202, D203, D204, D205, D206, D207, D208, D209, D21, D210, D211, D212, D213, D214, D215, D216, D217, D218, D219, D22, D220, D221, D222, D223, D224, D225, D226, D227, D228, D229, D23, D230, D231, D232, D233, D234, D235, D236, D237, D238, D239, D24, D240, D241, D242, D243, D244, D245, D246, D247, D248, D249, D25, D26, D27, D28, D29, D3, D30, D31, D32, D33, D34, D35, D36, D37, D38, D39, D4, D40, D41, D42, D43, D44, D45, D46, D47, D48, D49, D5, D50, D51, D52, D53, D54, D55, D56, D57, D58, D59, D6, D60, D69, D7, D70, D71, D72, D73, D74, D75, D76, D77, D78, D79, D8, D80, D81, D82, D83, D84, D85, D86, D87, D88, D89, D9, D90, D91, D92, D93, D94, D95, D96, D97, D98, D99: footprint (none) -> LED_THT:LED_D5.0mm
- D250, D251, D252, D253, D254, D255, D256, D257, D258, D259, D260, D261, D262, D263, D264, D265, D266, D267, D268, D269, D270, D271, D272, D273, D61, D62, D63, D64, D65, D66, D67, D68: renamed from D?; footprint (none) -> LED_THT:LED_D5.0mm
- F1: footprint (none) -> Fuse:Fuse_1812_4532Metric_Pad1.30x3.40mm_HandSolder
- J1: footprint (none) -> Connector_Coaxial:SMA_Amphenol_132203-12_Horizontal
- J2: footprint (none) -> Connector_PinHeader_2.54mm:PinHeader_2x13_P2.54mm_Vertical
- J3: footprint (none) -> Connector_AMASS:AMASS_XT30U-F_1x02_P5.0mm_Vertical
- J4: renamed from J?; footprint (none) -> Connector_PinHeader_2.54mm:PinHeader_1x04_P2.54mm_Vertical
- R1, R10, R100, R101, R102, R103, R104, R105, R106, R107, R108, R109, R11, R110, R111, R112, R113, R114, R115, R116, R117, R118, R119, R12, R120, R121, R122, R123, R124, R125, R126, R127, R128, R129, R13, R130, R131, R132, R133, R134, R135, R136, R137, R138, R139, R14, R140, R141, R142, R143, R144, R145, R146, R147, R148, R149, R15, R150, R151, R152, R153, R154, R155, R156, R157, R158, R159, R16, R160, R161, R162, R163, R164, R165, R166, R167, R168, R169, R17, R170, R171, R172, R173, R174, R175, R176, R177, R178, R179, R18, R180, R181, R182, R183, R184, R185, R186, R187, R188, R189, R19, R190, R191, R192, R193, R194, R195, R196, R197, R198, R199, R2, R20, R200, R201, R202, R203, R204, R205, R206, R207, R208, R209, R21, R210, R211, R212, R213, R214, R215, R216, R217, R218, R219, R22, R220, R221, R222, R223, R224, R225, R226, R227, R23, R24, R25, R26, R27, R28, R29, R3, R30, R31, R32, R33, R34, R35, R36, R38, R39, R4, R40, R41, R42, R43, R44, R45, R46, R47, R48, R49, R5, R50, R51, R52, R53, R54, R55, R56, R57, R58, R59, R6, R60, R61, R7, R70, R71, R72, R73, R74, R75, R76, R77, R78, R79, R8, R80, R81, R82, R83, R84, R85, R86, R87, R88, R89, R9, R90, R91, R92, R93, R94, R95, R96, R97, R98, R99: footprint (none) -> Resistor_SMD:R_0805_2012Metric_Pad1.15x1.40mm_HandSolder
- R228, R229, R230, R231, R232, R233, R234, R235, R236, R237, R238, R239, R240, R241, R242, R243, R244, R245, R246, R247, R248, R249, R250, R251, R252, R253, R254, R255, R256, R257, R258, R259, R260, R261: footprint (none) -> Resistor_SMD:R_0815_2038Metric_Pad1.53x4.00mm_HandSolder
- R262, R263, R264, R265, R266, R267, R268, R269, R270, R271, R272, R273, R274, R275, R276, R277, R278, R279, R280, R281, R282, R283, R284, R285, R286: renamed from R?; footprint (none) -> Resistor_SMD:R_0815_2038Metric_Pad1.53x4.00mm_HandSolder
- R37, R62, R63, R64, R65, R66, R67, R68, R69: renamed from R?; footprint (none) -> Resistor_SMD:R_0805_2012Metric_Pad1.15x1.40mm_HandSolder
- RV1: footprint (none) -> Potentiometer_THT:Potentiometer_Piher_PT-15-V02_Vertical
- SW1: footprint (none) -> Button_Switch_SMD:Panasonic_EVQPUK_EVQPUB
- SW2: footprint (none) -> Button_Switch_THT:Nidec_Copal_SH-7010C
- SW3: renamed from SW?; footprint (none) -> Button_Switch_THT:SW_DIP_SPSTx02_Slide_9.78x7.26mm_W7.62mm_P2.54mm
- U1, U10, U2, U37, U41, U42, U6, U62, U64, U65, U66, U67, U7, U8, U9: footprint (none) -> Package_DIP:DIP-14_W7.62mm_Socket_LongPads
- U11, U12, U13, U14, U15, U16, U17, U19, U20, U21, U22, U23, U24, U4, U40, U5: footprint (none) -> Package_DIP:DIP-16_W7.62mm_Socket_LongPads
- U18, U43, U44: footprint (none) -> Package_DIP:DIP-8_W7.62mm
- U25, U28, U3, U32, U33, U34, U35, U36, U71, U72, U73, U74, U75: footprint (none) -> Package_DIP:DIP-20_W7.62mm_Socket_LongPads
- U26, U27: renamed from U?; footprint (none) -> Package_DIP:DIP-24_W15.24mm_Socket_LongPads
- U29: renamed from U?; footprint (none) -> Package_DIP:DIP-14_W7.62mm_Socket_LongPads
- U30, U31: renamed from U?; footprint (none) -> Package_DIP:DIP-28_W15.24mm_Socket_LongPads
- U38, U39, U45, U46, U47, U48, U49, U50, U51, U52, U53, U54, U55, U56, U57, U58, U59, U60: footprint (none) -> Package_SO:SOIC-20W_7.5x12.8mm_P1.27mm
- U61, U63, U68, U69: footprint (none) -> Package_DIP:DIP-24_W15.24mm_Socket_LongPads
- U70, U76, U77, U78: renamed from U?; footprint (none) -> Package_DIP:DIP-16_W7.62mm_Socket_LongPads
Connections:
- net +5V: now also U31.28 (VCC)
- net ADDR0: now also U30.10 (A0), U31.10 (A0)
- net ADDR1: now also U30.9 (A1), U31.9 (A1)
- net ADDR2: now also U30.8 (A2), U31.8 (A2)
- net ADDR3: now also U30.7 (A3), U31.7 (A3)
- net ADDR4: now also U30.6 (A4), U31.6 (A4)
- net ADDR5: now also U30.5 (A5), U31.5 (A5)
- net ADDR6: now also U30.4 (A6), U31.4 (A6)
- net ADDR7: now also U30.3 (A7), U31.3 (A7)
Other:
- note removed: "altes rom\nNICHT EINBAUEN!"
- moved on the sheet: C86, D258, D259, D260, D261, D262, D263, D264, D265, D266, D267, D268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

Commit message: random push
Parts:
- removed C20: CP, Capacitor_Tantalum_SMD:CP_EIA-6032-15_Kemet-U_Pad2.25x2.35mm_HandSolder, symbol Device:CP
- removed C77, C78, C79, C80, C81: C, Capacitor_SMD:C_0805_2012Metric_Pad1.15x1.40mm_HandSolder, symbol Device:C
- removed J1: Conn_02x01_Row_Letter_First, Connector_Coaxial:SMA_Amphenol_132203-12_Horizontal, symbol Connector_Generic:Conn_02x01_Row_Letter_First
- removed U71, U72, U73, U74, U75: 74LS245, Package_DIP:DIP-20_W7.62mm_Socket_LongPads, symbol 74xx:74LS245
- added C? (x5): C, Capacitor_SMD:C_0805_2012Metric_Pad1.15x1.40mm_HandSolder, symbol Device:C
- added D274: LED, LED_THT:LED_D5.0mm, symbol Device:LED
- added J1: Conn_Coaxial, Connector_Coaxial:SMA_Amphenol_132134-16_Vertical, symbol Connector:Conn_Coaxial
- added R287: R, Resistor_SMD:R_0805_2012Metric_Pad1.15x1.40mm_HandSolder, symbol Device:R
- added U? (x5): 74LS245, Package_DIP:DIP-20_W7.62mm_Socket_LongPads, symbol 74xx:74LS245
- R228, R229, R230, R231, R232, R233, R234, R235, R236, R237, R238, R239, R240, R241, R242, R243, R244, R245, R246, R247, R248, R249, R250, R251, R252, R253, R254, R255, R256, R257, R258, R259, R260, R261, R262, R263, R264, R265, R266, R267, R268, R269, R270, R271, R272, R273, R274, R275, R276, R277, R278, R279, R280, R281, R282, R283, R284, R285, R286: footprint Resistor_SMD:R_0815_2038Metric_Pad1.53x4.00mm_HandSolder -> Resistor_SMD:R_0805_2012Metric_Pad1.15x1.40mm_HandSolder
- SW2: footprint Button_Switch_THT:Nidec_Copal_SH-7010C -> Button_Switch_THT:SW_CuK_OS102011MA1QN1_SPDT_Angled
Connections:
- net +5V: now also C?.1, C?.1, C?.1, C?.1, C?.1, R287.2, U?.1 (A->B), U?.1 (A->B), U?.1 (A->B), U?.1 (A->B), U?.1 (A->B), U?.20 (VCC), U?.20 (VCC), U?.20 (VCC), U?.20 (VCC), U?.20 (VCC), U?.6 (A4), U?.7 (A5), U?.8 (A6)
- net ADDR0: now also U?.18 (B0), U?.18 (B0)
- net ADDR1: now also U?.17 (B1), U?.17 (B1)
- net ADDR10: now also U?.12 (B6), U?.16 (B2)
- net ADDR11: now also U?.11 (B7), U?.15 (B3)
- net ADDR2: now also U?.16 (B2), U?.16 (B2)
- net ADDR3: now also U?.15 (B3), U?.15 (B3)
- net ADDR4: now also U?.14 (B4), U?.14 (B4)
- net ADDR5: now also U?.13 (B5), U?.13 (B5)
- net ADDR6: now also U?.12 (B6), U?.12 (B6)
- net ADDR7: now also U?.11 (B7), U?.11 (B7)
- net ADDR8: now also U?.14 (B4), U?.18 (B0)
- net ADDR9: now also U?.13 (B5), U?.17 (B1)
- net ARG0: now also U?.2 (A0), U?.2 (A0), U?.2 (A0)
- net ARG1: now also U?.3 (A1), U?.3 (A1), U?.3 (A1)
- net ARG10: now also U?.4 (A2), U?.4 (A2)
- net ARG11: now also U?.5 (A3), U?.5 (A3)
- net ARG2: now also U?.4 (A2), U?.4 (A2), U?.4 (A2)
- net ARG3: now also U?.5 (A3), U?.5 (A3), U?.5 (A3)
- net ARG4: now also U?.6 (A4), U?.6 (A4), U?.6 (A4)
- net ARG5: now also U?.7 (A5), U?.7 (A5), U?.7 (A5)
- net ARG6: now also U?.8 (A6), U?.8 (A6), U?.8 (A6)
- net ARG7: now also U?.9 (A7), U?.9 (A7), U?.9 (A7)
- net ARG8: now also U?.2 (A0), U?.2 (A0)
- net ARG9: now also U?.3 (A1), U?.3 (A1)
- net D0: now also U?.18 (B0)
- net D1: now also U?.17 (B1)
- net D2: now also U?.16 (B2)
- net D3: now also U?.15 (B3)
- net D4: now also U?.14 (B4)
- net D5: now also U?.13 (B5)
- net D6: now also U?.12 (B6)
- net D7: now also U?.11 (B7)
- net GFX0: now also U?.18 (B0)
- net GFX1: now also U?.17 (B1)
- net GFX2: now also U?.16 (B2)
- net GFX3: now also U?.15 (B3)
- net GND: now also C?.2, C?.2, C?.2, C?.2, C?.2, D274.1 (K), J1.2 (Ext), U?.10 (GND), U?.10 (GND), U?.10 (GND), U?.10 (GND), U?.10 (GND), U?.6 (A4), U?.7 (A5), U?.8 (A6), U?.9 (A7), U?.9 (A7); no longer D178.1 (K), D179.1 (K), D180.1 (K), D181.1 (K), D183.1 (K), D185.1 (K), D187.1 (K), D189.1 (K)
- net at U68.14 (O4): now also U?.19 (CE)
- net at U68.15 (O5): now also U?.19 (CE), U?.19 (CE)
- net at U68.16 (O6): now also U?.19 (CE), U?.19 (CE)
- net NE555A: now reaches U18.3 (Q), U42.1
- net NE555B: now reaches U42.10, U43.3 (Q)
- net NE555C: now reaches U41.1, U42.2, U44.3 (Q)
- net at J4.3 (Pin_3), R128.2: now also J1.1 (In)
- new net: D274.2 (A), R287.1
- new net: D178.1 (K), D179.1 (K), D180.1 (K), D181.1 (K), D183.1 (K), D185.1 (K), D187.1 (K), D189.1 (K)
Other:
- note removed: "SMA\n"
- moved on the sheet: C1, C10, C11, C12, C13, C15, C17, C18, C19, C22, C23, C24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
