File: Hardware/SPU2/SPU2.kicad_pcb (KiCad board)
At the start: 2 copper layers, 737 parts, among them J1 Conn_Coaxial, J2 Conn_02x13_Counter_Clockwise, J3 Conn_01x02, J4 Conn_01x04_Male, Q2 BC547, Q3 BC547, Q4 BC547, SW1 SW_Push, SW2 SW_SPDT, SW3 SW_DIP_x02, U1 74LS86, U10 74LS08, U11 74LS173, U12 74LS173, U13 74LS161, U14 74LS161, U15 74LS161, U16 74LS173, U17 74LS173, U18 NE555, U19 74LS173, U2 74LS86, U20 74LS173, U21 74LS173, U22 74LS173, U23 74LS173, U24 74LS173, U25 74LS245, U26 M84Z02, U27 M84Z02, U28 74LS245, U29 74LS00, U3 74LS245, U30 28c64, U31 28c64, U32 74LS245, U33 74LS245, U34 74LS245, U35 74LS245, U36 74LS245, U37 74LS08, U38 74HCT574, U39 74HCT574, U4 74LS283, U40 74LS161, U41 74LS04, U42 74LS08, U43 NE555, U44 NE555, U45 74HCT574, U46 74HCT574, U47 74HCT574, U48 74HCT574, U49 74HCT574, U5 74LS283, U50 74HCT574, U51 74HCT574, U52 74HCT574, U53 74HCT574, U54 74HCT574, U55 74HCT574, U56 74HCT574, U57 74HCT574, U58 74HCT574, U59 74HCT574, U6 4077, U60 74HCT574, U61 INTEL2716, U62 74LS08, U63 INTEL2716, U64 74LS08, U65 74LS08, U66 74LS08, U67 74LS08, U68 INTEL2716, U69 CD4514B, U7 4077, U70 74LS157, U71 74LS245, U72 74LS245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

Commit message: done stuff
Parts:
- removed C81: C, Capacitor_SMD:C_0805_2012Metric_Pad1.15x1.40mm_HandSolder
- C20: value CP -> C; footprint Capacitor_Tantalum_SMD:CP_EIA-6032-15_Kemet-U_Pad2.25x2.35mm_HandSolder -> Capacitor_SMD:C_0805_2012Metric_Pad1.15x1.40mm_HandSolder
- moved R84 394.9 mm to (220.2, 29.7), turned to 270 degrees
- moved R85 380.9 mm to (218.2, 29.7), turned to 270 degrees
- moved R81 359.2 mm to (226.2, 29.7), turned to 270 degrees
- moved R82 355.1 mm to (224.2, 29.7), turned to 270 degrees
- moved R80 329.1 mm to (228.1, 29.7), turned to 270 degrees
- moved R70 322.9 mm to (247.9, 29.7), turned to 270 degrees
- moved R78 322.5 mm to (232.1, 29.7), turned to 270 degrees
- moved R83 320.9 mm to (222.2, 29.7), turned to 270 degrees
- moved R76 314.4 mm to (236.1, 29.7), turned to 270 degrees
- moved R73 312.6 mm to (242.0, 29.7), turned to 270 degrees
- moved C59 311.3 mm to (314.8, 172.4)
- moved R79 305.6 mm to (230.1, 29.7), turned to 270 degrees
- moved R72 305.5 mm to (244.0, 29.7), turned to 270 degrees
- moved R77 304.2 mm to (234.1, 29.7), turned to 270 degrees
- moved R71 299.9 mm to (245.9, 29.7), turned to 270 degrees
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Connections:
- net Net-(R125-Pad2) renamed NE555_CLK
- net Net-(U18-Pad3) renamed NE555A
- net Net-(U41-Pad1) renamed NE555C
- net Net-(U42-Pad10) renamed NE555B
- D122 pad 1: GND -> Net-(D122-Pad1)
- D123 pad 1: GND -> Net-(D123-Pad1)
- D124 pad 1: GND -> Net-(D124-Pad1)
- D125 pad 1: GND -> Net-(D125-Pad1)
- D126 pad 1: GND -> Net-(D126-Pad1)
- D127 pad 1: GND -> Net-(D127-Pad1)
- D128 pad 1: GND -> Net-(D128-Pad1)
- D129 pad 1: GND -> Net-(D129-Pad1)
- D178 pad 1: GND -> Net-(D178-Pad1)
- D179 pad 1: GND -> Net-(D178-Pad1)
- D180 pad 1: GND -> Net-(D178-Pad1)
- D181 pad 1: GND -> Net-(D178-Pad1)
- D183 pad 1: GND -> Net-(D178-Pad1)
- D185 pad 1: GND -> Net-(D178-Pad1)
- D187 pad 1: GND -> Net-(D178-Pad1)
- D189 pad 1: GND -> Net-(D178-Pad1)
- U70 pad 10: /RAMOBUS2 -> /ROM2
- U70 pad 11: /ROM2 -> /RAMOBUS2
- U70 pad 13: /RAMOBUS3 -> /ROM3
- U70 pad 14: /ROM3 -> /RAMOBUS3
- U70 pad 2: /ROM0 -> /RAMOBUS0
- U70 pad 3: /RAMOBUS0 -> /ROM0
- U70 pad 5: /ROM1 -> /RAMOBUS1
- U70 pad 6: /RAMOBUS1 -> /ROM1
- U71 pad 11: /ADDR11 -> /D7
- U71 pad 12: /ADDR10 -> /D6
- U71 pad 13: /ADDR9 -> /D5
- U71 pad 14: /ADDR8 -> /D4
- U71 pad 15: /GFX3 -> /D3
- U71 pad 16: /GFX2 -> /D2
- U71 pad 17: /GFX1 -> /D1
- U71 pad 18: /GFX0 -> /D0
- U71 pad 19: Net-(U68-Pad16) -> Net-(U68-Pad14)
- U71 pad 2: /ARG8 -> /ARG0
- U71 pad 3: /ARG9 -> /ARG1
- U71 pad 4: /ARG10 -> /ARG2
- U71 pad 5: /ARG11 -> /ARG3
- U71 pad 6: +5V -> /ARG4
- U71 pad 7: +5V -> /ARG5
- U71 pad 8: +5V -> /ARG6
- U71 pad 9: GND -> /ARG7
- U72 pad 11: /ADDR7 -> Net-(U72-Pad11)
- U72 pad 12: /ADDR6 -> Net-(U72-Pad12)
- U72 pad 13: /ADDR5 -> Net-(U72-Pad13)
- U72 pad 14: /ADDR4 -> Net-(U72-Pad14)
- U72 pad 15: /ADDR3 -> /ADDR11
- U72 pad 16: /ADDR2 -> /ADDR10
- U72 pad 17: /ADDR1 -> /ADDR9
- U72 pad 18: /ADDR0 -> /ADDR8
- U72 pad 19: Net-(U68-Pad16) -> Net-(U68-Pad15)
- U72 pad 2: /ARG0 -> /ARG8
- U72 pad 3: /ARG1 -> /ARG9
- U72 pad 4: /ARG2 -> /ARG10
- U72 pad 5: /ARG3 -> /ARG11
- U72 pad 6: /ARG4 -> GND
- U72 pad 7: /ARG5 -> GND
- U72 pad 8: /ARG6 -> GND
- U72 pad 9: /ARG7 -> GND
- U73 pad 11: Net-(U73-Pad11) -> /ADDR7
- U73 pad 12: Net-(U73-Pad12) -> /ADDR6
- U73 pad 13: Net-(U73-Pad13) -> /ADDR5
- U73 pad 14: Net-(U73-Pad14) -> /ADDR4
- U73 pad 15: /ADDR11 -> /ADDR3
- U73 pad 16: /ADDR10 -> /ADDR2
- U73 pad 17: /ADDR9 -> /ADDR1
- U73 pad 18: /ADDR8 -> /ADDR0
- U73 pad 2: /ARG8 -> /ARG0
- U73 pad 3: /ARG9 -> /ARG1
- U73 pad 4: /ARG10 -> /ARG2
- U73 pad 5: /ARG11 -> /ARG3
- U73 pad 6: GND -> /ARG4
- U73 pad 7: GND -> /ARG5
- U73 pad 8: GND -> /ARG6
- U73 pad 9: GND -> /ARG7
- U74 pad 11: /ADDR7 -> /ADDR11
- U74 pad 12: /ADDR6 -> /ADDR10
- U74 pad 13: /ADDR5 -> /ADDR9
- U74 pad 14: /ADDR4 -> /ADDR8
- U74 pad 15: /ADDR3 -> /GFX3
- U74 pad 16: /ADDR2 -> /GFX2
- U74 pad 17: /ADDR1 -> /GFX1
- U74 pad 18: /ADDR0 -> /GFX0
- U74 pad 19: Net-(U68-Pad15) -> Net-(U68-Pad16)
- U74 pad 2: /ARG0 -> /ARG8
- U74 pad 3: /ARG1 -> /ARG9
- U74 pad 4: /ARG2 -> /ARG10
- U74 pad 5: /ARG3 -> /ARG11
- U74 pad 6: /ARG4 -> +5V
- U74 pad 7: /ARG5 -> +5V
- U74 pad 8: /ARG6 -> +5V
- U74 pad 9: /ARG7 -> GND
- U75 pad 11: /D7 -> /ADDR7
- U75 pad 12: /D6 -> /ADDR6
- U75 pad 13: /D5 -> /ADDR5
- U75 pad 14: /D4 -> /ADDR4
- U75 pad 15: /D3 -> /ADDR3
- U75 pad 16: /D2 -> /ADDR2
- U75 pad 17: /D1 -> /ADDR1
- U75 pad 18: /D0 -> /ADDR0
- U75 pad 19: Net-(U68-Pad14) -> Net-(U68-Pad16)
- U76 pad 10: /RAMOBUS6 -> /ROM6
- U76 pad 11: /ROM6 -> /RAMOBUS6
- U76 pad 13: /RAMOBUS7 -> /ROM7
- U76 pad 14: /ROM7 -> /RAMOBUS7
- U76 pad 2: /ROM4 -> /RAMOBUS4
- U76 pad 3: /RAMOBUS4 -> /ROM4
- U76 pad 5: /ROM5 -> /RAMOBUS5
- U76 pad 6: /RAMOBUS5 -> /ROM5
- U77 pad 10: /RAMOBUS10 -> /ROM10
- U77 pad 11: /ROM10 -> /RAMOBUS10
- U77 pad 13: /RAMOBUS11 -> /ROM11
- U77 pad 14: /ROM11 -> /RAMOBUS11
- U77 pad 2: /ROM8 -> /RAMOBUS8
- U77 pad 3: /RAMOBUS8 -> /ROM8
- U77 pad 5: /ROM9 -> /RAMOBUS9
- U77 pad 6: /RAMOBUS9 -> /ROM9
- U78 pad 10: /RAMOBUS14 -> /ROM14
- U78 pad 11: /ROM14 -> /RAMOBUS14
- U78 pad 13: /RAMOBUS15 -> /ROM15
- U78 pad 14: /ROM15 -> /RAMOBUS15
- U78 pad 2: /ROM12 -> /RAMOBUS12
- U78 pad 3: /RAMOBUS12 -> /ROM12
- U78 pad 5: /ROM13 -> /RAMOBUS13
- U78 pad 6: /RAMOBUS13 -> /ROM13
Routing:
- net /ADDR0: track 61.9 -> 302.6 mm, vias 0 -> 7
- net /ADDR1: track 59.2 -> 296.9 mm, vias 0 -> 9
- net /ADDR6: track 32.0 -> 236.4 mm, vias 0 -> 9
- net /ADDR2: track 101.1 -> 290.0 mm, vias 0 -> 9
- net /ADDR3: track 94.8 -> 283.2 mm, vias 0 -> 9
- net /ADDR4: track 63.8 -> 250.3 mm, vias 0 -> 9
- net /ADDR10: track 18.0 -> 203.3 mm, vias 0 -> 11
- net /ADDR5: track 58.5 -> 243.4 mm, vias 0 -> 9
- net /ADDR7: track 47.9 -> 230.3 mm, vias 0 -> 9
- net /ADDR9: track 23.6 -> 201.1 mm, vias 0 -> 11
- net /ADDR8: track 29.0 -> 203.5 mm, vias 0 -> 9
- net /ROM0: track 0.00 -> 161.6 mm, vias 0 -> 1
- net /ROM1: track 0.00 -> 160.5 mm, vias 0 -> 1
- net /ROM2: track 0.00 -> 159.3 mm, vias 0 -> 1
- net /ADDR11: track 12.7 -> 129.0 mm, vias 0 -> 7
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
Commit message: existance is pain
Parts:
- moved R45 335.1 mm to (239.0, 32.1), turned to 270 degrees
- moved R48 332.0 mm to (219.0, 32.1), turned to 270 degrees
- moved R47 328.0 mm to (225.7, 32.1), turned to 270 degrees
- moved R44 315.1 mm to (245.7, 32.1), turned to 270 degrees
- moved C26 312.9 mm to (214.5, 49.1), turned to 270 degrees
- moved R42 299.4 mm to (259.1, 32.1), turned to 270 degrees
- moved R49 291.4 mm to (212.4, 32.1), turned to 270 degrees
- moved R43 290.7 mm to (251.9, 32.1), turned to 270 degrees
- moved R40 283.3 mm to (272.0, 32.1), turned to 270 degrees
- moved R46 278.7 mm to (232.3, 32.1), turned to 270 degrees
- moved D44 272.4 mm to (238.8, 25.2), turned to 270 degrees
- moved D46 271.3 mm to (225.7, 25.2), turned to 270 degrees
- moved D48 268.1 mm to (212.5, 25.2), turned to 270 degrees
- moved R41 255.2 mm to (265.2, 32.0), turned to 270 degrees
- moved D47 249.8 mm to (219.1, 25.2), turned to 270 degrees
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Connections:
- U30 pad 10: /ADDR0 -> /MEMADDR0
- U30 pad 21: /ADDR10 -> /MEMADDR10
- U30 pad 24: /ADDR9 -> /MEMADDR9
- U30 pad 25: /ADDR8 -> /MEMADDR8
- U30 pad 3: /ADDR7 -> /MEMADDR7
- U30 pad 4: /ADDR6 -> /MEMADDR6
- U30 pad 5: /ADDR5 -> /MEMADDR5
- U30 pad 6: /ADDR4 -> /MEMADDR4
- U30 pad 7: /ADDR3 -> /MEMADDR3
- U30 pad 8: /ADDR2 -> /MEMADDR2
- U30 pad 9: /ADDR1 -> /MEMADDR1
- U31 pad 10: /ADDR0 -> /MEMADDR0
- U31 pad 21: /ADDR10 -> /MEMADDR10
- U31 pad 24: /ADDR9 -> /MEMADDR9
- U31 pad 25: /ADDR8 -> /MEMADDR8
- U31 pad 3: /ADDR7 -> /MEMADDR7
- U31 pad 4: /ADDR6 -> /MEMADDR6
- U31 pad 5: /ADDR5 -> /MEMADDR5
- U31 pad 6: /ADDR4 -> /MEMADDR4
- U31 pad 7: /ADDR3 -> /MEMADDR3
- U31 pad 8: /ADDR2 -> /MEMADDR2
- U31 pad 9: /ADDR1 -> /MEMADDR1
Routing:
- net +5V: track 256.6 -> 753.1 mm, vias 7 -> 11
- net /MEMADDR0: track 0.00 -> 355.0 mm, vias 0 -> 8
- net /MEMADDR1: track 0.00 -> 343.9 mm, vias 0 -> 12
- net /MEMADDR2: track 0.00 -> 330.0 mm, vias 0 -> 12
- net /MEMADDR3: track 0.00 -> 314.6 mm, vias 0 -> 12
- net /MEMADDR10: track 0.00 -> 284.7 mm, vias 0 -> 14
- net /MEMADDR4: track 0.00 -> 275.5 mm, vias 0 -> 12
- net /MEMADDR9: track 0.00 -> 269.0 mm, vias 0 -> 14
- net /MEMADDR5: track 0.00 -> 262.1 mm, vias 0 -> 12
- net /MEMADDR8: track 0.00 -> 260.9 mm, vias 0 -> 12
- net /MEMADDR7: track 0.00 -> 259.5 mm, vias 0 -> 12
- net /MEMADDR6: track 0.00 -> 254.1 mm, vias 0 -> 12
- net /ROM13: track 46.4 -> 266.9 mm, vias 1 -> 5
- net /ROM12: track 46.9 -> 264.4 mm, vias 1 -> 5
- net /ROM14: track 45.8 -> 262.2 mm, vias 1 -> 7
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Other:
- rule via_min_size: 0.4 -> 0.45
- board text added: "ADDRESS BUS"
- board text added: "ADDRESS SPACE CONTOL UNIT"
- board text added: "MEMORY ADDRESS BUS"
- board text added: "MEMORY ADDRESS REGISTER"
- board text added: "PROGRAM COUNTER"
- board text added: "READ ONLY MEMORY 4x 2Kx16"
- board text added: "ROM BUS"

Commit message: random push
Routing:
- net /RAMOBUS14: track 0.00 -> 88.8 mm, vias 0 -> 2
- net /RAMOBUS13: track 0.00 -> 87.0 mm, vias 0 -> 4
- net /RAMOBUS15: track 0.00 -> 84.8 mm, vias 0 -> 2
- net /RAMOBUS12: track 0.00 -> 73.7 mm
- net /RAMOBUS10: track 0.00 -> 67.5 mm, vias 0 -> 2
- net /RAMOBUS9: track 0.00 -> 65.9 mm, vias 0 -> 4
- net /RAMOBUS11: track 0.00 -> 63.3 mm, vias 0 -> 2
- net /RAMOBUS8: track 0.00 -> 52.3 mm
- net /RAMOBUS6: track 0.00 -> 44.2 mm, vias 0 -> 2
- net /RAMOBUS5: track 0.00 -> 42.7 mm, vias 0 -> 4
- net /RAMOBUS7: track 0.00 -> 40.2 mm, vias 0 -> 2
- net /RAMOBUS4: track 0.00 -> 29.2 mm
- net /ROM9: track 251.6 -> 255.0 mm
- net /ROM13: track 266.9 -> 270.0 mm
- net /ROM12: track 264.4 -> 266.3 mm
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
Commit message: done stuff
Parts:
- moved R62 423.1 mm to (327.1, 121.9), turned to 270 degrees
- moved D64 397.5 mm to (333.6, 115.5), turned to 270 degrees
- moved R264 387.8 mm to (359.8, 121.9), turned to 270 degrees
- moved D255 387.3 mm to (366.4, 115.5), turned to 270 degrees
- moved U33 371.7 mm to (509.4, 196.7)
- moved U32 370.5 mm to (499.1, 195.4)
- moved R63 366.1 mm to (386.1, 121.9), turned to 270 degrees
- moved R69 359.6 mm to (405.7, 121.9), turned to 270 degrees
- moved R66 349.9 mm to (340.2, 121.9), turned to 270 degrees
- moved D65 348.6 mm to (392.6, 115.5), turned to 270 degrees
- moved U27 347.9 mm to (396.4, 175.2), turned to 180 degrees
- moved U29 339.2 mm to (413.6, 168.2), turned to 180 degrees
- moved R268 319.7 mm to (372.9, 121.9), turned to 270 degrees
- moved R68 319.1 mm to (346.7, 121.9), turned to 270 degrees
- moved U26 316.2 mm to (369.9, 175.5), turned to 180 degrees
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Connections:
- D122 pad 1: Net-(D122-Pad1) -> GND
- D123 pad 1: Net-(D123-Pad1) -> GND
- D124 pad 1: Net-(D124-Pad1) -> GND
- D125 pad 1: Net-(D125-Pad1) -> GND
- D126 pad 1: Net-(D126-Pad1) -> GND
- D127 pad 1: Net-(D127-Pad1) -> GND
- D128 pad 1: Net-(D128-Pad1) -> GND
- D129 pad 1: Net-(D129-Pad1) -> GND
- D178 pad 1: Net-(D178-Pad1) -> GND
- D179 pad 1: Net-(D178-Pad1) -> GND
- D180 pad 1: Net-(D178-Pad1) -> GND
- D181 pad 1: Net-(D178-Pad1) -> GND
- D183 pad 1: Net-(D178-Pad1) -> GND
- D185 pad 1: Net-(D178-Pad1) -> GND
- D187 pad 1: Net-(D178-Pad1) -> GND
- D189 pad 1: Net-(D178-Pad1) -> GND
- U36 pad 6: /MEM12 -> GND
- U36 pad 7: /MEM13 -> GND
- U36 pad 8: /MEM14 -> GND
- U36 pad 9: /MEM15 -> GND
Routing:
- net +5V: track 753.1 -> 1590.7 mm, vias 11 -> 26
- net /RAMOBUS0: track 7.67 -> 231.8 mm, vias 0 -> 2
- net /MEMADDR0: track 355.0 -> 576.9 mm, vias 8 -> 12
- net CLK: track 193.1 -> 414.7 mm, vias 5 -> 8
- net /MEMADDR1: track 343.9 -> 557.7 mm, vias 12 -> 16
- net /RAMOBUS1: track 21.2 -> 233.4 mm, vias 4 -> 6
- net /MEMADDR2: track 330.0 -> 535.9 mm, vias 12 -> 16
- net /MEM11: track 0.00 -> 205.5 mm, vias 0 -> 2
- net /RAMOBUS2: track 22.9 -> 226.3 mm, vias 2 -> 4
- net /MEMADDR3: track 314.6 -> 512.0 mm, vias 12 -> 16
- net /MEM10: track 0.00 -> 197.2 mm
- net /RAMOBUS3: track 18.9 -> 212.1 mm, vias 2 -> 4
- net /RAMOBUS5: track 42.7 -> 235.4 mm, vias 4 -> 6
- net /MEMADDR4: track 275.5 -> 465.2 mm, vias 12 -> 16
- net /RAMOBUS4: track 29.2 -> 217.8 mm, vias 0 -> 2
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- added copper zone on B.Cu, net +5V
- added copper zone on B.Cu, net GND
Other:
- board outline added: 400 x 300 mm
- board text added: "RANDOM ACCESS MEMORY"

Commit message: tmp push
Parts:
- moved R30 568.5 mm to (144.0, 94.8), turned to 270 degrees
- moved D36 550.6 mm to (104.6, 88.4), turned to 270 degrees
- moved D34 538.4 mm to (117.8, 88.4), turned to 270 degrees
- moved R35 527.5 mm to (111.2, 94.8), turned to 270 degrees
- moved R25 526.0 mm to (176.7, 94.8), turned to 270 degrees
- moved R26 521.7 mm to (170.2, 94.8), turned to 270 degrees
- moved U21 519.3 mm to (119.7, 101.1), turned to 270 degrees
- moved D35 489.0 mm to (111.2, 88.4), turned to 270 degrees
- moved U20 486.8 mm to (148.3, 101.0), turned to 270 degrees
- moved R36 476.9 mm to (104.6, 94.8), turned to 270 degrees
- moved D31 469.5 mm to (137.4, 88.4), turned to 270 degrees
- moved R28 464.2 mm to (157.1, 94.8), turned to 270 degrees
- moved R34 459.9 mm to (117.7, 94.8), turned to 270 degrees
- moved U19 457.7 mm to (176.2, 101.1), turned to 270 degrees
- moved R32 457.0 mm to (130.9, 94.8), turned to 270 degrees
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Routing:
- net +5V: track 1590.7 -> 1828.9 mm, vias 26 -> 27
- net /ADDR10: track 265.1 -> 495.8 mm
- net /ADDR4: track 305.5 -> 476.2 mm
- net /ADDR5: track 299.7 -> 469.6 mm
- net /ADDR6: track 295.5 -> 462.7 mm
- net /ADDR7: track 290.5 -> 456.5 mm
- net /ADDR0: track 336.3 -> 499.7 mm
- net /ADDR1: track 332.1 -> 494.1 mm
- net /ADDR2: track 327.1 -> 487.7 mm
- net /ADDR3: track 327.1 -> 486.4 mm
- net /ADDR8: track 275.3 -> 418.8 mm
- net /ADDR9: track 269.9 -> 412.6 mm
- net /ADDR11: track 260.7 -> 400.1 mm
- net CLK: track 414.7 -> 532.3 mm, vias 8 -> 10
- net /BJAB4: track 0.00 -> 110.1 mm
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- added copper zone on F.Cu, net CLK
Other:
- board text added: "2x 28c64"
- board text added: "2x ??????"
- board text added: "JUMP REGISTER"
- board text added: "MEMORY OUTPUT CONTROL"
- board text added: "READ ONLY MEMORY"
- board text removed: "READ ONLY MEMORY 4x 2Kx16"

Commit message: started with reg a & b
Parts:
- moved U5 526.1 mm to (152.1, 216.7), turned to 270 degrees
- moved U17 507.6 mm to (152.1, 179.5), turned to 270 degrees
- moved U16 465.9 mm to (177.0, 179.3), turned to 270 degrees
- moved C2 461.6 mm to (472.8, 284.3)
- moved C66 455.3 mm to (458.5, 284.3)
- moved C67 451.1 mm to (491.8, 282.2)
- moved D19 447.3 mm to (470.3, 279.1)
- moved D109 445.7 mm to (522.8, 277.5)
- moved D114 445.0 mm to (540.9, 263.2)
- moved C42 444.5 mm to (537.7, 276.0)
- moved R20 444.5 mm to (542.5, 276.0)
- moved C4 443.7 mm to (468.0, 284.3)
- moved D91 437.5 mm to (525.9, 262.4)
- moved R22 425.5 mm to (560.5, 258.1)
- moved U57 424.6 mm to (489.0, 251.6)
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Routing:
- net CLK: track 532.3 -> 695.4 mm, vias 10 -> 12
- net /D5: track 24.6 -> 168.0 mm
- net /D6: track 24.6 -> 168.0 mm
- net /D4: track 24.6 -> 168.0 mm
- net /D7: track 24.6 -> 167.8 mm
- net +5V: track 1828.9 -> 1964.9 mm, vias 27 -> 29
- net /D0: track 24.6 -> 153.4 mm
- net /D1: track 24.7 -> 153.3 mm
- net /D3: track 24.7 -> 153.2 mm
- net /D2: track 24.7 -> 153.1 mm
- net /RA7: track 0.00 -> 44.5 mm
- net /RA6: track 0.00 -> 41.9 mm
- net /REGB6: track 0.00 -> 41.3 mm
- net /RA5: track 0.00 -> 39.2 mm
- net /REGB5: track 0.00 -> 38.9 mm
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Other:
- board text added: "ALU"
- board text added: "DATA BUS"
- board text added: "REGISTER A"
- board text added: "REGISTER B"
