File: Hardware/CLUSTERFCK/MAR/MAR/MAR.sch (KiCad schematic (older format))
At the start: 30 parts

Commit message: 0027 | 0,2h | updated CLUSTERFCK/MAR
Parts:
- added C? (x2): C, symbol Device:C
- added U? (x2): 74LS245, symbol 74xx:74LS245
Connections:
- net +5V: now also C?.1, C?.1, U?.1 (A->B), U?.1 (A->B), U?.20 (VCC), U?.20 (VCC), U?.5 (A3)
- net ADDR0: now also U?.18 (B0)
- net ADDR1: now also U?.17 (B1)
- net ADDR10: now also U?.16 (B2)
- net ADDR11: now also U?.15 (B3)
- net ADDR2: now also U?.16 (B2)
- net ADDR3: now also U?.15 (B3)
- net ADDR4: now also U?.14 (B4)
- net ADDR5: now also U?.13 (B5)
- net ADDR6: now also U?.12 (B6)
- net ADDR7: now also U?.11 (B7)
- net ADDR8: now also U?.18 (B0)
- net ADDR9: now also U?.17 (B1)
- net GND: now also C?.2, C?.2, U?.10 (GND), U?.10 (GND), U?.6 (A4), U?.7 (A5), U?.8 (A6), U?.9 (A7)
- new net: U?.2 (A0), U?.2 (A0), U?.3 (A1), U?.3 (A1), U?.4 (A2), U?.4 (A2), U?.5 (A3), U?.6 (A4), U?.7 (A5), U?.8 (A6), U?.9 (A7)
- new net ~CONST: U?.19 (CE), U?.19 (CE)
- no-connect marks 0 -> 4
