File: Hardware/CLUSTERFCK/RAM/RAM/RAM.sch (KiCad schematic (older format))
At the start: 24 parts

Commit message: 0011 | 1,5 | modified CLUSTERFCK/RAM
Parts:
- added C? (x6): C, symbol Device:C
- added J?: Conn_02x04_Counter_Clockwise, symbol Connector_Generic:Conn_02x04_Counter_Clockwise
- added R? (x4): R, symbol Device:R
- added U? (x4): 74HCT164, symbol 74xx:74HCT164
- added U? (x2): 74LS245, symbol 74xx:74LS245
Connections:
- net +5V: now also C?.1, C?.1, C?.1, C?.1, C?.1, C?.1, J?.5 (Pin_5), R?.2, U?.1 (A->B), U?.1 (A->B), U?.14 (VCC), U?.14 (VCC), U?.14 (VCC), U?.14 (VCC), U?.20 (VCC), U?.20 (VCC), U?.9 (~MR), U?.9 (~MR), U?.9 (~MR), U?.9 (~MR)
- net GND: now also C?.2, C?.2, C?.2, C?.2, C?.2, C?.2, J?.4 (Pin_4), R?.2, R?.2, R?.2, U?.10 (GND), U?.10 (GND), U?.5 (A3), U?.6 (A4), U?.7 (A5), U?.7 (GND), U?.7 (GND), U?.7 (GND), U?.7 (GND), U?.8 (A6), U?.9 (A7); no longer U?.10, U?.12, U?.13, U?.4, U?.5, U?.9
- net MEMADDR0: now also U?.2 (A0); no longer U?.8 (A0), U?.8 (A0)
- net MEMADDR1: now also U?.3 (A1); no longer U?.7 (A1), U?.7 (A1)
- net MEMADDR10: now also U?.4 (A2); no longer U?.19 (A10), U?.19 (A10)
- net MEMADDR2: now also U?.4 (A2); no longer U?.6 (A2), U?.6 (A2)
- net MEMADDR3: now also U?.5 (A3); no longer U?.5 (A3), U?.5 (A3)
- net MEMADDR4: now also U?.6 (A4); no longer U?.4 (A4), U?.4 (A4)
- net MEMADDR5: now also U?.7 (A5); no longer U?.3 (A5), U?.3 (A5)
- net MEMADDR6: now also U?.8 (A6); no longer U?.2 (A6), U?.2 (A6)
- net MEMADDR7: now also U?.9 (A7); no longer U?.1 (A7), U?.1 (A7)
- net MEMADDR8: now also U?.2 (A0); no longer U?.23 (A8), U?.23 (A8)
- net MEMADDR9: now also U?.3 (A1); no longer U?.22 (A9), U?.22 (A9)
- net RAMOBUS0: now also U?.3 (Q0)
- net RAMOBUS1: now also U?.4 (Q1)
- net RAMOBUS10: now also U?.5 (Q2)
- net RAMOBUS11: now also U?.6 (Q3)
- net RAMOBUS12: now also U?.10 (Q4)
- net RAMOBUS13: now also U?.11 (Q5)
- net RAMOBUS14: now also U?.12 (Q6)
- net RAMOBUS15: now also U?.13 (Q7)
- net RAMOBUS2: now also U?.5 (Q2)
- net RAMOBUS3: now also U?.6 (Q3)
- net RAMOBUS4: now also U?.10 (Q4)
- net RAMOBUS5: now also U?.11 (Q5)
- net RAMOBUS6: now also U?.12 (Q6)
- net RAMOBUS7: now also U?.1 (DSA), U?.13 (Q7), U?.2 (DSB)
- net RAMOBUS8: now also U?.3 (Q0)
- net RAMOBUS9: now also U?.4 (Q1)
- net at U?.6: now also U?.9
- net at U?.8: now also U?.21 (~W), U?.21 (~W)
- net at U?.11: now also U?.10
- net ~RAMAI: no longer names the net of U?.11, U?.5
- net ~RAMDI: no longer names the net of U?.4, U?.8
- new net: U?.12, U?.13, U?.3
- new net: J?.7 (Pin_7), U?.1 (DSA), U?.2 (DSB)
- new net: J?.2 (Pin_2), U?.1 (DSA), U?.2 (DSB)
- new net: U?.10 (Q4), U?.14 (B4), U?.4 (A4), U?.4 (A4)
- new net: U?.11 (Q5), U?.13 (B5), U?.3 (A5), U?.3 (A5)
- new net: U?.12 (B6), U?.12 (Q6), U?.2 (A6), U?.2 (A6)
- new net: U?.1 (A7), U?.1 (A7), U?.1 (DSA), U?.11 (B7), U?.13 (Q7), U?.2 (DSB)
- new net: U?.18 (B0), U?.3 (Q0), U?.8 (A0), U?.8 (A0)
- new net: U?.17 (B1), U?.4 (Q1), U?.7 (A1), U?.7 (A1)
- new net: U?.16 (B2), U?.5 (Q2), U?.6 (A2), U?.6 (A2)
- new net: U?.15 (B3), U?.5 (A3), U?.5 (A3), U?.6 (Q3)
- new net: U?.18 (B0), U?.23 (A8), U?.23 (A8), U?.3 (Q0)
- new net: U?.17 (B1), U?.22 (A9), U?.22 (A9), U?.4 (Q1)
- new net: U?.16 (B2), U?.19 (A10), U?.19 (A10), U?.5 (Q2)
- new net BLOCK: J?.6 (Pin_6), R?.1, U?.19 (CE), U?.19 (CE)
- new net CLK_A: J?.1 (Pin_1), R?.1, U?.8 (CP), U?.8 (CP)
- new net CLK_D: J?.8 (Pin_8), R?.1, U?.8 (CP), U?.8 (CP)
- new net READ: J?.3 (Pin_3), R?.1, U?.4, U?.5
- no-connect marks 8 -> 14
Other:
- moved on the sheet: C?, U?, U?A, U?B, U?C, U?D, U?E

Commit message: 0025 | 0,3h | mirrored stackpointer to LED-array
Parts:
- added C? (x3): C, symbol Device:C
- added D? (x12): LED, symbol Device:LED
- added R? (x12): R, symbol Device:R
- added U? (x2): 74HCT574, symbol 74xx:74HCT574
- added U? (x5): 74LS00, symbol 74xx:74LS00
Connections:
- net +5V: now also C?.1, C?.1, C?.1, U?.1 (OE), U?.1 (OE), U?.14 (VCC), U?.20 (VCC), U?.20 (VCC)
- net ADDR0: now also U?.2 (D0)
- net ADDR1: now also U?.3 (D1)
- net ADDR10: now also U?.4 (D2)
- net ADDR11: now also U?.5 (D3)
- net ADDR2: now also U?.4 (D2)
- net ADDR3: now also U?.5 (D3)
- net ADDR4: now also U?.6 (D4)
- net ADDR5: now also U?.7 (D5)
- net ADDR6: now also U?.8 (D6)
- net ADDR7: now also U?.9 (D7)
- net ADDR8: now also U?.2 (D0)
- net ADDR9: now also U?.3 (D1)
- net CLK: now also U?.1
- net GND: now also C?.2, C?.2, C?.2, D?.1 (K), D?.1 (K), D?.1 (K), D?.1 (K), D?.1 (K), D?.1 (K), D?.1 (K), D?.1 (K), D?.1 (K), D?.1 (K), D?.1 (K), D?.1 (K), U?.10, U?.10 (GND), U?.10 (GND), U?.12, U?.13, U?.6 (D4), U?.7 (D5), U?.7 (GND), U?.8 (D6), U?.9, U?.9 (D7)
- new net: U?.11 (Cp), U?.11 (Cp), U?.6
- new net: R?.2, U?.12 (Q7)
- new net: R?.2, U?.13 (Q6)
- new net: R?.2, U?.14 (Q5)
- new net: R?.2, U?.15 (Q4)
- new net: R?.2, U?.16 (Q3) (x2)
- new net: R?.2, U?.17 (Q2) (x2)
- new net: R?.2, U?.18 (Q1) (x2)
- new net: R?.2, U?.19 (Q0) (x2)
- new net: D?.2 (A), R?.1 (x12)
- new net: U?.3, U?.4, U?.5
- new net CONST: U?.2
- no-connect marks 14 -> 20
Other:
- note added: "ACHTUNG!\nEIGENTLICH 74FCT2574T\n=> gleiches pinout"
- moved on the sheet: C?, J?, R?, U?, U?A, U?B, U?C, U?D, U?E

Commit message: 0030 | 4,5h | Review GFX
Parts:
- removed C? (x3): C, symbol Device:C
- removed D? (x12): LED, symbol Device:LED
- removed R? (x12): R, symbol Device:R
- removed U? (x2): 74HCT574, symbol 74xx:74HCT574
- removed U? (x5): 74LS00, symbol 74xx:74LS00
- added C86: C, Capacitor_SMD:C_0805_2012Metric_Pad1.15x1.40mm_HandSolder, symbol Device:C
- added U29: 74LS00, Package_DIP:DIP-14_W7.62mm_Socket_LongPads, symbol 74xx:74LS00
- U? (x2): symbol custom:M84Z02 -> RAM-rescue:M84Z02-custom
Connections:
- net +5V: now also C86.1, U29.14 (VCC)
- net GND: now also C86.2, U29.7 (GND)
- no-connect marks 20 -> 23
Other:
- note added: "excess NAND gates (RAM)\n"
- note removed: "ACHTUNG!\nEIGENTLICH 74FCT2574T\n=> gleiches pinout"
- moved on the sheet: C?, J?, R?, U?, U?A, U?B, U?C, U?D, U?E
