File: Hardware/CLUSTERFCK/RAM/RAM/RAM.kicad_pcb (KiCad board)
At the start: 4 copper layers, 142 x 62 mm, 44 parts, among them J1 Conn_02x10_Counter_Clockwise, J2 Conn_02x06_Counter_Clockwise, J3 Conn_02x08_Counter_Clockwise, J5 Conn_02x06_Counter_Clockwise, J6 Conn_02x08_Counter_Clockwise, J7 Conn_02x04_Odd_Even, J8 Conn_02x06_Odd_Even, U1 74LS245, U10 74HCT164, U11 74LS157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

Commit message: 0072 | 3h | make silkscreen prettier
Changed lines of the file:
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@@
     (property "Schaltplanname" "")
     (attr smd)
-    (fp_text reference "C12" (at -0.52 1.6) (layer "F.SilkS")
+    (fp_text reference "C12" (at -0.78 1.7) (layer "F.SilkS")
       (effects (font (size 1 1) (thickness 0.15)))
     )
@@
     (tags "mounting hole 4.3mm no annular m4")
     (attr exclude_from_pos_files exclude_from_bom)
-    (fp_text reference "REF**" (at 0.15 -2.96) (layer "F.SilkS")
+    (fp_text reference "REF**" (at -0.105 -3.67) (layer "F.SilkS")
       (effects (font (size 1 1) (thickness 0.15)))
     )
@@
     (property "Schaltplanname" "")
     (attr smd)
-    (fp_text reference "C13" (at -0.56 1.62) (layer "F.SilkS")
+    (fp_text reference "C13" (at -1.005 1.65) (layer "F.SilkS")
       (effects (font (size 1 1) (thickness 0.15)))
     )
@@
     (property "Schaltplanname" "")
     (attr smd)
-    (fp_text reference "C10" (at -0.49 1.63) (layer "F.SilkS")
+    (fp_text reference "C10" (at -0.775 1.6) (layer "F.SilkS")
       (effects (font (size 1 1) (thickness 0.15)))
     )
@@
     (property "Schaltplanname" "")
     (attr smd)
-    (fp_text reference "C14" (at 0 -1.65 90) (layer "F.SilkS")
-      (effects (font (size 1 1) (thickness 0.15)))
-    )
+    (fp_text reference "C14" (at 0.075 1.7 90) (layer "F.SilkS")
+      (effects (font (size 1 1) (thickness 0.15)))
+    )
