File: Hardware/CLUSTERFCK/MARMEM/MARMEM/MARMEM.kicad_pcb (KiCad board)
At the start: 2 copper layers, 140.1 x 92.7 mm, 84 parts, among them J1 Conn_02x20_Counter_Clockwise, J2 Conn_02x20_Counter_Clockwise, J3 Conn_02x08_Counter_Clockwise, J4 Conn_02x08_Counter_Clockwise, U1 74LS245, U10 74LS245, U11 74LS245, U12 74LS245, U2 74LS245, U3 74LS173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

Commit message: unstable switching device push
Routing:
- net GND: track 212.9 -> 199.3 mm, vias 54 -> 60
- net MEMADDR7: track 47.7 -> 43.9 mm
- net +5V: track 544.9 -> 546.9 mm, vias 23 -> 18
- net MEM2: track 92.4 -> 91.9 mm

Commit message: 0034 | 1h | review of MARMEM Module
Parts:
- moved J2 2.34 mm to (219.9, 140.2)
- moved J1 0.38 mm to (93.1, 91.4)
Routing:
- net +5V: track 546.9 -> 516.3 mm, vias 18 -> 19
- net CLK: track 267.0 -> 272.1 mm, vias 6 -> 8
- net GND: track 199.3 -> 196.0 mm, vias 60 -> 196
- net ~MEMAO: track 180.6 -> 181.9 mm
- net DATA6: track 45.9 -> 44.6 mm
- net DATA5: track 50.7 -> 49.5 mm
- net DATA4: track 49.5 -> 48.2 mm
- net DATA3: track 54.3 -> 53.1 mm
- net DATA2: track 53.1 -> 51.9 mm
- net DATA1: track 58.0 -> 56.8 mm
- net DATA7: track 47.0 -> 45.8 mm
- net DATA0: track 56.7 -> 55.8 mm
- net ADDR1: track 121.8 -> 122.6 mm
- net MEMADDR11: track 129.1 -> 129.8 mm
- net ADDR9: track 127.9 -> 128.4 mm
Other:
- board size 140.1 x 92.7 mm -> 142 x 93 mm
