File: Hardware/CLUSTERFCK/MARMEM/MARMEM/MARMEM.kicad_pcb (KiCad board)
At the start: 2 copper layers, 142 x 93 mm, 84 parts, among them J1 Conn_02x20_Counter_Clockwise, J2 Conn_02x20_Counter_Clockwise, J3 Conn_02x08_Counter_Clockwise, J4 Conn_02x08_Counter_Clockwise, U1 74LS245, U10 74LS245, U11 74LS245, U12 74LS245, U2 74LS245, U3 74LS173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

Commit message: 0035 | 1,5h | Correction MARMEM
Parts:
- added J5: Conn_02x06_Counter_Clockwise, Connector_PinHeader_2.54mm:PinHeader_2x06_P2.54mm_Horizontal, F.Cu at (133.3, 72.4)
- added J6: Conn_02x06_Counter_Clockwise, Connector_PinHeader_2.54mm:PinHeader_2x06_P2.54mm_Horizontal, F.Cu at (147.3, 157.5)
Routing:
- net MEMADDR4: track 61.1 -> 320.0 mm, vias 0 -> 4
- net MEMADDR5: track 55.4 -> 304.5 mm, vias 0 -> 4
- net MEMADDR0: track 74.5 -> 291.8 mm, vias 0 -> 4
- net MEMADDR3: track 57.5 -> 266.3 mm, vias 0 -> 3
- net MEMADDR1: track 68.8 -> 273.9 mm, vias 0 -> 1
- net MEMADDR2: track 63.1 -> 257.9 mm, vias 0 -> 3
- net MEMADDR7: track 43.9 -> 237.8 mm, vias 0 -> 3
- net MEMADDR6: track 49.7 -> 240.3 mm, vias 0 -> 3
- net MEMADDR9: track 53.3 -> 236.1 mm, vias 0 -> 2
- net MEMADDR11: track 129.8 -> 311.6 mm, vias 12 -> 14
- net MEMADDR10: track 53.7 -> 231.5 mm, vias 0 -> 2
- net MEMADDR8: track 54.1 -> 228.3 mm, vias 0 -> 3
- added copper zone on B.Cu, net MEMADDR0
- added copper zone on F.Cu, net MEMADDR0
Other:
- board size 142 x 93 mm -> 142 x 100.2 mm

Commit message: 0038 | 0,5h | review marmem
Routing:
- net CLK: track 272.1 -> 247.5 mm
- net MEMADDR5: track 304.5 -> 303.2 mm
- net ~MC: track 118.4 -> 117.6 mm
- net MEMADDR3: track 266.3 -> 265.6 mm
- net GND: vias 196 -> 256
Other:
- board text added: "Address"
- board text added: "Data"
- board text added: "Memory Address Register and Memory selection"

Commit message: quick fix MARMEM
Other:
- board text added: "Memory Address Register and MEMory space control"
- board text removed: "Memory Address Register and Memory selection"
Changed lines of the file:
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@@
       (dielectric_constraints no)
     )
-    (last_trace_width 0.2)
+    (last_trace_width 0.25)
     (user_trace_width 0.2)
     (user_trace_width 0.5)
@@
     (effects (font (size 1.5 1.5) (thickness 0.3)))
   )
-  (gr_text "Memory Address Register \nand Memory selection" (at 102.4 68.68) (layer "F.SilkS")
+  (gr_text "Memory Address Register \nand MEMory space control" (at 102.4 68.68) (layer "F.SilkS")
     (effects (font (size 1.5 1.5) (thickness 0.3)))
   )

Commit message: 0052 | 4h | MARMEM update
Connections:
- J1 pad 24: Net-(J1-Pad24) -> (no net)
- J1 pad 25: Net-(J1-Pad25) -> (no net)
- J1 pad 26: Net-(J1-Pad26) -> (no net)
- J1 pad 27: Net-(J1-Pad27) -> (no net)
- J1 pad 28: Net-(J1-Pad28) -> (no net)
- J1 pad 29: Net-(J1-Pad29) -> (no net)
- J1 pad 30: Net-(J1-Pad30) -> (no net)
- J1 pad 31: Net-(J1-Pad31) -> (no net)
- J1 pad 32: Net-(J1-Pad32) -> (no net)
- J1 pad 33: Net-(J1-Pad33) -> (no net)
- J1 pad 34: Net-(J1-Pad34) -> (no net)
- J1 pad 35: Net-(J1-Pad35) -> (no net)
- J1 pad 36: Net-(J1-Pad36) -> (no net)
- J1 pad 37: Net-(J1-Pad37) -> (no net)
- J1 pad 38: Net-(J1-Pad38) -> (no net)
- J2 pad 12: Net-(J2-Pad12) -> MEM0
- J2 pad 13: Net-(J2-Pad13) -> MEM1
- J2 pad 14: Net-(J2-Pad14) -> MEM2
- J2 pad 15: Net-(J2-Pad15) -> MEM3
- J2 pad 16: Net-(J2-Pad16) -> MEM4
- J2 pad 17: Net-(J2-Pad17) -> MEM5
- J2 pad 18: Net-(J2-Pad18) -> MEM6
- J2 pad 23: Net-(J2-Pad23) -> MEM7
- J2 pad 24: Net-(J2-Pad24) -> MEM8
- J2 pad 25: Net-(J2-Pad25) -> MEM9
- J2 pad 26: Net-(J2-Pad26) -> MEM10
- J2 pad 27: Net-(J2-Pad27) -> MEM11
- J2 pad 28: Net-(J2-Pad28) -> MEM12
- J2 pad 29: Net-(J2-Pad29) -> MEM13
- J2 pad 30: Net-(J2-Pad30) -> MEM14
- J2 pad 31: Net-(J2-Pad31) -> MEM15
- J2 pad 32: Net-(J2-Pad32) -> (no net)
- J2 pad 33: Net-(J2-Pad33) -> (no net)
- J2 pad 34: Net-(J2-Pad34) -> (no net)
- J2 pad 35: Net-(J2-Pad35) -> (no net)
- J2 pad 36: Net-(J2-Pad36) -> (no net)
- J2 pad 37: Net-(J2-Pad37) -> (no net)
- J2 pad 38: Net-(J2-Pad38) -> (no net)
- U1 pad 11: Net-(U1-Pad11) -> (no net)
- U1 pad 12: Net-(U1-Pad12) -> (no net)
- U1 pad 13: Net-(U1-Pad13) -> (no net)
- U1 pad 14: Net-(U1-Pad14) -> (no net)
- U12 pad 11: Net-(U12-Pad11) -> (no net)
- U12 pad 12: Net-(U12-Pad12) -> (no net)
- U12 pad 13: Net-(U12-Pad13) -> (no net)
- U12 pad 14: Net-(U12-Pad14) -> (no net)
Routing:
- net MEM15: track 63.8 -> 255.1 mm
- net MEM14: track 54.2 -> 229.0 mm, vias 2 -> 5
- net MEM12: track 35.3 -> 205.6 mm, vias 2 -> 7
- net MEM13: track 41.3 -> 210.3 mm, vias 2 -> 7
- net MEM11: track 65.0 -> 223.8 mm, vias 2 -> 7
- net MEM10: track 50.4 -> 171.5 mm, vias 2 -> 7
- net MEM8: track 65.5 -> 125.8 mm, vias 5 -> 8
- net MEM9: track 52.0 -> 111.9 mm, vias 4 -> 7
- net MEM7: track 114.1 -> 172.3 mm, vias 5 -> 9
- net MEM6: track 107.9 -> 139.0 mm, vias 4 -> 7
- net MEM2: track 91.9 -> 121.0 mm, vias 4 -> 7
- net MEM4: track 132.9 -> 161.6 mm, vias 4 -> 7
- net MEM3: track 95.6 -> 121.8 mm, vias 4 -> 7
- net MEM5: track 115.5 -> 141.3 mm, vias 5 -> 8
- net MEM0: track 116.0 -> 139.5 mm
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- removed copper zone on B.Cu, net MEMADDR0
- removed copper zone on B.Cu, net RAMOBUS0

Commit message: 0050 | 5h | Ram module
Other:
- net class Default removed

Commit message: 0066 | 6h | made holes in pcbs
Parts:
- added REF**: MountingHole_4.3mm_M4, MountingHole:MountingHole_4.3mm_M4, F.Cu at (90.8, 159.9)
- added REF**: MountingHole_4.3mm_M4, MountingHole:MountingHole_4.3mm_M4, F.Cu at (222.3, 160.1)
- added REF**: MountingHole_4.3mm_M4, MountingHole:MountingHole_4.3mm_M4, F.Cu at (222.5, 70.1)
- added REF**: MountingHole_4.3mm_M4, MountingHole:MountingHole_4.3mm_M4, F.Cu at (90.9, 70.2)
