File: Hardware/CLUSTERFCK/MARMEM/MARMEM/MARMEM.kicad_sch (KiCad schematic)
At the start: 86 parts, among them J1 Conn_02x20_Counter_Clockwise, J2 Conn_02x20_Counter_Clockwise, J3 Conn_02x08_Counter_Clockwise, J4 Conn_02x08_Counter_Clockwise, J5 Conn_02x06_Counter_Clockwise, J6 Conn_02x06_Counter_Clockwise, U1 74LS245, U10 74LS245, U11 74LS245, U12 74LS245, U2 74LS245, U3 74LS173, U4 74LS173, U5 74LS173, U6 74LS157, U7 74LS157, U8 74LS157, U9 74LS157

Commit message: 0049 | 1h | review ROM
Parts:
- removed C1, C10, C11, C12, C2, C3, C4, C5, C6, C7, C8, C9: C, Capacitor_SMD:C_0805_2012Metric_Pad1.15x1.40mm_HandSolder, symbol Device:C
- removed D1, D10, D11, D12, D2, D3, D4, D5, D6, D69, D7, D70, D71, D72, D73, D74, D75, D76, D77, D78, D79, D8, D80, D81, D82, D83, D84, D9: LED, LED_THT:LED_D5.0mm, symbol Device:LED
- removed J1, J2: Conn_02x20_Counter_Clockwise, Connector_PinSocket_2.54mm:PinSocket_2x20_P2.54mm_Horizontal, symbol Connector_Generic:Conn_02x20_Counter_Clockwise
- removed J3, J4: Conn_02x08_Counter_Clockwise, Connector_PinHeader_2.54mm:PinHeader_2x08_P2.54mm_Horizontal, symbol Connector_Generic:Conn_02x08_Counter_Clockwise
- removed J5, J6: Conn_02x06_Counter_Clockwise, Connector_PinHeader_2.54mm:PinHeader_2x06_P2.54mm_Horizontal, symbol Connector_Generic:Conn_02x06_Counter_Clockwise
- removed R1, R10, R11, R12, R2, R3, R4, R5, R6, R7, R70, R71, R72, R73, R74, R75, R76, R77, R78, R79, R8, R80, R81, R82, R83, R84, R85, R9: R, Resistor_SMD:R_0805_2012Metric_Pad1.15x1.40mm_HandSolder, symbol Device:R
- removed U1, U10, U11, U12, U2: 74LS245, Package_SO:SOIC-20W_7.5x12.8mm_P1.27mm, symbol 74xx:74LS245
- removed U3, U4, U5: 74LS173, Package_SO:SOP-16_3.9x9.9mm_P1.27mm, symbol 74xx:74LS173
- removed U6, U7, U8, U9: 74LS157, Package_SO:SOP-16_3.9x9.9mm_P1.27mm, symbol 74xx:74LS157
Connections:
- no-connect marks 46 -> 0
Other:
- note removed: "To ADDR-Bus"
- note removed: "To DATA-Bus"
- company: Wilhelm-Maybach-Schule Heilbronn -> (none)
- title: MARMEM -> (none)

Commit message: marmem wieder in git
Parts:
- added C1, C10, C11, C12, C2, C3, C4, C5, C6, C7, C8, C9: C, Capacitor_SMD:C_0805_2012Metric_Pad1.15x1.40mm_HandSolder, symbol Device:C
- added D1, D10, D11, D12, D2, D3, D4, D5, D6, D69, D7, D70, D71, D72, D73, D74, D75, D76, D77, D78, D79, D8, D80, D81, D82, D83, D84, D9: LED, LED_THT:LED_D5.0mm, symbol Device:LED
- added J1, J2: Conn_02x20_Counter_Clockwise, Connector_PinSocket_2.54mm:PinSocket_2x20_P2.54mm_Horizontal, symbol Connector_Generic:Conn_02x20_Counter_Clockwise
- added J3, J4: Conn_02x08_Counter_Clockwise, Connector_PinHeader_2.54mm:PinHeader_2x08_P2.54mm_Horizontal, symbol Connector_Generic:Conn_02x08_Counter_Clockwise
- added J5, J6: Conn_02x06_Counter_Clockwise, Connector_PinHeader_2.54mm:PinHeader_2x06_P2.54mm_Horizontal, symbol Connector_Generic:Conn_02x06_Counter_Clockwise
- added R1, R10, R11, R12, R2, R3, R4, R5, R6, R7, R70, R71, R72, R73, R74, R75, R76, R77, R78, R79, R8, R80, R81, R82, R83, R84, R85, R9: R, Resistor_SMD:R_0805_2012Metric_Pad1.15x1.40mm_HandSolder, symbol Device:R
- added U1, U10, U11, U12, U2: 74LS245, Package_SO:SOIC-20W_7.5x12.8mm_P1.27mm, symbol 74xx:74LS245
- added U3, U4, U5: 74LS173, Package_SO:SOP-16_3.9x9.9mm_P1.27mm, symbol 74xx:74LS173
- added U6, U7, U8, U9: 74LS157, Package_SO:SOP-16_3.9x9.9mm_P1.27mm, symbol 74xx:74LS157
Connections:
- new net: D1.2 (A), R1.1
- new net: D2.2 (A), R2.1
- new net: D3.2 (A), R3.1
- new net: D4.2 (A), R4.1
- new net: D5.2 (A), R5.1
- new net: D6.2 (A), R6.1
- new net: D7.2 (A), R7.1
- new net: D8.2 (A), R8.1
- new net: D9.2 (A), R9.1
- new net: D10.2 (A), R10.1
- new net: D11.2 (A), R11.1
- new net: D12.2 (A), R12.1
- new net: D80.2 (A), R81.1
- new net: D79.2 (A), R80.1
- new net: D78.2 (A), R79.1
- new net: D77.2 (A), R78.1
- new net: D76.2 (A), R77.1
- new net: D75.2 (A), R76.1
- new net: D74.2 (A), R75.1
- new net: D73.2 (A), R74.1
- new net: D72.2 (A), R73.1
- new net: D71.2 (A), R72.1
- new net: D70.2 (A), R71.1
- new net: D69.2 (A), R70.1
- new net: D84.2 (A), R85.1
- new net: D83.2 (A), R84.1
- new net: D82.2 (A), R83.1
- new net: D81.2 (A), R82.1
- new net +5V: C1.1, C10.1, C11.1, C12.1, C2.1, C3.1, C4.1, C5.1, C6.1, C7.1, C8.1, C9.1, J1.21 (Pin_21), J1.22 (Pin_22), J1.39 (Pin_39), J1.40 (Pin_40), J2.21 (Pin_21), J2.22 (Pin_22), J2.39 (Pin_39), J2.40 (Pin_40), U1.1 (A->B), U1.20 (VCC), U1.5 (A3), U10.1 (A->B), U10.20 (VCC), U11.1 (A->B), U11.20 (VCC), U12.1 (A->B), U12.20 (VCC), U2.1 (A->B), U2.20 (VCC), U3.16 (VCC), U4.16 (VCC), U5.16 (VCC), U6.16 (VCC), U7.16 (VCC), U8.16 (VCC), U9.16 (VCC)
- new net ADDR0: J1.3 (Pin_3), U11.18 (B0), U2.18 (B0), U3.14 (D0)
- new net ADDR1: J1.4 (Pin_4), U11.17 (B1), U2.17 (B1), U3.13 (D1)
- new net ADDR10: J1.13 (Pin_13), U1.16 (B2), U12.16 (B2), U5.12 (D2)
- new net ADDR11: J1.14 (Pin_14), U1.15 (B3), U12.15 (B3), U5.11 (D3)
- new net ADDR2: J1.5 (Pin_5), U11.16 (B2), U2.16 (B2), U3.12 (D2)
- new net ADDR3: J1.6 (Pin_6), U11.15 (B3), U2.15 (B3), U3.11 (D3)
- new net ADDR4: J1.7 (Pin_7), U11.14 (B4), U2.14 (B4), U4.14 (D0)
- new net ADDR5: J1.8 (Pin_8), U11.13 (B5), U2.13 (B5), U4.13 (D1)
- new net ADDR6: J1.9 (Pin_9), U11.12 (B6), U2.12 (B6), U4.12 (D2)
- new net ADDR7: J1.10 (Pin_10), U11.11 (B7), U2.11 (B7), U4.11 (D3)
- new net ADDR8: J1.11 (Pin_11), U1.18 (B0), U12.18 (B0), U5.14 (D0)
- new net ADDR9: J1.12 (Pin_12), U1.17 (B1), U12.17 (B1), U5.13 (D1)
- new net CLK: J1.15 (Pin_15), J2.11 (Pin_11), U3.7 (Cp), U4.7 (Cp), U5.7 (Cp)
- new net DATA0: J2.3 (Pin_3), U10.18 (B0)
- new net DATA1: J2.4 (Pin_4), U10.17 (B1)
- new net DATA2: J2.5 (Pin_5), U10.16 (B2)
- new net DATA3: J2.6 (Pin_6), U10.15 (B3)
- new net DATA4: J2.7 (Pin_7), U10.14 (B4)
- new net DATA5: J2.8 (Pin_8), U10.13 (B5)
- new net DATA6: J2.9 (Pin_9), U10.12 (B6)
- new net DATA7: J2.10 (Pin_10), U10.11 (B7)
- new net GND: C1.2, C10.2, C11.2, C12.2, C2.2, C3.2, C4.2, C5.2, C6.2, C7.2, C8.2, C9.2, D1.1 (K), D10.1 (K), D11.1 (K), D12.1 (K), D2.1 (K), D3.1 (K), D4.1 (K), D5.1 (K), D6.1 (K), D69.1 (K), D7.1 (K), D70.1 (K), D71.1 (K), D72.1 (K), D73.1 (K), D74.1 (K), D75.1 (K), D76.1 (K), D77.1 (K), D78.1 (K), D79.1 (K), D8.1 (K), D80.1 (K), D81.1 (K), D82.1 (K), D83.1 (K), D84.1 (K), D9.1 (K), J1.1 (Pin_1), J1.19 (Pin_19), J1.2 (Pin_2), J1.20 (Pin_20), J2.1 (Pin_1), J2.19 (Pin_19), J2.2 (Pin_2), J2.20 (Pin_20), U1.10 (GND), U1.2 (A0), U1.3 (A1), U1.4 (A2), U1.6 (A4), U1.7 (A5), U1.8 (A6), U1.9 (A7), U10.10 (GND), U11.10 (GND), U12.10 (GND), U12.6 (A4), U12.7 (A5), U12.8 (A6), U12.9 (A7), U2.10 (GND), U2.2 (A0), U2.3 (A1), U2.4 (A2), U2.5 (A3), U2.6 (A4), U2.7 (A5), U2.8 (A6), U2.9 (A7), U3.1 (Oe1), U3.15 (Mr), U3.2 (Oe2), U3.8 (GND), U4.1 (Oe1), U4.15 (Mr), U4.2 (Oe2), U4.8 (GND), U5.1 (Oe1), U5.15 (Mr), U5.2 (Oe2), U5.8 (GND), U6.15 (E), U6.8 (GND), U7.15 (E), U7.8 (GND), U8.15 (E), U8.8 (GND), U9.15 (E), U9.8 (GND)
- new net MEM0: R70.2, U10.2 (A0), U11.2 (A0), U6.4 (Za)
- new net MEM1: R71.2, U10.3 (A1), U11.3 (A1), U6.7 (Zb)
- new net MEM10: R80.2, U12.4 (A2), U8.9 (Zc)
- new net MEM11: R81.2, U12.5 (A3), U8.12 (Zd)
- new net MEM12: R82.2, U9.4 (Za)
- new net MEM13: R83.2, U9.7 (Zb)
- new net MEM14: R84.2, U9.9 (Zc)
- new net MEM15: R85.2, U9.12 (Zd)
- new net MEM2: R72.2, U10.4 (A2), U11.4 (A2), U6.9 (Zc)
- new net MEM3: R73.2, U10.5 (A3), U11.5 (A3), U6.12 (Zd)
- new net MEM4: R74.2, U10.6 (A4), U11.6 (A4), U7.4 (Za)
- new net MEM5: R75.2, U10.7 (A5), U11.7 (A5), U7.7 (Zb)
- new net MEM6: R76.2, U10.8 (A6), U11.8 (A6), U7.9 (Zc)
- new net MEM7: R77.2, U10.9 (A7), U11.9 (A7), U7.12 (Zd)
- new net MEM8: R78.2, U12.2 (A0), U8.4 (Za)
- new net MEM9: R79.2, U12.3 (A1), U8.7 (Zb)
- new net MEMADDR0: J5.1 (Pin_1), J6.1 (Pin_1), R1.2, U3.3 (Q0)
- new net MEMADDR1: J5.2 (Pin_2), J6.2 (Pin_2), R2.2, U3.4 (Q1)
- new net MEMADDR10: J5.11 (Pin_11), J6.11 (Pin_11), R11.2, U5.5 (Q2)
- new net MEMADDR11: J5.12 (Pin_12), J6.12 (Pin_12), R12.2, U5.6 (Q3), U6.1 (S), U7.1 (S), U8.1 (S), U9.1 (S)
- new net MEMADDR2: J5.3 (Pin_3), J6.3 (Pin_3), R3.2, U3.5 (Q2)
- new net MEMADDR3: J5.4 (Pin_4), J6.4 (Pin_4), R4.2, U3.6 (Q3)
- new net MEMADDR4: J5.5 (Pin_5), J6.5 (Pin_5), R5.2, U4.3 (Q0)
- new net MEMADDR5: J5.6 (Pin_6), J6.6 (Pin_6), R6.2, U4.4 (Q1)
- new net MEMADDR6: J5.7 (Pin_7), J6.7 (Pin_7), R7.2, U4.5 (Q2)
- new net MEMADDR7: J5.8 (Pin_8), J6.8 (Pin_8), R8.2, U4.6 (Q3)
- new net MEMADDR8: J5.9 (Pin_9), J6.9 (Pin_9), R9.2, U5.3 (Q0)
- new net MEMADDR9: J5.10 (Pin_10), J6.10 (Pin_10), R10.2, U5.4 (Q1)
- new net RAMOBUS0: J3.1 (Pin_1), U6.2 (I0a)
- new net RAMOBUS1: J3.2 (Pin_2), U6.5 (I0b)
- new net RAMOBUS10: J3.11 (Pin_11), U8.11 (I0c)
- new net RAMOBUS11: J3.12 (Pin_12), U8.14 (I0d)
- new net RAMOBUS12: J3.13 (Pin_13), U9.2 (I0a)
- new net RAMOBUS13: J3.14 (Pin_14), U9.5 (I0b)
- new net RAMOBUS14: J3.15 (Pin_15), U9.11 (I0c)
- new net RAMOBUS15: J3.16 (Pin_16), U9.14 (I0d)
- new net RAMOBUS2: J3.3 (Pin_3), U6.11 (I0c)
- new net RAMOBUS3: J3.4 (Pin_4), U6.14 (I0d)
- new net RAMOBUS4: J3.5 (Pin_5), U7.2 (I0a)
- new net RAMOBUS5: J3.6 (Pin_6), U7.5 (I0b)
- new net RAMOBUS6: J3.7 (Pin_7), U7.11 (I0c)
- new net RAMOBUS7: J3.8 (Pin_8), U7.14 (I0d)
- new net RAMOBUS8: J3.9 (Pin_9), U8.2 (I0a)
- new net RAMOBUS9: J3.10 (Pin_10), U8.5 (I0b)
- new net ROM0: J4.1 (Pin_1), U6.3 (I1a)
- new net ROM1: J4.2 (Pin_2), U6.6 (I1b)
- new net ROM10: J4.11 (Pin_11), U8.10 (I1c)
- new net ROM11: J4.12 (Pin_12), U8.13 (I1d)
- new net ROM12: J4.13 (Pin_13), U9.3 (I1a)
- new net ROM13: J4.14 (Pin_14), U9.6 (I1b)
- new net ROM14: J4.15 (Pin_15), U9.10 (I1c)
- new net ROM15: J4.16 (Pin_16), U9.13 (I1d)
- new net ROM2: J4.3 (Pin_3), U6.10 (I1c)
- new net ROM3: J4.4 (Pin_4), U6.13 (I1d)
- new net ROM4: J4.5 (Pin_5), U7.3 (I1a)
- new net ROM5: J4.6 (Pin_6), U7.6 (I1b)
- new net ROM6: J4.7 (Pin_7), U7.10 (I1c)
- new net ROM7: J4.8 (Pin_8), U7.13 (I1d)
- new net ROM8: J4.9 (Pin_9), U8.3 (I1a)
- new net ROM9: J4.10 (Pin_10), U8.6 (I1b)
- new net ~CONST: J1.23 (Pin_23), U1.19 (CE), U2.19 (CE)
- new net ~MC: J1.18 (Pin_18), U3.10 (E2), U3.9 (E1), U4.10 (E2), U4.9 (E1), U5.10 (E2), U5.9 (E1)
- new net ~MEMAO: J1.17 (Pin_17), U11.19 (CE), U12.19 (CE)
- new net ~MEMDO: J1.16 (Pin_16), U10.19 (CE)
- no-connect marks 0 -> 46
Other:
- note added: "To ADDR-Bus"
- note added: "To DATA-Bus"
- company: (none) -> Wilhelm-Maybach-Schule Heilbronn
- title: (none) -> MARMEM
