File: Hardware/CLUSTERFCK/MARMEM/MARMEM/MARMEM.kicad_sch (KiCad schematic)
At the start: 84 parts, among them J1 Conn_02x20_Counter_Clockwise, J2 Conn_02x20_Counter_Clockwise, J3 Conn_02x08_Counter_Clockwise, J4 Conn_02x08_Counter_Clockwise, U1 74LS245, U10 74LS245, U11 74LS245, U12 74LS245, U2 74LS245, U3 74LS173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

Commit message: 0035 | 1,5h | Correction MARMEM
Parts:
- added J5, J6: Conn_02x06_Counter_Clockwise, Connector_PinHeader_2.54mm:PinHeader_2x06_P2.54mm_Horizontal, symbol Connector_Generic:Conn_02x06_Counter_Clockwise
Connections:
- net MEMADDR0: now also J5.1 (Pin_1), J6.1 (Pin_1)
- net MEMADDR1: now also J5.2 (Pin_2), J6.2 (Pin_2)
- net MEMADDR10: now also J5.11 (Pin_11), J6.11 (Pin_11)
- net MEMADDR11: now also J5.12 (Pin_12), J6.12 (Pin_12)
- net MEMADDR2: now also J5.3 (Pin_3), J6.3 (Pin_3)
- net MEMADDR3: now also J5.4 (Pin_4), J6.4 (Pin_4)
- net MEMADDR4: now also J5.5 (Pin_5), J6.5 (Pin_5)
- net MEMADDR5: now also J5.6 (Pin_6), J6.6 (Pin_6)
- net MEMADDR6: now also J5.7 (Pin_7), J6.7 (Pin_7)
- net MEMADDR7: now also J5.8 (Pin_8), J6.8 (Pin_8)
- net MEMADDR8: now also J5.9 (Pin_9), J6.9 (Pin_9)
- net MEMADDR9: now also J5.10 (Pin_10), J6.10 (Pin_10)

Commit message: 0052 | 4h | MARMEM update
Connections:
- net MEM0: now also J2.12 (Pin_12)
- net MEM1: now also J2.13 (Pin_13)
- net MEM10: now also J2.26 (Pin_26)
- net MEM11: now also J2.27 (Pin_27)
- net MEM12: now also J2.28 (Pin_28)
- net MEM13: now also J2.29 (Pin_29)
- net MEM14: now also J2.30 (Pin_30)
- net MEM15: now also J2.31 (Pin_31)
- net MEM2: now also J2.14 (Pin_14)
- net MEM3: now also J2.15 (Pin_15)
- net MEM4: now also J2.16 (Pin_16)
- net MEM5: now also J2.17 (Pin_17)
- net MEM6: now also J2.18 (Pin_18)
- net MEM7: now also J2.23 (Pin_23)
- net MEM8: now also J2.24 (Pin_24)
- net MEM9: now also J2.25 (Pin_25)
- no-connect marks 46 -> 30
Other:
- moved on the sheet: J2
