File: Hardware/CLUSTERFCK/ALU/ALU/ALU.kicad_sch (KiCad schematic)
At the start: 30 parts, among them U1 74LS86, U10 74LS08, U2 74LS86, U3 74LS245, U4 74LS283, U5 74LS283, U8 74LS02

Commit message: unstable switching device push
Parts:
- added J1: Conn_02x20_Counter_Clockwise, Connector_PinSocket_2.54mm:PinSocket_2x20_P2.54mm_Horizontal, symbol Connector_Generic:Conn_02x20_Counter_Clockwise
Connections:
- net +5V: now also J1.21 (Pin_21), J1.22 (Pin_22), J1.39 (Pin_39), J1.40 (Pin_40)
- net CARRY: now also J1.15 (Pin_15)
- net GND: now also U10.12, U10.13, J1.1 (Pin_1), J1.19 (Pin_19), J1.2 (Pin_2), J1.20 (Pin_20)
- net SU: now also J1.16 (Pin_16)
- net ZERO: now also J1.13 (Pin_13)
- net ~EO: now also J1.14 (Pin_14)
- no-connect marks 1 -> 19
Other:
- note added: "To DATA BUS"
- moved on the sheet: C18, C19, C30, C31, U10E, U8E

Commit message: temporary unstable push
Parts:
- removed J1: Conn_02x20_Counter_Clockwise, Connector_PinSocket_2.54mm:PinSocket_2x20_P2.54mm_Horizontal, symbol Connector_Generic:Conn_02x20_Counter_Clockwise
- added J1, J2, J3: Conn_02x08_Counter_Clockwise, symbol Connector_Generic:Conn_02x08_Counter_Clockwise
- U2: renamed from U5; footprint Package_DIP:DIP-16_W7.62mm_Socket_LongPads -> Package_SO:SOIC-16W_5.3x10.2mm_P1.27mm
- U3: renamed from U4; footprint Package_DIP:DIP-16_W7.62mm_Socket_LongPads -> Package_SO:SOIC-16W_5.3x10.2mm_P1.27mm
- U5: renamed from U8; footprint Package_DIP:DIP-14_W7.62mm_Socket_LongPads -> Package_SO:SOIC-14_3.9x8.7mm_P1.27mm
- U6: renamed from U10; footprint Package_DIP:DIP-14_W7.62mm_Socket_LongPads -> Package_SO:SOIC-14_3.9x8.7mm_P1.27mm
- U7: renamed from U3; footprint Package_DIP:DIP-20_W7.62mm_Socket_LongPads -> Package_SO:SOIC-20W_7.5x12.8mm_P1.27mm
- renumbered C18 to C1, C19 to C2, C1 to C3, C30 to C5, C31 to C6, C5 to C7, D9 to D1, D10 to D2, D11 to D3, D12 to D4, D13 to D5, D14 to D6, D15 to D7, D16 to D8, R9 to R1, R10 to R2, R11 to R3, R12 to R4, R13 to R5, R14 to R6, R15 to R7, R16 to R8, U2 to U1, U1 to U4, U2 to U4
Connections:
- net +5V: now also J1.15 (Pin_15), J1.16 (Pin_16), J2.15 (Pin_15), J2.16 (Pin_16), J3.15 (Pin_15), J3.16 (Pin_16)
- net CARRY: now also J1.11 (Pin_11), J2.11 (Pin_11), J3.11 (Pin_11)
- net D0: now also J3.1 (Pin_1)
- net D1: now also J3.2 (Pin_2)
- net D2: now also J3.3 (Pin_3)
- net D3: now also J3.4 (Pin_4)
- net D4: now also J3.5 (Pin_5)
- net D5: now also J3.6 (Pin_6)
- net D6: now also J3.7 (Pin_7)
- net D7: now also J3.8 (Pin_8)
- net GND: now also J1.13 (Pin_13), J1.14 (Pin_14), J2.13 (Pin_13), J2.14 (Pin_14), J3.13 (Pin_13), J3.14 (Pin_14)
- net RA0: now also J2.8 (Pin_8)
- net RA1: now also J2.7 (Pin_7)
- net RA2: now also J2.6 (Pin_6)
- net RA3: now also J2.5 (Pin_5)
- net RA4: now also J2.4 (Pin_4)
- net RA5: now also J2.3 (Pin_3)
- net RA6: now also J2.2 (Pin_2)
- net RA7: now also J2.1 (Pin_1)
- net REGB0: now also J1.8 (Pin_8)
- net REGB1: now also J1.7 (Pin_7)
- net REGB2: now also J1.6 (Pin_6)
- net REGB3: now also J1.5 (Pin_5)
- net REGB4: now also J1.4 (Pin_4)
- net REGB5: now also J1.3 (Pin_3)
- net REGB6: now also J1.2 (Pin_2)
- net REGB7: now also J1.1 (Pin_1)
- net SU: now also J1.12 (Pin_12), J2.12 (Pin_12), J3.12 (Pin_12)
- net ZERO: now also J1.9 (Pin_9), J2.9 (Pin_9), J3.9 (Pin_9)
- net ~EO: now also J1.10 (Pin_10), J2.10 (Pin_10), J3.10 (Pin_10)
- no-connect marks 19 -> 1
Other:
- note added: "To Register A"
- note added: "To Register B"
- moved on the sheet: C5, C6, D1, D2, D3, D4, D5, D6, D7, D8, R1, R2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

Commit message: 0046|6|Alu Module
Parts:
- J1, J2, J3: footprint (none) -> Connector_PinHeader_2.54mm:PinHeader_2x08_P2.54mm_Horizontal
- U2, U3: footprint Package_SO:SOIC-16W_5.3x10.2mm_P1.27mm -> Package_SO:SO-16_5.3x10.2mm_P1.27mm
Changed lines of the file:
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@@
   (junction (at 148.3614 63.119) (diameter 0) (color 0 0 0 0))
   (junction (at 213.36 100.33) (diameter 0) (color 0 0 0 0))
+  (junction (at 82.55 64.77) (diameter 0) (color 0 0 0 0))
   (no_connect (at 198.12 100.33))
   (bus_entry (at 39.37 118.11) (size 2.54 2.54)
@@
     (stroke (width 0) (type solid) (color 0 0 0 0))
   )
-  (bus (pts (xy 46.99 33.02) (xy 46.99 35.56))
-    (stroke (width 0) (type solid) (color 0 0 0 0))
-  )
-  (bus (pts (xy 46.99 35.56) (xy 46.99 40.64))
-    (stroke (width 0) (type solid) (color 0 0 0 0))
-  )
-  (bus (pts (xy 46.99 40.64) (xy 46.99 41.91))
-    (stroke (width 0) (type solid) (color 0 0 0 0))
-  )
-  (bus (pts (xy 46.99 45.72) (xy 46.99 50.8))
-    (stroke (width 0) (type solid) (color 0 0 0 0))
-  )
-  (bus (pts (xy 46.99 50.8) (xy 46.99 54.61))
+  (bus (pts (xy 46.99 33.02) (xy 46.99 38.1))
+    (stroke (width 0) (type solid) (color 0 0 0 0))
+  )
+  (bus (pts (xy 46.99 38.1) (xy 46.99 41.91))
+    (stroke (width 0) (type solid) (color 0 0 0 0))
+  )
+  (bus (pts (xy 46.99 45.72) (xy 46.99 48.26))
+    (stroke (width 0) (type solid) (color 0 0 0 0))
+  )
+  (bus (pts (xy 46.99 48.26) (xy 46.99 53.34))
+    (stroke (width 0) (type solid) (color 0 0 0 0))
+  )
+  (bus (pts (xy 46.99 53.34) (xy 46.99 54.61))
     (stroke (width 0) (type solid) (color 0 0 0 0))
   )
@@
     (stroke (width 0) (type solid) (color 0 0 0 0))
   )
-  (bus (pts (xy 66.04 168.91) (xy 69.85 168.91))
+  (bus (pts (xy 66.04 168.91) (xy 77.47 168.91))
     (stroke (width 0) (type solid) (color 0 0 0 0))
   )
@@
     (stroke (width 0) (type solid) (color 0 0 0 0))
   )
-  (bus (pts (xy 69.85 168.91) (xy 80.01 168.91))
-    (stroke (width 0) (type solid) (color 0 0 0 0))
-  )
-  (bus (pts (xy 80.01 168.91) (xy 85.09 168.91))
+  (bus (pts (xy 77.47 168.91) (xy 85.09 168.91))
     (stroke (width 0) (type solid) (color 0 0 0 0))
   )
@@
     (stroke (width 0) (type solid) (color 0 0 0 0))
   )
-  (bus (pts (xy 82.55 82.55) (xy 82.55 92.71))
+  (bus (pts (xy 82.55 64.77) (xy 82.55 92.71))
     (stroke (width 0) (type solid) (color 0 0 0 0))
   )
@@
     (stroke (width 0) (type solid) (color 0 0 0 0))
   )
-  (bus (pts (xy 85.09 82.55) (xy 82.55 82.55))
-    (stroke (width 0) (type solid) (color 0 0 0 0))
-  )
-  (bus (pts (xy 92.456 71.882) (xy 93.726 71.882))
-    (stroke (width 0) (type solid) (color 0 0 0 0))
-  )
-  (bus (pts (xy 92.583 98.552) (xy 92.583 103.632))
-    (stroke (width 0) (type solid) (color 0 0 0 0))
-  )
-  (bus (pts (xy 92.583 103.632) (xy 92.583 108.712))
-    (stroke (width 0) (type solid) (color 0 0 0 0))
-  )
-  (bus (pts (xy 92.583 108.712) (xy 92.583 113.792))
-    (stroke (width 0) (type solid) (color 0 0 0 0))
-  )
-  (bus (pts (xy 92.583 113.792) (xy 92.583 116.332))
-    (stroke (width 0) (type solid) (color 0 0 0 0))
-  )
-  (bus (pts (xy 92.583 116.332) (xy 92.583 121.412))
-    (stroke (width 0) (type solid) (color 0 0 0 0))
-  )
-  (bus (pts (xy 93.853 70.104) (xy 93.853 73.66))
-    (stroke (width 0) (type solid) (color 0 0 0 0))
-  )
-  (bus (pts (xy 93.853 73.66) (xy 96.647 73.66))
+  (bus (pts (xy 92.583 98.552) (xy 92.583 106.172))
+    (stroke (width 0) (type solid) (color 0 0 0 0))
+  )
+  (bus (pts (xy 92.583 106.172) (xy 92.583 111.252))
+    (stroke (width 0) (type solid) (color 0 0 0 0))
+  )
+  (bus (pts (xy 92.583 111.252) (xy 92.583 113.792))
+    (stroke (width 0) (type solid) (color 0 0 0 0))
+  )
+  (bus (pts (xy 92.583 113.792) (xy 92.583 118.872))
+    (stroke (width 0) (type solid) (color 0 0 0 0))
+  )
+  (bus (pts (xy 92.583 118.872) (xy 92.583 121.412))
     (stroke (width 0) (type solid) (color 0 0 0 0))
   )
@@
     (stroke (width 0) (type solid) (color 0 0 0 0))
   )
-  (bus (pts (xy 96.393 70.104) (xy 93.853 70.104))
-    (stroke (width 0) (type solid) (color 0 0 0 0))
-  )
   (bus (pts (xy 125.603 174.879) (xy 130.683 174.879))
     (stroke (width 0) (type solid) (color 0 0 0 0))
   )
-  (bus (pts (xy 130.683 174.879) (xy 133.223 174.879))
-    (stroke (width 0) (type solid) (color 0 0 0 0))
-  )
-  (bus (pts (xy 133.223 174.879) (xy 138.303 174.879))
-    (stroke (width 0) (type solid) (color 0 0 0 0))
-  )
-  (bus (pts (xy 138.303 174.879) (xy 143.383 174.879))
-    (stroke (width 0) (type solid) (color 0 0 0 0))
-  )
-  (bus (pts (xy 143.383 174.879) (xy 148.59 174.879))
+  (bus (pts (xy 130.683 174.879) (xy 135.763 174.879))
+    (stroke (width 0) (type solid) (color 0 0 0 0))
+  )
+  (bus (pts (xy 135.763 174.879) (xy 140.843 174.879))
+    (stroke (width 0) (type solid) (color 0 0 0 0))
+  )
+  (bus (pts (xy 140.843 174.879) (xy 148.59 174.879))
     (stroke (width 0) (type solid) (color 0 0 0 0))
   )
@@
     (stroke (width 0) (type solid) (color 0 0 0 0))
   )
-  (bus (pts (xy 271.78 49.53) (xy 271.78 52.07))
-    (stroke (width 0) (type solid) (color 0 0 0 0))
-  )
-  (bus (pts (xy 271.78 52.07) (xy 271.78 57.15))
+  (bus (pts (xy 271.78 49.53) (xy 271.78 54.61))
+    (stroke (width 0) (type solid) (color 0 0 0 0))
+  )
+  (bus (pts (xy 271.78 54.61) (xy 271.78 57.15))
     (stroke (width 0) (type solid) (color 0 0 0 0))
   )
@@
     (effects (font (size 1.27 1.27)) (justify left))
   )
-  (global_label "ALU[4..7]" (shape bidirectional) (at 85.09 64.77 0)
-    (effects (font (size 1.27 1.27)) (justify left))
-  )
-  (global_label "ALU[0..3]" (shape bidirectional) (at 85.09 82.55 0)
+  (global_label "ALU[0..7]" (shape bidirectional) (at 85.09 64.77 0)
     (effects (font (size 1.27 1.27)) (justify left))
   )
@@
     (effects (font (size 1.27 1.27)) (justify left))
   )
-  (global_label "ALU[0..7]" (shape bidirectional) (at 92.456 71.882 180)
-    (effects (font (size 1.27 1.27)) (justify right))
-  )
   (global_label "ALU[0..7]" (shape bidirectional) (at 93.853 98.552 0)
-    (effects (font (size 1.27 1.27)) (justify left))
-  )
-  (global_label "ALU[4..7]" (shape bidirectional) (at 96.393 70.104 0)
-    (effects (font (size 1.27 1.27)) (justify left))
-  )
-  (global_label "ALU[0..3]" (shape bidirectional) (at 96.647 73.66 0)
     (effects (font (size 1.27 1.27)) (justify left))
   )
@@
     (property "Reference" "J1" (id 0) (at 116.205 152.527 0))
     (property "Value" "Conn_02x08_Counter_Clockwise" (id 1) (at 118.745 152.527 0))
-    (property "Footprint" "" (id 2) (at 130.683 154.559 0)
+    (property "Footprint" "Connector_PinHeader_2.54mm:PinHeader_2x08_P2.54mm_Horizontal" (id 2) (at 130.683 154.559 0)
       (effects (font (size 1.27 1.27)) hide)
     )
@@
     (property "Reference" "J2" (id 0) (at 168.021 137.795 0))
     (property "Value" "Conn_02x08_Counter_Clockwise" (id 1) (at 170.561 137.795 0))
-    (property "Footprint" "" (id 2) (at 182.499 139.827 0)
+    (property "Footprint" "Connector_PinHeader_2.54mm:PinHeader_2x08_P2.54mm_Horizontal" (id 2) (at 182.499 139.827 0)
       (effects (font (size 1.27 1.27)) hide)
     )
@@
     (property "Reference" "J3" (id 0) (at 223.52 121.539 0))
     (property "Value" "Conn_02x08_Counter_Clockwise" (id 1) (at 226.06 121.539 0))
-    (property "Footprint" "" (id 2) (at 237.998 123.571 0)
+    (property "Footprint" "Connector_PinHeader_2.54mm:PinHeader_2x08_P2.54mm_Horizontal" (id 2) (at 237.998 123.571 0)
       (effects (font (size 1.27 1.27)) hide)
     )
@@
     (property "Reference" "U2" (id 0) (at 64.77 68.0974 0))
     (property "Value" "74LS283" (id 1) (at 64.77 65.786 0))
-    (property "Footprint" "Package_SO:SOIC-16W_5.3x10.2mm_P1.27mm" (id 2) (at 64.77 43.18 0)
+    (property "Footprint" "Package_SO:SO-16_5.3x10.2mm_P1.27mm" (id 2) (at 64.77 43.18 0)
       (effects (font (size 1.27 1.27)) hide)
     )
@@
     (property "Reference" "U3" (id 0) (at 64.77 115.0874 0))
     (property "Value" "74LS283" (id 1) (at 64.77 112.776 0))
-    (property "Footprint" "Package_SO:SOIC-16W_5.3x10.2mm_P1.27mm" (id 2) (at 64.77 90.17 0)
-      (effects (font (size 1.27 1.27)) hide)
-    )
+    (property "Footprint" "Package_SO:SO-16_5.3x10.2mm_P1.27mm" (id 2) (at 64.77 90.17 0)
+      (effects (font (size 1.27 1.27)) hide)
+    )
