File: Hardware/CLUSTERFCK/ALU/ALU/ALU.kicad_pcb (KiCad board)
At the start: 2 copper layers, 33 parts, among them J1 Conn_02x20_Counter_Clockwise, J2 Conn_02x20_Counter_Clockwise, J3 Conn_02x20_Counter_Clockwise, U1 74LS86, U2 74LS283, U3 74LS283, U4 74LS86, U5 74LS02, U6 74LS08, U7 74LS245

Commit message: 0046|6|Alu Module
Parts:
- removed U7: 74LS245, Package_SO:SOIC-20W_7.5x12.8mm_P1.27mm
- added Ueee: 74LS245, Package_SO:SOIC-20W_7.5x12.8mm_P1.27mm, F.Cu at (50.5, 85.9)
- J1, J2, J3: value Conn_02x20_Counter_Clockwise -> Conn_02x08_Counter_Clockwise; footprint Connector_PinSocket_2.54mm:PinSocket_2x20_P2.54mm_Horizontal -> Connector_PinHeader_2.54mm:PinHeader_2x08_P2.54mm_Horizontal
- U2, U3: footprint Package_SO:SOIC-16W_5.3x10.2mm_P1.27mm -> Package_SO:SO-16_5.3x10.2mm_P1.27mm
- moved J1 104.5 mm to (88.0, 123.3), turned to -90 degrees
- moved R3 103.7 mm to (68.2, 106.0), turned to 90 degrees
- moved D2 98.8 mm to (60.6, 113.6), turned to 90 degrees
- moved R4 97.1 mm to (75.8, 106.0), turned to 90 degrees
- moved R6 96.8 mm to (91.0, 106.0), turned to 90 degrees
- moved R7 89.0 mm to (98.7, 106.0), turned to 90 degrees
- moved D5 85.0 mm to (83.4, 113.6), turned to 90 degrees
- moved R2 83.9 mm to (60.6, 106.0), turned to 90 degrees
- moved R1 81.7 mm to (53.0, 106.0), turned to 90 degrees
- moved C2 81.3 mm to (75.2, 79.0), turned to 180 degrees
- moved J3 72.3 mm to (27.7, 90.0), turned to 180 degrees
- moved D8 71.0 mm to (106.2, 113.6), turned to 90 degrees
- moved C7 70.3 mm to (54.3, 78.0), turned to 180 degrees
- moved U6 70.1 mm to (63.5, 65.3)
- moved R5 67.2 mm to (83.4, 106.0), turned to 90 degrees
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Connections:
- J1 pad 1: GND -> REGB7
- J1 pad 10: D7 -> ~EO
- J1 pad 11: ZERO -> CARRY
- J1 pad 12: ~EO -> SU
- J1 pad 13: CARRY -> GND
- J1 pad 14: SU -> GND
- J1 pad 15: Net-(J1-Pad15) -> +5V
- J1 pad 16: Net-(J1-Pad16) -> +5V
- J1 pad 2: GND -> REGB6
- J1 pad 3: D0 -> REGB5
- J1 pad 4: D1 -> REGB4
- J1 pad 5: D2 -> REGB3
- J1 pad 6: D3 -> REGB2
- J1 pad 7: D4 -> REGB1
- J1 pad 8: D5 -> REGB0
- J1 pad 9: D6 -> ZERO
- J2 pad 1: GND -> RA7
- J2 pad 10: REGB0 -> ~EO
- J2 pad 11: ZERO -> CARRY
- J2 pad 12: ~EO -> SU
- J2 pad 13: CARRY -> GND
- J2 pad 14: SU -> GND
- J2 pad 15: Net-(J2-Pad15) -> +5V
- J2 pad 16: Net-(J2-Pad16) -> +5V
- J2 pad 2: GND -> RA6
- J2 pad 3: REGB7 -> RA5
- J2 pad 4: REGB6 -> RA4
- J2 pad 5: REGB5 -> RA3
- J2 pad 6: REGB4 -> RA2
- J2 pad 7: REGB3 -> RA1
- J2 pad 8: REGB2 -> RA0
- J2 pad 9: REGB1 -> ZERO
- J3 pad 1: GND -> D0
- J3 pad 10: RA0 -> ~EO
- J3 pad 11: ZERO -> CARRY
- J3 pad 12: ~EO -> SU
- J3 pad 13: CARRY -> GND
- J3 pad 14: SU -> GND
- J3 pad 15: Net-(J3-Pad15) -> +5V
- J3 pad 16: Net-(J3-Pad16) -> +5V
- J3 pad 2: GND -> D1
- J3 pad 3: RA7 -> D2
- J3 pad 4: RA6 -> D3
- J3 pad 5: RA5 -> D4
- J3 pad 6: RA4 -> D5
- J3 pad 7: RA3 -> D6
- J3 pad 8: RA2 -> D7
- J3 pad 9: RA1 -> ZERO
- R1 pad 2: ALU3 -> ALU7
- R2 pad 2: ALU2 -> ALU6
- R3 pad 2: ALU1 -> ALU5
- R4 pad 2: ALU0 -> ALU4
- U2 pad 1: ALU1 -> ALU5
- U2 pad 10: ALU3 -> ALU7
- U2 pad 13: ALU2 -> ALU6
- U2 pad 4: ALU0 -> ALU4
- U5 pad 2: ALU3 -> ALU7
- U5 pad 3: ALU2 -> ALU6
- U5 pad 5: ALU1 -> ALU5
- U5 pad 6: ALU0 -> ALU4
Routing:
- net SU: track 0.00 -> 303.7 mm
- net +5V: track 0.00 -> 266.1 mm, vias 0 -> 12
- net ZERO: track 0.00 -> 215.3 mm, vias 0 -> 3
- net CARRY: track 0.00 -> 207.3 mm, vias 0 -> 2
- net ~EO: track 0.00 -> 207.2 mm, vias 0 -> 1
- net ALU0: track 0.00 -> 111.9 mm, vias 0 -> 9
- net ALU3: track 0.00 -> 105.7 mm, vias 0 -> 12
- net REGB5: track 0.00 -> 104.9 mm, vias 0 -> 3
- net REGB4: track 0.00 -> 103.5 mm, vias 0 -> 7
- net ALU1: track 0.00 -> 96.3 mm, vias 0 -> 8
- net ALU2: track 0.00 -> 93.7 mm, vias 0 -> 12
- net REGB0: track 0.00 -> 87.2 mm, vias 0 -> 2
- net ALU7: track 0.00 -> 85.6 mm, vias 0 -> 7
- net REGB6: track 0.00 -> 84.0 mm, vias 0 -> 2
- net ALU6: track 0.00 -> 79.1 mm, vias 0 -> 4
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- added copper zone on B.Cu, net D0
- added copper zone on B.Cu, net GND
- added copper zone on B.Cu, net RA7
- added copper zone on B.Cu, net REGB0
- added copper zone on B.Cu, net REGB4
- added copper zone on B.Cu, net REGB7
Other:
- board outline added: 119 x 96 mm

Commit message: 0047 | 0.5h | review ALU Module
Parts:
- renumbered C7 to Ceee
Routing:
- net GND: track 19.8 -> 134.2 mm, vias 14 -> 73
- net SU: track 303.7 -> 292.6 mm
- net +5V: track 266.1 -> 267.1 mm
- net ~EO: track 207.2 -> 207.7 mm, vias 1 -> 3
- net D2: track 28.6 -> 28.1 mm
- net REGB4: track 103.5 -> 103.2 mm, vias 7 -> 8
- net REGB0: track 87.2 -> 87.4 mm, vias 2 -> 3
- net REGB7: vias 7 -> 8
- net RA7: vias 1 -> 2
- net D0: vias 1 -> 2
- added copper zone on F.Cu, net D0
- added copper zone on F.Cu, net RA7
- added copper zone on F.Cu, net REGB0
- added copper zone on F.Cu, net REGB4
- added copper zone on F.Cu, net REGB7
- removed copper zone on B.Cu, net D0
- removed copper zone on B.Cu, net RA7
- removed copper zone on B.Cu, net REGB0
- removed copper zone on B.Cu, net REGB4
- removed copper zone on B.Cu, net REGB7
Other:
- board text added: "A(L)U Module Rev1.0 Tom Schädler 2020"

Commit message: 0053 | 3h | Layout REG_A
Routing:
- net GND: track 134.2 -> 140.5 mm, vias 73 -> 74
Changed lines of the file:
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@@
     (thickness 1.6)
     (drawings 5)
-    (tracks 1033)
+    (tracks 1037)
     (modules 33)
     (nets 63)
@@
       (dielectric_constraints no)
     )
-    (last_trace_width 0.5)
+    (last_trace_width 1)
     (user_trace_width 0.2)
     (user_trace_width 0.5)
@@
   (gr_line (start 140 34) (end 140 130) (layer "Edge.Cuts") (width 0.05))
   (gr_line (start 21 34) (end 140 34) (layer "Edge.Cuts") (width 0.05))
+  (via (at 73.93 120.1) (size 0.8) (drill 0.4) (layers "F.Cu" "B.Cu") (net 1))
+  (segment (start 73.93 122.1616) (end 73.93 120.1) (width 1) (layer "F.Cu") (net 1))
+  (segment (start 72.76 123.3316) (end 73.93 122.1616) (width 1) (layer "F.Cu") (net 1))
+  (segment (start 72.76 125.8716) (end 72.76 123.3316) (width 1) (layer "F.Cu") (net 1))
   (segment (start 58.1 36.1) (end 57.3 36.1) (width 0.5) (layer "F.Cu") (net 1))
   (segment (start 57.3 36.1) (end 56.7 35.5) (width 0.5) (layer "F.Cu") (net 1))

Commit message: 0050 | 5h | Ram module
Other:
- net class Default removed

Commit message: 0066 | 6h | made holes in pcbs
Parts:
- added REF**: MountingHole_4.3mm_M4, MountingHole:MountingHole_4.3mm_M4, F.Cu at (134.8, 124.7)
- added REF**: MountingHole_4.3mm_M4, MountingHole:MountingHole_4.3mm_M4, F.Cu at (134.8, 39.0)
- added REF**: MountingHole_4.3mm_M4, MountingHole:MountingHole_4.3mm_M4, F.Cu at (26.1, 124.7)
- added REF**: MountingHole_4.3mm_M4, MountingHole:MountingHole_4.3mm_M4, F.Cu at (26.1, 49.1)
Changed lines of the file:
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@@
   (net 61 "ALU5")
   (net 62 "ALU4")
+  (footprint "MountingHole:MountingHole_4.3mm_M4" (layer "F.Cu")
+    (at 134.78 124.66)
+    (descr "Mounting Hole 4.3mm, no annular, M4")
+    (tags "mounting hole 4.3mm no annular m4")
+    (attr exclude_from_pos_files exclude_from_bom)
+    (fp_text reference "REF**" (at 0.06 -2.99) (layer "F.SilkS")
+      (effects (font (size 1 1) (thickness 0.15)))
+    )
+    (fp_text value "MountingHole_4.3mm_M4" (at 0 5.3) (layer "F.Fab")
+      (effects (font (size 1 1) (thickness 0.15)))
+    )
+    (fp_text user "${REFERENCE}" (at 0.3 0) (layer "F.Fab")
+      (effects (font (size 1 1) (thickness 0.15)))
+    )
+    (fp_circle (center 0 0) (end 4.3 0) (layer "Cmts.User") (width 0.15) (fill none))
+    (fp_circle (center 0 0) (end 4.55 0) (layer "F.CrtYd") (width 0.05) (fill none))
+    (pad "1" np_thru_hole circle (at 0 0) (size 4.3 4.3) (drill 4.3) (layers *.Cu *.Mask))
+  )
+  (footprint "MountingHole:MountingHole_4.3mm_M4" (layer "F.Cu")
+    (at 134.78 39.02)
+    (descr "Mounting Hole 4.3mm, no annular, M4")
+    (tags "mounting hole 4.3mm no annular m4")
+    (attr exclude_from_pos_files exclude_from_bom)
+    (fp_text reference "REF**" (at 0.06 -2.99) (layer "F.SilkS")
+      (effects (font (size 1 1) (thickness 0.15)))
+    )
+    (fp_text value "MountingHole_4.3mm_M4" (at 0 5.3) (layer "F.Fab")
+      (effects (font (size 1 1) (thickness 0.15)))
+    )
+    (fp_text user "${REFERENCE}" (at 0.3 0) (layer "F.Fab")
+      (effects (font (size 1 1) (thickness 0.15)))
+    )
+    (fp_circle (center 0 0) (end 4.3 0) (layer "Cmts.User") (width 0.15) (fill none))
+    (fp_circle (center 0 0) (end 4.55 0) (layer "F.CrtYd") (width 0.05) (fill none))
+    (pad "1" np_thru_hole circle (at 0 0) (size 4.3 4.3) (drill 4.3) (layers *.Cu *.Mask))
+  )
   (footprint "Package_DIP:DIP-14_W7.62mm_Socket_LongPads" (layer "F.Cu")
     (at 104.36 80.64)
@@
       (rotate (xyz 0 0 0))
     )
+  )
+  (footprint "MountingHole:MountingHole_4.3mm_M4" (layer "F.Cu")
+    (at 26.05 124.66)
+    (descr "Mounting Hole 4.3mm, no annular, M4")
+    (tags "mounting hole 4.3mm no annular m4")
+    (attr exclude_from_pos_files exclude_from_bom)
+    (fp_text reference "REF**" (at 0.06 -2.99) (layer "F.SilkS")
+      (effects (font (size 1 1) (thickness 0.15)))
+    )
+    (fp_text value "MountingHole_4.3mm_M4" (at 0 5.3) (layer "F.Fab")
+      (effects (font (size 1 1) (thickness 0.15)))
+    )
+    (fp_text user "${REFERENCE}" (at 0.3 0) (layer "F.Fab")
+      (effects (font (size 1 1) (thickness 0.15)))
+    )
+    (fp_circle (center 0 0) (end 4.3 0) (layer "Cmts.User") (width 0.15) (fill none))
+    (fp_circle (center 0 0) (end 4.55 0) (layer "F.CrtYd") (width 0.05) (fill none))
+    (pad "1" np_thru_hole circle (at 0 0) (size 4.3 4.3) (drill 4.3) (layers *.Cu *.Mask))
   )
   (footprint "Connector_PinHeader_2.54mm:PinHeader_2x08_P2.54mm_Horizontal" (layer "F.Cu")
@@
       (rotate (xyz 0 0 0))
     )
+  )
+  (footprint "MountingHole:MountingHole_4.3mm_M4" (layer "F.Cu")
+    (at 26.05 49.1)
+    (descr "Mounting Hole 4.3mm, no annular, M4")
+    (tags "mounting hole 4.3mm no annular m4")
+    (attr exclude_from_pos_files exclude_from_bom)
+    (fp_text reference "REF**" (at 0.06 -2.99) (layer "F.SilkS")
+      (effects (font (size 1 1) (thickness 0.15)))
+    )
+    (fp_text value "MountingHole_4.3mm_M4" (at 0 5.3) (layer "F.Fab")
+      (effects (font (size 1 1) (thickness 0.15)))
+    )
+    (fp_text user "${REFERENCE}" (at 0.3 0) (layer "F.Fab")
+      (effects (font (size 1 1) (thickness 0.15)))
+    )
+    (fp_circle (center 0 0) (end 4.3 0) (layer "Cmts.User") (width 0.15) (fill none))
+    (fp_circle (center 0 0) (end 4.55 0) (layer "F.CrtYd") (width 0.05) (fill none))
+    (pad "1" np_thru_hole circle (at 0 0) (size 4.3 4.3) (drill 4.3) (layers *.Cu *.Mask))
   )
   (footprint "Resistor_SMD:R_0805_2012Metric_Pad1.15x1.40mm_HandSolder" (layer "F.Cu")
@@
   (segment (start 54.475 89.055) (end 55.18 89.055) (width 0.2) (layer "F.Cu") (net 12))
   (segment (start 27.7368 87.46) (end 28.73179 88.45499) (width 0.2) (layer "F.Cu") (net 12))
+  (segment (start 47.72 94.93) (end 52.325 90.325) (width 0.2) (layer "F.Cu") (net 13))
   (segment (start 47.71 94.94) (end 47.72 94.93) (width 0.25) (layer "F.Cu") (net 13))
-  (segment (start 47.72 94.93) (end 52.325 90.325) (width 0.2) (layer "F.Cu") (net 13))
   (segment (start 52.325 90.325) (end 55.18 90.325) (width 0.2) (layer "F.Cu") (net 13))
   (via (at 47.72 94.93) (size 0.43) (drill 0.3) (layers "F.Cu" "B.Cu") (net 13))
@@
   (segment (start 109.01 83.88) (end 109.01 82.84) (width 0.2) (layer "B.Cu") (net 15))
   (segment (start 117.37 89.67) (end 113.83 86.13) (width 0.2) (layer "B.Cu") (net 15))
+  (segment (start 109.01 82.84) (end 106.855 80.685) (width 0.2) (layer "B.Cu") (net 15))
   (segment (start 106.855 80.685) (end 106.83 80.66) (width 0.2) (layer "B.Cu") (net 15))
-  (segment (start 109.01 82.84) (end 106.855 80.685) (width 0.2) (layer "B.Cu") (net 15))
   (segment (start 87.15 105.47) (end 87.15 116.5616) (width 0.2) (layer "F.Cu") (net 16))
   (segment (start 87.15 116.5616) (end 80.38 123.3316) (width 0.2) (layer "F.Cu") (net 16))
@@
   (via (at 73.835 57.165) (size 0.43) (drill 0.3) (layers "F.Cu" "B.Cu") (net 27))
   (via (at 71.825 59.175) (size 0.43) (drill 0.3) (layers "F.Cu" "B.Cu") (net 27))
+  (segment (start 73.835 57.165) (end 71.825 59.175) (width 0.2) (layer "B.Cu") (net 27))
   (segment (start 71.825 59.175) (end 71.82 59.18) (width 0.2) (layer "B.Cu") (net 27))
-  (segment (start 73.835 57.165) (end 71.825 59.175) (width 0.2) (layer "B.Cu") (net 27))
   (segment (start 76.54 55.94) (end 73.87 58.61) (width 0.2) (layer "F.Cu") (net 28))
   (segment (start 71.88 60.48) (end 71.88 63.082798) (width 0.2) (layer "F.Cu") (net 28))
@@
   (via (at 83.43 75.84) (size 0.43) (drill 0.3) (layers "F.Cu" "B.Cu") (net 38))
   (via (at 79.59 79.68) (size 0.43) (drill 0.3) (layers "F.Cu" "B.Cu") (net 38))
+  (segment (start 83.43 75.84) (end 83.46 75.81) (width 0.2) (layer "B.Cu") (net 38))
   (segment (start 79.59 79.68) (end 83.43 75.84) (width 0.2) (layer "B.Cu") (net 38))
-  (segment (start 83.43 75.84) (end 83.46 75.81) (width 0.2) (layer "B.Cu") (net 38))
   (via (at 92.8 82.26) (size 0.43) (drill 0.3) (layers "F.Cu" "B.Cu") (net 39))
   (segment (start 92.8 82.26) (end 95.11 84.57) (width 0.2) (layer "B.Cu") (net 39))
@@
   (zone (net 14) (net_name "D0") (layer "F.Cu") (hatch edge 0.508)
     (connect_pads (clearance 0.508))
-    (min_thickness 0.254)
+    (min_thickness 0.254) (filled_areas_thickness no)
     (fill yes (thermal_gap 0.508) (thermal_bridge_width 0.508))
     (polygon
@@
   (zone (net 22) (net_name "REGB7") (layer "F.Cu") (hatch edge 0.508)
     (connect_pads (clearance 0.508))
-    (min_thickness 0.254)
+    (min_thickness 0.254) (filled_areas_thickness no)
     (fill yes (thermal_gap 0.508) (thermal_bridge_width 0.508))
     (polygon
@@
   (zone (net 15) (net_name "REGB0") (layer "F.Cu") (hatch edge 0.508)
     (connect_pads (clearance 0.508))
-    (min_thickness 0.254)
+    (min_thickness 0.254) (filled_areas_thickness no)
     (fill yes (thermal_gap 0.508) (thermal_bridge_width 0.508))
     (polygon
@@
   (zone (net 19) (net_name "REGB4") (layer "F.Cu") (hatch edge 0.508)
     (connect_pads (clearance 0.508))
-    (min_thickness 0.254)
+    (min_thickness 0.254) (filled_areas_thickness no)
     (fill yes (thermal_gap 0.508) (thermal_bridge_width 0.508))
     (polygon
@@
   (zone (net 30) (net_name "RA7") (layer "F.Cu") (hatch edge 0.508)
     (connect_pads (clearance 0.508))
-    (min_thickness 0.254)
+    (min_thickness 0.254) (filled_areas_thickness no)
     (fill yes (thermal_gap 0.508) (thermal_bridge_width 0.508))
     (polygon
@@
   (zone (net 1) (net_name "GND") (layer "B.Cu") (hatch edge 0.508)
     (connect_pads (clearance 0.508))
-    (min_thickness 0.254)
+    (min_thickness 0.254) (filled_areas_thickness no)
     (fill yes (thermal_gap 0.508) (thermal_bridge_width 0.508))
     (polygon
