File: Hardware/CLUSTERFCK/ALU/ALU/ALU.kicad_pcb (KiCad board)
At the start: 2 copper layers, 119 x 96 mm, 37 parts, among them J1 Conn_02x08_Counter_Clockwise, J2 Conn_02x08_Counter_Clockwise, J3 Conn_02x08_Counter_Clockwise, U1 74LS86, U2 74LS283, U3 74LS283, U4 74LS86, U5 74LS02, U6 74LS08

Commit message: 0072 | 3h | make silkscreen prettier
Changed lines of the file:
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@@
     (tags "THT DIP DIL PDIP 2.54mm 7.62mm 300mil Socket LongPads")
     (attr through_hole)
-    (fp_text reference "U4" (at 3.35 -2.53) (layer "F.SilkS")
+    (fp_text reference "U4" (at 1.71 -2.3) (layer "F.SilkS")
       (effects (font (size 1 1) (thickness 0.15)))
     )
@@
     (tags "resistor handsolder")
     (attr smd)
-    (fp_text reference "R1" (at 0 -1.65 90) (layer "F.SilkS")
+    (fp_text reference "R1" (at 0.03 -1.9 180) (layer "F.SilkS")
       (effects (font (size 1 1) (thickness 0.15)))
     )
@@
     (tags "capacitor handsolder")
     (attr smd)
-    (fp_text reference "C6" (at -2.8618 0.1284) (layer "F.SilkS")
+    (fp_text reference "C6" (at -0.0918 1.6684) (layer "F.SilkS")
       (effects (font (size 1 1) (thickness 0.15)))
     )
@@
     (tags "Through hole angled pin header THT 2x08 2.54mm double row")
     (attr through_hole)
-    (fp_text reference "J3" (at 5.655 -2.27) (layer "F.SilkS")
+    (fp_text reference "J3" (at 1.1968 20.16) (layer "F.SilkS")
       (effects (font (size 1 1) (thickness 0.15)))
     )
@@
     (tags "SO SO")
     (attr smd)
-    (fp_text reference "U2" (at -1.1 -6.2352) (layer "F.SilkS")
+    (fp_text reference "U2" (at -1.79 -6.2552) (layer "F.SilkS")
       (effects (font (size 1 1) (thickness 0.15)))
     )
@@
     (tags "SOIC SO")
     (attr smd)
-    (fp_text reference "U6" (at -2.165 -5.67) (layer "F.SilkS")
+    (fp_text reference "U6" (at -2.735 -5.27) (layer "F.SilkS")
       (effects (font (size 1 1) (thickness 0.15)))
     )
@@
     (tags "THT DIP DIL PDIP 2.54mm 7.62mm 300mil Socket LongPads")
     (attr through_hole)
-    (fp_text reference "U1" (at 3.81 -2.33) (layer "F.SilkS")
+    (fp_text reference "U1" (at 1.62 -2.27) (layer "F.SilkS")
       (effects (font (size 1 1) (thickness 0.15)))
     )
@@
     (tags "SOIC SO")
     (attr smd)
-    (fp_text reference "U5" (at -2.5212 -5.512) (layer "F.SilkS")
+    (fp_text reference "U5" (at -2.6412 -5.302) (layer "F.SilkS")
       (effects (font (size 1 1) (thickness 0.15)))
     )
@@
     (tags "capacitor handsolder")
     (attr smd)
-    (fp_text reference "C1" (at -3.115 -0.08) (layer "F.SilkS")
+    (fp_text reference "C1" (at -0.015 1.6) (layer "F.SilkS")
       (effects (font (size 1 1) (thickness 0.15)))
     )
@@
     (tags "capacitor handsolder")
     (attr smd)
-    (fp_text reference "C3" (at -2.92 -0.13) (layer "F.SilkS")
+    (fp_text reference "C3" (at 0.12 1.74) (layer "F.SilkS")
       (effects (font (size 1 1) (thickness 0.15)))
     )
@@
     (tags "SOIC SO")
     (attr smd)
-    (fp_text reference "Ueee" (at 0 -7.35) (layer "F.SilkS")
+    (fp_text reference "Ueee" (at -2.88 -7.41) (layer "F.SilkS")
       (effects (font (size 1 1) (thickness 0.15)))
     )
@@
     (tags "Through hole angled pin header THT 2x08 2.54mm double row")
     (attr through_hole)
-    (fp_text reference "J2" (at 5.655 -2.27 90) (layer "F.SilkS")
+    (fp_text reference "J2" (at 1.3 -2.49 180) (layer "F.SilkS")
       (effects (font (size 1 1) (thickness 0.15)))
     )
@@
     (tags "SO SO")
     (attr smd)
-    (fp_text reference "U3" (at -1.03125 -6.23375) (layer "F.SilkS")
+    (fp_text reference "U3" (at -2.54125 -6.44375) (layer "F.SilkS")
       (effects (font (size 1 1) (thickness 0.15)))
     )
@@
     (tags "resistor handsolder")
     (attr smd)
-    (fp_text reference "R7" (at 0 -1.65 90) (layer "F.SilkS")
+    (fp_text reference "R7" (at -0.05 -1.8492 180) (layer "F.SilkS")
       (effects (font (size 1 1) (thickness 0.15)))
     )
@@
     (tags "resistor handsolder")
     (attr smd)
-    (fp_text reference "R8" (at 0 -1.65 90) (layer "F.SilkS")
+    (fp_text reference "R8" (at -0.06 -1.813 180) (layer "F.SilkS")
       (effects (font (size 1 1) (thickness 0.15)))
     )
@@
     (tags "resistor handsolder")
     (attr smd)
-    (fp_text reference "R4" (at 0 -1.65 90) (layer "F.SilkS")
+    (fp_text reference "R4" (at 0.04 -1.8392 180) (layer "F.SilkS")
       (effects (font (size 1 1) (thickness 0.15)))
     )
@@
     (tags "Through hole angled pin header THT 2x08 2.54mm double row")
     (attr through_hole)
-    (fp_text reference "J1" (at 5.655 -2.27 90) (layer "F.SilkS")
+    (fp_text reference "J1" (at 1.3584 20.21 180) (layer "F.SilkS")
       (effects (font (size 1 1) (thickness 0.15)))
     )
@@
     (tags "resistor handsolder")
     (attr smd)
-    (fp_text reference "R5" (at 0 -1.65 90) (layer "F.SilkS")
+    (fp_text reference "R5" (at -0.06 -1.8392 180) (layer "F.SilkS")
       (effects (font (size 1 1) (thickness 0.15)))
     )
@@
     (tags "capacitor handsolder")
     (attr smd)
-    (fp_text reference "C2" (at -2.88 -0.19) (layer "F.SilkS")
+    (fp_text reference "C2" (at 0.02 1.7) (layer "F.SilkS")
       (effects (font (size 1 1) (thickness 0.15)))
     )
@@
     (tags "resistor handsolder")
     (attr smd)
-    (fp_text reference "R6" (at 0 -1.65 90) (layer "F.SilkS")
+    (fp_text reference "R6" (at -0.11 -1.8192 180) (layer "F.SilkS")
       (effects (font (size 1 1) (thickness 0.15)))
     )
@@
     (tags "capacitor handsolder")
     (attr smd)
-    (fp_text reference "C4" (at -2.985 0) (layer "F.SilkS")
+    (fp_text reference "C4" (at 0.035 1.66) (layer "F.SilkS")
       (effects (font (size 1 1) (thickness 0.15)))
     )
@@
     (tags "resistor handsolder")
     (attr smd)
-    (fp_text reference "R2" (at 0 -1.65 90) (layer "F.SilkS")
+    (fp_text reference "R2" (at 0.01 -1.8392 180) (layer "F.SilkS")
       (effects (font (size 1 1) (thickness 0.15)))
     )
@@
     (tags "capacitor handsolder")
     (attr smd)
-    (fp_text reference "Ceee" (at -3.66 -0.094) (layer "F.SilkS")
+    (fp_text reference "Ceee" (at -0.1 1.726) (layer "F.SilkS")
       (effects (font (size 1 1) (thickness 0.15)))
     )
@@
     (tags "capacitor handsolder")
     (attr smd)
-    (fp_text reference "C5" (at -2.78 -0.14) (layer "F.SilkS")
+    (fp_text reference "C5" (at 0.02 1.64) (layer "F.SilkS")
       (effects (font (size 1 1) (thickness 0.15)))
     )
@@
     (tags "resistor handsolder")
     (attr smd)
-    (fp_text reference "R3" (at 0 -1.65 90) (layer "F.SilkS")
+    (fp_text reference "R3" (at -0.04 -1.8592 180) (layer "F.SilkS")
       (effects (font (size 1 1) (thickness 0.15)))
     )
@@
   (segment (start 94.57 69.23) (end 94.75 69.05) (width 0.2) (layer "F.Cu") (net 1))
   (segment (start 92.19 91.51) (end 91.64 91.51) (width 0.2) (layer "F.Cu") (net 1))
+  (segment (start 90.17 79) (end 89 79) (width 0.5) (layer "F.Cu") (net 1))
+  (segment (start 109.89 78) (end 108.72 78) (width 0.5) (layer "F.Cu") (net 1))
   (segment (start 110.02 49.05) (end 108.85 49.05) (width 0.5) (layer "F.Cu") (net 1))
-  (segment (start 109.89 78) (end 108.72 78) (width 0.5) (layer "F.Cu") (net 1))
-  (segment (start 90.17 79) (end 89 79) (width 0.5) (layer "F.Cu") (net 1))
   (segment (start 73.93 122.1616) (end 73.93 120.1) (width 1) (layer "F.Cu") (net 1))
   (segment (start 94.57 69.13) (end 94.49 69.05) (width 0.2) (layer "F.Cu") (net 1))
@@
   (via (at 42.8 52.1) (size 0.43) (drill 0.3) (layers "F.Cu" "B.Cu") (net 1))
   (via (at 108.72 78) (size 0.8) (drill 0.4) (layers "F.Cu" "B.Cu") (net 1))
+  (via (at 89 79) (size 0.8) (drill 0.4) (layers "F.Cu" "B.Cu") (net 1))
   (via (at 108.85 49.05) (size 0.8) (drill 0.4) (layers "F.Cu" "B.Cu") (net 1))
-  (via (at 89 79) (size 0.8) (drill 0.4) (layers "F.Cu" "B.Cu") (net 1))
   (via (at 62.95 62.42) (size 0.43) (drill 0.3) (layers "F.Cu" "B.Cu") (net 1))
   (via (at 87.03 86.37) (size 0.43) (drill 0.3) (layers "F.Cu" "B.Cu") (net 1))
@@
   (segment (start 54.475 89.055) (end 55.18 89.055) (width 0.2) (layer "F.Cu") (net 12))
   (segment (start 27.7368 87.46) (end 28.73179 88.45499) (width 0.2) (layer "F.Cu") (net 12))
+  (segment (start 47.71 94.94) (end 47.72 94.93) (width 0.25) (layer "F.Cu") (net 13))
   (segment (start 47.72 94.93) (end 52.325 90.325) (width 0.2) (layer "F.Cu") (net 13))
-  (segment (start 47.71 94.94) (end 47.72 94.93) (width 0.25) (layer "F.Cu") (net 13))
   (segment (start 52.325 90.325) (end 55.18 90.325) (width 0.2) (layer "F.Cu") (net 13))
   (via (at 47.72 94.93) (size 0.43) (drill 0.3) (layers "F.Cu" "B.Cu") (net 13))
@@
   (segment (start 105.06 59.32) (end 106.49999 60.75999) (width 0.2) (layer "B.Cu") (net 20))
   (segment (start 99.88 128.35) (end 99.88 128.33) (width 0.2) (layer "B.Cu") (net 20))
+  (segment (start 114.18001 60.75999) (end 116.44501 63.02499) (width 0.2) (layer "B.Cu") (net 20))
   (segment (start 116.44501 63.02499) (end 116.5 63.07998) (width 0.2) (layer "B.Cu") (net 20))
-  (segment (start 114.18001 60.75999) (end 116.44501 63.02499) (width 0.2) (layer "B.Cu") (net 20))
   (segment (start 97.48 125.93) (end 97.48 125.91) (width 0.2) (layer "B.Cu") (net 20))
   (segment (start 104.4 59.32) (end 105.06 59.32) (width 0.2) (layer "B.Cu") (net 20))
