File: Hardware/CLUSTERFCK/ROM/ROM.kicad_sch (KiCad schematic)
At the start: 11 parts, among them J1 Conn_02x20_Counter_Clockwise, J2 Conn_02x20_Counter_Clockwise, J4 Conn_02x08_Counter_Clockwise, J6 Conn_02x06_Counter_Clockwise, SW3 SW_DIP_x02, U30 28c64, U31 28c64

Commit message: 0048 | 5h | Layout ROM
Connections:
- net MEMADDR0: now also J6.11 (Pin_11); no longer J6.1 (Pin_1)
- net MEMADDR1: now also J6.12 (Pin_12); no longer J6.2 (Pin_2)
- net MEMADDR10: now also J6.1 (Pin_1); no longer J6.11 (Pin_11)
- net MEMADDR11: now also J6.2 (Pin_2); no longer J6.12 (Pin_12)
- net MEMADDR2: now also J6.9 (Pin_9); no longer J6.3 (Pin_3)
- net MEMADDR3: now also J6.10 (Pin_10); no longer J6.4 (Pin_4)
- net MEMADDR4: now also J6.7 (Pin_7); no longer J6.5 (Pin_5)
- net MEMADDR5: now also J6.8 (Pin_8); no longer J6.6 (Pin_6)
- net MEMADDR6: now also J6.5 (Pin_5); no longer J6.7 (Pin_7)
- net MEMADDR7: now also J6.6 (Pin_6); no longer J6.8 (Pin_8)
- net MEMADDR8: now also J6.3 (Pin_3); no longer J6.9 (Pin_9)
- net MEMADDR9: now also J6.4 (Pin_4); no longer J6.10 (Pin_10)
- net ROM0: now also J4.15 (Pin_15); no longer J4.1 (Pin_1)
- net ROM1: now also J4.16 (Pin_16); no longer J4.2 (Pin_2)
- net ROM10: now also J4.5 (Pin_5); no longer J4.11 (Pin_11)
- net ROM11: now also J4.6 (Pin_6); no longer J4.12 (Pin_12)
- net ROM12: now also J4.3 (Pin_3); no longer J4.13 (Pin_13)
- net ROM13: now also J4.4 (Pin_4); no longer J4.14 (Pin_14)
- net ROM14: now also J4.1 (Pin_1); no longer J4.15 (Pin_15)
- net ROM15: now also J4.2 (Pin_2); no longer J4.16 (Pin_16)
- net ROM2: now also J4.13 (Pin_13); no longer J4.3 (Pin_3)
- net ROM3: now also J4.14 (Pin_14); no longer J4.4 (Pin_4)
- net ROM4: now also J4.11 (Pin_11); no longer J4.5 (Pin_5)
- net ROM5: now also J4.12 (Pin_12); no longer J4.6 (Pin_6)
- net ROM6: now also J4.9 (Pin_9); no longer J4.7 (Pin_7)
- net ROM7: now also J4.10 (Pin_10); no longer J4.8 (Pin_8)
- net ROM8: now also J4.7 (Pin_7); no longer J4.9 (Pin_9)
- net ROM9: now also J4.8 (Pin_8); no longer J4.10 (Pin_10)
