File: Hardware/CLUSTERFCK/REG_A/REG_A/REG_A.kicad_sch (KiCad schematic)
At the start: 20 parts, among them U11 74LS173, U12 74LS173

Commit message: 17 | 1h | beautifyed several scematics
Other:
- company: (none) -> Wilhelm-Maybach-Schule Heilbronn
- title: (none) -> REGISTER A
Changed lines of the file:
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@@
   (page 1 1)
   (paper "A4")
+  (title_block
+    (title "REGISTER A")
+    (date "2020-10-10")
+    (rev "1")
+    (company "Wilhelm-Maybach-Schule Heilbronn")
+    (comment 1 "Leon Hellmich")
+  )
   (junction (at 76.2 89.535) (diameter 0) (color 0 0 0 0))
   (junction (at 77.47 81.915) (diameter 0) (color 0 0 0 0))
@@
     (stroke (width 0) (type solid) (color 0 0 0 0))
   )
-  (bus (pts (xy 101.6 84.455) (xy 101.6 88.265))
-    (stroke (width 0) (type solid) (color 0 0 0 0))
-  )
-  (bus (pts (xy 101.6 88.265) (xy 101.6 93.345))
-    (stroke (width 0) (type solid) (color 0 0 0 0))
-  )
-  (bus (pts (xy 101.6 93.345) (xy 101.6 95.885))
+  (bus (pts (xy 101.6 84.455) (xy 101.6 90.805))
+    (stroke (width 0) (type solid) (color 0 0 0 0))
+  )
+  (bus (pts (xy 101.6 90.805) (xy 101.6 95.885))
     (stroke (width 0) (type solid) (color 0 0 0 0))
   )
@@
     (stroke (width 0) (type solid) (color 0 0 0 0))
   )
-  (bus (pts (xy 130.81 61.595) (xy 133.35 61.595))
-    (stroke (width 0) (type solid) (color 0 0 0 0))
-  )
-  (bus (pts (xy 133.35 61.595) (xy 138.43 61.595))
-    (stroke (width 0) (type solid) (color 0 0 0 0))
-  )
-  (bus (pts (xy 138.43 61.595) (xy 140.97 61.595))
-    (stroke (width 0) (type solid) (color 0 0 0 0))
-  )
+  (bus (pts (xy 130.81 61.595) (xy 135.89 61.595))
+    (stroke (width 0) (type solid) (color 0 0 0 0))
+  )
+  (bus (pts (xy 135.89 61.595) (xy 140.97 61.595))
+    (stroke (width 0) (type solid) (color 0 0 0 0))
+  )

Commit message: 0053 | 3h | Layout REG_A
Parts:
- added J1: Conn_02x20_Counter_Clockwise, Connector_PinHeader_2.54mm:PinHeader_2x20_P2.54mm_Horizontal, symbol Connector_Generic:Conn_02x20_Counter_Clockwise
- added J2, J3: Conn_02x08_Counter_Clockwise, Connector_PinHeader_2.54mm:PinHeader_2x08_P2.54mm_Horizontal, symbol Connector_Generic:Conn_02x08_Counter_Clockwise
- U11, U12: footprint Package_DIP:DIP-16_W7.62mm_Socket_LongPads -> Package_SO:SOIC-16W_7.5x10.3mm_P1.27mm
Connections:
- net +5V: now also J1.21 (Pin_21), J1.22 (Pin_22), J1.39 (Pin_39), J1.40 (Pin_40), J2.1 (Pin_1), J2.2 (Pin_2), J3.1 (Pin_1), J3.2 (Pin_2)
- net CLK: now also J1.11 (Pin_11)
- net D0: now also J1.3 (Pin_3)
- net D1: now also J1.4 (Pin_4)
- net D2: now also J1.5 (Pin_5)
- net D3: now also J1.6 (Pin_6)
- net D4: now also J1.7 (Pin_7)
- net D5: now also J1.8 (Pin_8)
- net D6: now also J1.9 (Pin_9)
- net D7: now also J1.10 (Pin_10)
- net GND: now also J1.1 (Pin_1), J1.19 (Pin_19), J1.2 (Pin_2), J1.20 (Pin_20), J2.3 (Pin_3), J2.4 (Pin_4), J3.3 (Pin_3), J3.4 (Pin_4)
- net RA0: now also J2.10 (Pin_10), J3.10 (Pin_10)
- net RA1: now also J2.9 (Pin_9), J3.9 (Pin_9)
- net RA2: now also J2.12 (Pin_12), J3.12 (Pin_12)
- net RA3: now also J2.11 (Pin_11), J3.11 (Pin_11)
- net RA4: now also J2.14 (Pin_14), J3.14 (Pin_14)
- net RA5: now also J2.13 (Pin_13), J3.13 (Pin_13)
- net RA6: now also J2.16 (Pin_16), J3.16 (Pin_16)
- net RA7: now also J2.15 (Pin_15), J3.15 (Pin_15)
- net ~AI: now also J1.12 (Pin_12)
- no-connect marks 0 -> 30
