File: Hardware/CLUSTERFCK/REG_A/REG_A/REG_A.kicad_pcb (KiCad board)
At the start: 2 copper layers, 119 x 79.3 mm, 23 parts, among them J1 Conn_02x20_Counter_Clockwise, J2 Conn_02x08_Counter_Clockwise, J3 Conn_02x08_Counter_Clockwise, U11 74LS173, U12 74LS173

Commit message: 0054 | 0,5h | review REG_A
Routing:
- net GND: vias 65 -> 75
Other:
- board text added: "Register A / B"
- board text removed: "REGister A / B"
Changed lines of the file:
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@@
     (thickness 1.6)
     (drawings 8)
-    (tracks 316)
+    (tracks 327)
     (modules 23)
     (nets 29)
@@
       (dielectric_constraints no)
     )
-    (last_trace_width 1)
+    (last_trace_width 0.25)
     (user_trace_width 0.2)
     (user_trace_width 0.5)
@@
     (pad_drill 0.762)
     (pad_to_mask_clearance 0)
-    (visible_elements 7FFFFFFF)
+    (visible_elements 7FFFF7FF)
     (pcbplotparams
       (layerselection 0x010fc_ffffffff)
@@
     (effects (font (size 1.5 1.5) (thickness 0.2)))
   )
-  (gr_text "REGister A / B" (at 98.552 5.588) (layer "F.SilkS")
+  (gr_text "Register A / B" (at 98.552 5.588) (layer "F.SilkS")
     (effects (font (size 3 3) (thickness 0.4)))
   )
@@
   )
   (gr_line (start 0 0) (end 119 0) (layer "Edge.Cuts") (width 0.05))
+  (segment (start 51.73 25.7) (end 33.057 25.7) (width 0.2) (layer "F.Cu") (net 26))
+  (segment (start 57.72 31.69) (end 51.73 25.7) (width 0.2) (layer "F.Cu") (net 26))
+  (segment (start 33.057 25.7) (end 31.496 24.139) (width 0.2) (layer "F.Cu") (net 26))
+  (via (at 11.03 51.71) (size 0.45) (drill 0.3) (layers "F.Cu" "B.Cu") (net 1))
+  (segment (start 11.03 51.71) (end 59.93 51.71) (width 0.2) (layer "B.Cu") (net 1))
+  (via (at 16.23 51.37) (size 0.45) (drill 0.3) (layers "F.Cu" "B.Cu") (net 1))
+  (via (at 50.22 51.36) (size 0.45) (drill 0.3) (layers "F.Cu" "B.Cu") (net 1))
+  (via (at 50.21 53.39) (size 0.45) (drill 0.3) (layers "F.Cu" "B.Cu") (net 1))
+  (via (at 13.68 53.47) (size 0.8) (drill 0.4) (layers "F.Cu" "B.Cu") (net 1))
+  (via (at 20.96 41.43) (size 0.8) (drill 0.4) (layers "F.Cu" "B.Cu") (net 1))
+  (via (at 66.76 35.89) (size 0.8) (drill 0.4) (layers "F.Cu" "B.Cu") (net 1))
+  (via (at 66.67 41.09) (size 0.8) (drill 0.4) (layers "F.Cu" "B.Cu") (net 1))
+  (via (at 65.65 26.71) (size 0.8) (drill 0.4) (layers "F.Cu" "B.Cu") (net 1))
+  (via (at 76.99 11.63) (size 0.8) (drill 0.4) (layers "F.Cu" "B.Cu") (net 1))
   (via (at 58.928 44.196) (size 0.8) (drill 0.4) (layers "F.Cu" "B.Cu") (net 1))
   (via (at 55.372 44.196) (size 0.8) (drill 0.4) (layers "F.Cu" "B.Cu") (net 1))
@@
   (via (at 51.649986 63.880028) (size 0.8) (drill 0.4) (layers "F.Cu" "B.Cu") (net 2))
   (via (at 59.93 51.71) (size 0.45) (drill 0.3) (layers "F.Cu" "B.Cu") (net 1))
-  (segment (start 8.99 51.71) (end 59.93 51.71) (width 0.2) (layer "B.Cu") (net 1))
+  (segment (start 8.99 51.71) (end 11.03 51.71) (width 0.2) (layer "B.Cu") (net 1))
   (via (at 8.99 52.96) (size 0.45) (drill 0.3) (layers "F.Cu" "B.Cu") (net 1))
   (via (at 8.99 51.71) (size 0.45) (drill 0.3) (layers "F.Cu" "B.Cu") (net 1))
@@
   (segment (start 57.72 31.69) (end 57.72 16.48) (width 0.2) (layer "B.Cu") (net 26))
   (via (at 57.72 31.69) (size 0.45) (drill 0.3) (layers "F.Cu" "B.Cu") (net 26))
-  (segment (start 57.72 31.69) (end 51.44402 25.41402) (width 0.2) (layer "F.Cu") (net 26))
   (segment (start 57.177673 15.982327) (end 65.73 7.43) (width 0.2) (layer "F.Cu") (net 25))
   (segment (start 65.73 7.43) (end 65.73 5.37) (width 0.2) (layer "F.Cu") (net 25))
@@
   (via (at 57.177673 30.122327) (size 0.45) (drill 0.3) (layers "F.Cu" "B.Cu") (net 25))
   (segment (start 57.177673 30.122327) (end 52.069356 25.01401) (width 0.2) (layer "F.Cu") (net 25))
-  (segment (start 51.44402 25.41402) (end 32.77102 25.41402) (width 0.2) (layer "F.Cu") (net 26))
-  (segment (start 32.77102 25.41402) (end 31.496 24.139) (width 0.2) (layer "F.Cu") (net 26))
   (segment (start 56.625 15.475) (end 64.46 7.64) (width 0.2) (layer "F.Cu") (net 24))
   (segment (start 64.46 7.64) (end 64.46 6.64) (width 0.2) (layer "F.Cu") (net 24))

Commit message: 0066 | 6h | made holes in pcbs
Parts:
- added REF**: MountingHole_4.3mm_M4, MountingHole:MountingHole_4.3mm_M4, F.Cu at (5.51, 73.7)
- added REF**: MountingHole_4.3mm_M4, MountingHole:MountingHole_4.3mm_M4, F.Cu at (113.1, 5.87)
- added REF**: MountingHole_4.3mm_M4, MountingHole:MountingHole_4.3mm_M4, F.Cu at (113.1, 73.7)
- added REF**: MountingHole_4.3mm_M4, MountingHole:MountingHole_4.3mm_M4, F.Cu at (5.51, 5.87)
Other:
- net class Default removed

Commit message: 0072 | 3h | make silkscreen prettier
Other:
- board text removed: "bei mouser bestellen"
Changed lines of the file:
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@@
     (tags "SOIC SO")
     (attr smd)
-    (fp_text reference "U11" (at 0 -6.1) (layer "F.SilkS")
+    (fp_text reference "U11" (at -1.720014 -6.089972) (layer "F.SilkS")
       (effects (font (size 1 1) (thickness 0.15)))
     )
@@
     (tags "LED diameter 5.0mm 2 pins")
     (attr through_hole)
-    (fp_text reference "D5" (at 1.27 -3.96 90) (layer "F.SilkS")
+    (fp_text reference "D5" (at 0.931 -4.019 90) (layer "F.SilkS")
       (effects (font (size 1 1) (thickness 0.15)))
     )
@@
   )
   (gr_line (start 0 79.3) (end 0 0) (layer "Edge.Cuts") (width 0.05))
+  (gr_line (start 0 0) (end 119 0) (layer "Edge.Cuts") (width 0.05))
   (gr_line (start 0 79.3) (end 119 79.3) (layer "Edge.Cuts") (width 0.05))
-  (gr_line (start 0 0) (end 119 0) (layer "Edge.Cuts") (width 0.05))
   (gr_line (start 119 0) (end 119 79.3) (layer "Edge.Cuts") (width 0.05))
-  (gr_text "bei mouser bestellen" (at 71.044986 41.020028) (layer "F.SilkS")
-    (effects (font (size 1 1) (thickness 0.15)))
-  )
   (gr_text "Kevin da Silva Fernandes 2020" (at 89.84 8.34) (layer "F.SilkS")
     (effects (font (size 1.5 1.5) (thickness 0.2)))
   )
-  (gr_text "bei mouser bestellen" (at 71.12 56.388) (layer "F.SilkS")
-    (effects (font (size 1 1) (thickness 0.15)))
-  )
   (gr_text "Register A / B" (at 90.348 4.276) (layer "F.SilkS")
