File: Hardware/CLUSTERFCK/CLK/CLK/CLK.kicad_sch (KiCad schematic)
At the start: 39 parts, among them J1 Conn_01x04_Male, J2 Conn_Coaxial, J3 Conn_01x02, J4 Conn_02x20_Counter_Clockwise, SW1 SW_Push, SW2 SW_SPDT, SW3 SW_SPDT, U1 74LS08, U2 74LS04, U3 NE555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

Commit message: 0045 | 6h | CLK module rev 3
Parts:
- R7: renamed from R?; footprint (none) -> Resistor_SMD:R_0805_2012Metric_Pad1.15x1.40mm_HandSolder
- U1, U2: footprint Package_DIP:DIP-14_W7.62mm_Socket -> Package_SO:SOIC-14_3.9x8.7mm_P1.27mm
- U6: footprint (none) -> Package_SO:SOIC-14_3.9x8.7mm_P1.27mm
- gave numbers to parts that had none: 1
