File: Hardware/CLUSTERFCK/CLK/CLK/CLK.kicad_pcb (KiCad board)
At the start: 2 copper layers, 142 x 60 mm, 41 parts, among them J1 Conn_01x04_Male, J2 Conn_Coaxial, J3 Conn_01x02, J4 Conn_02x20_Counter_Clockwise, SW1 SW_Push, SW2 SW_SPDT, SW3 SW_SPDT, SW4 SW_Push, U1 74LS08, U2 74LS04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

Commit message: 0066 | 6h | made holes in pcbs
Parts:
- added REF**: MountingHole_4.3mm_M4, MountingHole:MountingHole_4.3mm_M4, F.Cu at (113.3, 52.8)
- added REF**: MountingHole_4.3mm_M4, MountingHole:MountingHole_4.3mm_M4, F.Cu at (113.3, 98.7)
- added REF**: MountingHole_4.3mm_M4, MountingHole:MountingHole_4.3mm_M4, F.Cu at (221.5, 83.5)
Changed lines of the file:
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@@
     )
+  )
+  (footprint "MountingHole:MountingHole_4.3mm_M4" (layer "F.Cu")
+    (at 113.3 52.84)
+    (descr "Mounting Hole 4.3mm, no annular, M4")
+    (tags "mounting hole 4.3mm no annular m4")
+    (attr exclude_from_pos_files exclude_from_bom)
+    (fp_text reference "REF**" (at 0.05 -3.05) (layer "F.SilkS")
+      (effects (font (size 1 1) (thickness 0.15)))
+    )
+    (fp_text value "MountingHole_4.3mm_M4" (at 0 5.3) (layer "F.Fab")
+      (effects (font (size 1 1) (thickness 0.15)))
+    )
+    (fp_text user "${REFERENCE}" (at 0.3 0) (layer "F.Fab")
+      (effects (font (size 1 1) (thickness 0.15)))
+    )
+    (fp_circle (center 0 0) (end 4.3 0) (layer "Cmts.User") (width 0.15) (fill none))
+    (fp_circle (center 0 0) (end 4.55 0) (layer "F.CrtYd") (width 0.05) (fill none))
+    (pad "1" np_thru_hole circle (at 0 0) (size 4.3 4.3) (drill 4.3) (layers *.Cu *.Mask))
   )
   (footprint "LED_THT:LED_D5.0mm" (layer "F.Cu")
@@
     )
   )
+  (footprint "MountingHole:MountingHole_4.3mm_M4" (layer "F.Cu")
+    (at 113.3 98.66)
+    (descr "Mounting Hole 4.3mm, no annular, M4")
+    (tags "mounting hole 4.3mm no annular m4")
+    (attr exclude_from_pos_files exclude_from_bom)
+    (fp_text reference "REF**" (at 0.01 -3.09) (layer "F.SilkS")
+      (effects (font (size 1 1) (thickness 0.15)))
+    )
+    (fp_text value "MountingHole_4.3mm_M4" (at 0 5.3) (layer "F.Fab")
+      (effects (font (size 1 1) (thickness 0.15)))
+    )
+    (fp_text user "${REFERENCE}" (at 0.3 0) (layer "F.Fab")
+      (effects (font (size 1 1) (thickness 0.15)))
+    )
+    (fp_circle (center 0 0) (end 4.3 0) (layer "Cmts.User") (width 0.15) (fill none))
+    (fp_circle (center 0 0) (end 4.55 0) (layer "F.CrtYd") (width 0.05) (fill none))
+    (pad "1" np_thru_hole circle (at 0 0) (size 4.3 4.3) (drill 4.3) (layers *.Cu *.Mask))
+  )
   (footprint "Resistor_SMD:R_0805_2012Metric_Pad1.15x1.40mm_HandSolder" (layer "F.Cu")
     (at 96.925 86.375 90)
@@
     )
   )
+  (footprint "MountingHole:MountingHole_4.3mm_M4" (layer "F.Cu")
+    (at 221.54 83.5)
+    (descr "Mounting Hole 4.3mm, no annular, M4")
+    (tags "mounting hole 4.3mm no annular m4")
+    (attr exclude_from_pos_files exclude_from_bom)
+    (fp_text reference "REF**" (at 0.2 -3.23) (layer "F.SilkS")
+      (effects (font (size 1 1) (thickness 0.15)))
+    )
+    (fp_text value "MountingHole_4.3mm_M4" (at 0 5.3) (layer "F.Fab")
+      (effects (font (size 1 1) (thickness 0.15)))
+    )
+    (fp_text user "${REFERENCE}" (at 0.3 0) (layer "F.Fab")
+      (effects (font (size 1 1) (thickness 0.15)))
+    )
+    (fp_circle (center 0 0) (end 4.3 0) (layer "Cmts.User") (width 0.15) (fill none))
+    (fp_circle (center 0 0) (end 4.55 0) (layer "F.CrtYd") (width 0.05) (fill none))
+    (pad "1" np_thru_hole circle (at 0 0) (size 4.3 4.3) (drill 4.3) (layers *.Cu *.Mask))
+  )
   (footprint "Capacitor_SMD:C_0805_2012Metric_Pad1.15x1.40mm_HandSolder" (layer "F.Cu")
     (at 163.875 77.775 90)
@@
     (effects (font (size 4 4) (thickness 0.7)))
   )
-  (gr_text "50Ω" (at 118.55 54) (layer "F.SilkS")
+  (gr_text "50Ω" (at 121.23 57.72) (layer "F.SilkS")
     (effects (font (size 1 1) (thickness 0.15)))
   )

Commit message: 0072 | 3h | make silkscreen prettier
Routing:
- net +5V: track 297.6 -> 295.2 mm
Changed lines of the file:
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@@
     (property "Schaltplanname" "")
     (attr through_hole)
-    (fp_text reference "F1" (at 11.25 -6 90) (layer "F.SilkS")
+    (fp_text reference "F1" (at -1.02 3.54 180) (layer "F.SilkS")
       (effects (font (size 1 1) (thickness 0.15)))
     )
@@
     (property "Schaltplanname" "")
     (attr through_hole)
-    (fp_text reference "D274" (at 1.27 -3.96 90) (layer "F.SilkS")
+    (fp_text reference "D274" (at 1.285 4.975 180) (layer "F.SilkS")
       (effects (font (size 1 1) (thickness 0.15)))
     )
@@
     (property "Schaltplanname" "")
     (attr smd)
-    (fp_text reference "R287" (at 0 -1.65 90) (layer "F.SilkS")
+    (fp_text reference "R287" (at -0.075 -2.765 180) (layer "F.SilkS")
       (effects (font (size 1 1) (thickness 0.15)))
     )
@@
     (property "Schaltplanname" "")
     (attr through_hole)
-    (fp_text reference "J4" (at -2.445 -2.13) (layer "F.SilkS")
+    (fp_text reference "J4" (at -1.31 50.53) (layer "F.SilkS")
       (effects (font (size 1 1) (thickness 0.15)))
     )
@@
     (property "Schaltplanname" "")
     (attr smd)
-    (fp_text reference "C3" (at 2.275 0.1 180) (layer "F.SilkS")
+    (fp_text reference "C3" (at 2.465 -0.225 180) (layer "F.SilkS")
       (effects (font (size 1 1) (thickness 0.15)))
     )
@@
     (property "Schaltplanname" "")
     (attr smd)
-    (fp_text reference "C5" (at -0.025 1.425) (layer "F.SilkS")
+    (fp_text reference "C5" (at -0.045 1.595) (layer "F.SilkS")
       (effects (font (size 1 1) (thickness 0.15)))
     )
@@
     (property "Schaltplanname" "")
     (attr through_hole)
-    (fp_text reference "J3" (at 2.5 -4) (layer "F.SilkS")
+    (fp_text reference "J3" (at 2.89 3.52) (layer "F.SilkS")
       (effects (font (size 1 1) (thickness 0.15)))
     )
@@
     (property "Schaltplanname" "")
     (attr smd)
-    (fp_text reference "C17" (at 0.125 1.575) (layer "F.SilkS")
+    (fp_text reference "C17" (at 0.025 1.675) (layer "F.SilkS")
       (effects (font (size 1 1) (thickness 0.15)))
     )
@@
   (segment (start 139.2 66.4) (end 139.225 66.375) (width 0.2) (layer "F.Cu") (net 2))
   (segment (start 139.425 66.375) (end 139.525 66.375) (width 0.2) (layer "F.Cu") (net 2))
-  (segment (start 121.25 82.5) (end 121.25 78.475) (width 1) (layer "F.Cu") (net 2))
-  (segment (start 121.25 78.475) (end 121.55 78.175) (width 1) (layer "F.Cu") (net 2))
   (segment (start 155.48 56.585) (end 157.235 56.585) (width 1) (layer "F.Cu") (net 2))
   (segment (start 150.967821 74.94499) (end 150.76999 74.94499) (width 0.5) (layer "F.Cu") (net 2))
@@
   (segment (start 161.65 68.625) (end 161.655 68.63) (width 1) (layer "F.Cu") (net 2))
   (segment (start 151.56 78.815) (end 153 77.375) (width 0.5) (layer "F.Cu") (net 2))
+  (segment (start 121.25 78.71) (end 121.83 78.13) (width 1) (layer "F.Cu") (net 2))
   (segment (start 130.005 69.35) (end 129.815 69.54) (width 0.5) (layer "F.Cu") (net 2))
+  (segment (start 121.25 82.5) (end 121.25 78.71) (width 1) (layer "F.Cu") (net 2))
   (segment (start 135.2 59.05) (end 134.6875 59.5625) (width 0.5) (layer "F.Cu") (net 2))
   (segment (start 147.7 66.45) (end 145.7 64.45) (width 1) (layer "F.Cu") (net 2))
@@
   (segment (start 139.2 68.6) (end 139.2 66.6) (width 0.2) (layer "F.Cu") (net 2))
   (segment (start 151.52 78.815) (end 151.56 78.815) (width 0.5) (layer "F.Cu") (net 2))
+  (via (at 121.83 78.13) (size 0.8) (drill 0.4) (layers "F.Cu" "B.Cu") (net 2))
   (via (at 140.675 65.8) (size 0.43) (drill 0.3) (layers "F.Cu" "B.Cu") (net 2))
   (via (at 177.025 71.725) (size 0.8) (drill 0.5) (layers "F.Cu" "B.Cu") (net 2))
   (via (at 133.425 69.375) (size 0.43) (drill 0.3) (layers "F.Cu" "B.Cu") (net 2))
-  (via (at 121.55 78.175) (size 0.8) (drill 0.5) (layers "F.Cu" "B.Cu") (net 2))
   (via (at 131.15 69.35) (size 0.43) (drill 0.3) (layers "F.Cu" "B.Cu") (net 2))
   (via (at 179.025 71.675) (size 0.8) (drill 0.5) (layers "F.Cu" "B.Cu") (net 2))
-  (segment (start 121.55 78.175) (end 121.55 76.675) (width 1) (layer "B.Cu") (net 2))
   (segment (start 133.425 69.375) (end 131.175 69.375) (width 0.5) (layer "B.Cu") (net 2))
-  (segment (start 129.515 72.225) (end 123.45 72.225) (width 1) (layer "B.Cu") (net 2))
   (segment (start 131.175 69.375) (end 131.15 69.35) (width 0.5) (layer "B.Cu") (net 2))
+  (segment (start 125.19 72.18) (end 129.56 72.18) (width 1) (layer "B.Cu") (net 2))
   (segment (start 129.56 72.18) (end 129.515 72.225) (width 1) (layer "B.Cu") (net 2))
-  (segment (start 123.45 72.225) (end 121.55 74.125) (width 1) (layer "B.Cu") (net 2))
   (segment (start 140.675 65.8) (end 141.34 65.8) (width 0.2) (layer "B.Cu") (net 2))
+  (segment (start 121.83 78.13) (end 121.83 75.54) (width 1) (layer "B.Cu") (net 2))
   (segment (start 141.34 65.8) (end 143.17 63.97) (width 0.2) (layer "B.Cu") (net 2))
+  (segment (start 121.83 75.54) (end 125.19 72.18) (width 1) (layer "B.Cu") (net 2))
   (segment (start 178.975 71.725) (end 179.025 71.675) (width 1) (layer "B.Cu") (net 2))
   (segment (start 177.025 71.725) (end 178.975 71.725) (width 1) (layer "B.Cu") (net 2))
-  (segment (start 121.55 74.125) (end 121.55 78.175) (width 1) (layer "B.Cu") (net 2))
   (segment (start 163.875 78.8) (end 161.695 78.8) (width 0.5) (layer "F.Cu") (net 3))
   (segment (start 161.695 78.8) (end 161.68 78.815) (width 0.5) (layer "F.Cu") (net 3))
