File: Hardware/CLUSTERFCK/PO/PO/PO.kicad_sch (KiCad schematic)
At the start: 2 parts, among them J1 Conn_02x08_Counter_Clockwise, J2 Conn_02x20_Counter_Clockwise

Commit message: 0061|1h|PO Module Versuch 2
Parts:
- removed J1: Conn_02x08_Counter_Clockwise, Connector_PinHeader_2.54mm:PinHeader_2x08_P2.54mm_Vertical_SMD, symbol Connector_Generic:Conn_02x08_Counter_Clockwise
- added J1: Conn_02x14_Counter_Clockwise, Connector_PinHeader_2.54mm:PinHeader_2x14_P2.54mm_Horizontal, symbol Connector_Generic:Conn_02x14_Counter_Clockwise
Connections:
- net +5V: now also J1.14 (Pin_14)
- net ADDR0: now also J2.34 (Pin_34), J1.1 (Pin_1); no longer J2.23 (Pin_23)
- net ADDR1: now also J2.33 (Pin_33), J1.2 (Pin_2); no longer J2.24 (Pin_24)
- net ADDR10: now also J2.24 (Pin_24), J1.11 (Pin_11); no longer J2.33 (Pin_33)
- net ADDR11: now also J2.23 (Pin_23), J1.12 (Pin_12); no longer J2.34 (Pin_34)
- net ADDR2: now also J2.32 (Pin_32), J1.3 (Pin_3); no longer J2.25 (Pin_25)
- net ADDR3: now also J2.31 (Pin_31), J1.4 (Pin_4); no longer J2.26 (Pin_26)
- net ADDR4: now also J2.30 (Pin_30), J1.5 (Pin_5); no longer J2.27 (Pin_27)
- net ADDR5: now also J2.29 (Pin_29), J1.6 (Pin_6); no longer J2.28 (Pin_28)
- net ADDR6: now also J2.28 (Pin_28), J1.7 (Pin_7); no longer J2.29 (Pin_29)
- net ADDR7: now also J2.27 (Pin_27), J1.8 (Pin_8); no longer J2.30 (Pin_30)
- net ADDR8: now also J2.26 (Pin_26), J1.9 (Pin_9); no longer J2.31 (Pin_31)
- net ADDR9: now also J2.25 (Pin_25), J1.10 (Pin_10); no longer J2.32 (Pin_32)
- net CLK: now also J1.16 (Pin_16)
- net DATA0: now also J1.17 (Pin_17)
- net DATA1: now also J1.18 (Pin_18)
- net DATA2: now also J1.19 (Pin_19)
- net DATA3: now also J1.20 (Pin_20)
- net DATA4: now also J1.21 (Pin_21)
- net DATA5: now also J1.22 (Pin_22)
- net DATA6: now also J1.23 (Pin_23)
- net DATA7: now also J1.24 (Pin_24)
- net EXT0: now also J1.25 (Pin_25)
- net EXT1: now also J1.26 (Pin_26)
- net EXT2: now also J1.27 (Pin_27)
- net GND: now also J1.15 (Pin_15)
- net HLT: now also J1.13 (Pin_13)
- net IRPT: now also J1.28 (Pin_28)

Commit message: 0062 | 0 | review PO 2
Parts:
- J1: footprint Connector_PinHeader_2.54mm:PinHeader_2x14_P2.54mm_Horizontal -> Connector_PinHeader_2.54mm:PinHeader_2x14_P2.54mm_Vertical
Changed lines of the file:
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@@
     (comment 1 "Kevin da Silva Fernandes")
   )
-  (no_connect (at 68.199 98.552))
-  (no_connect (at 65.659 98.552))
-  (no_connect (at 70.739 98.552))
   (no_connect (at 101.219 111.252))
   (no_connect (at 98.679 111.252))
+  (no_connect (at 70.739 98.552))
+  (no_connect (at 65.659 98.552))
   (no_connect (at 63.119 98.552))
+  (no_connect (at 68.199 98.552))
   (bus_entry (at 63.119 117.602) (size 2.54 2.54)
     (stroke (width 0.1524) (type solid) (color 0 0 0 0))
@@
       (effects (font (size 1.27 1.27)) (justify left))
     )
-    (property "Footprint" "Connector_PinHeader_2.54mm:PinHeader_2x14_P2.54mm_Horizontal" (id 2) (at 181.61 105.41 0)
+    (property "Footprint" "Connector_PinHeader_2.54mm:PinHeader_2x14_P2.54mm_Vertical" (id 2) (at 181.61 105.41 0)
       (effects (font (size 1.27 1.27)) hide)
     )
@@
     )
     (path "/478c227d-7dd5-442a-91bb-663adcbaad62"
-      (reference "J1") (unit 1) (value "Conn_02x14_Counter_Clockwise") (footprint "Connector_PinHeader_2.54mm:PinHeader_2x14_P2.54mm_Horizontal")
+      (reference "J1") (unit 1) (value "Conn_02x14_Counter_Clockwise") (footprint "Connector_PinHeader_2.54mm:PinHeader_2x14_P2.54mm_Vertical")
     )
     (path "/5a640586-e2ea-43fa-9dc4-1e50b50ad4de"
