File: Hardware/CLUSTERFCK/JUMPER/JUMPER/JUMPER.kicad_sch (KiCad schematic)
At the start: 2 parts, among them J1 Conn_02x20_Counter_Clockwise, J2 Conn_02x20_Counter_Clockwise

Commit message: 0065 | 24h | ADDR & DATA & PLACEHOLDER etc
Connections:
- net DATA0: now reaches J1.31 (Pin_31)
- net DATA0: now also J2.10 (Pin_10)
- net DATA1: now reaches J1.32 (Pin_32)
- net DATA1: now also J2.9 (Pin_9)
- net DATA2: now reaches J1.33 (Pin_33)
- net DATA2: now also J2.8 (Pin_8)
- net DATA3: now reaches J1.34 (Pin_34)
- net DATA3: now also J2.7 (Pin_7)
- net DATA4: now reaches J1.35 (Pin_35)
- net DATA4: now also J2.6 (Pin_6)
- net DATA5: now reaches J1.36 (Pin_36)
- net DATA5: now also J2.5 (Pin_5)
- net DATA6: now reaches J1.37 (Pin_37)
- net DATA6: now also J2.4 (Pin_4)
- net DATA7: now reaches J1.38 (Pin_38)
- net DATA7: now also J2.3 (Pin_3)
- net carry renamed CARRY
- net zero renamed ZERO
- no-connect marks 18 -> 2
Other:
- moved on the sheet: J1, J2
