File: Hardware/CLUSTERFCK/MIM/MIM/MIM.kicad_pcb (KiCad board)
At the start: 2 copper layers, 142.1 x 108 mm, 22 parts, among them J1 Conn_02x20_Counter_Clockwise, J2 Conn_02x20_Counter_Clockwise, U1 74LS00, U10 74LS245, U2 INTEL2716, U3 INTEL2716, U4 74LS161, U5 INTEL2716, U6 74LS245, U7 74LS245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

Commit message: 0039 | 0,5h | review MIM
Routing:
- net GND: track 303.2 -> 375.6 mm, vias 43 -> 67
- net (no net): track 0.00 -> 0.80 mm
Other:
- board text added: "Kevin da Silva Fernandes 2020"
- board text added: "Micro Instrucion Manager"
Changed lines of the file:
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@@
   (general
     (thickness 1.6)
-    (drawings 6)
-    (tracks 898)
+    (drawings 8)
+    (tracks 939)
     (modules 22)
     (nets 85)
@@
       (dielectric_constraints no)
     )
-    (last_trace_width 1)
+    (last_trace_width 0.2)
     (user_trace_width 0.2)
     (user_trace_width 0.5)
@@
     )
   )
+  (gr_text "Micro Instrucion Manager" (at 149.97 38.76) (layer "F.SilkS")
+    (effects (font (size 3 3) (thickness 0.7)))
+  )
+  (gr_text "Kevin da Silva Fernandes 2020\n" (at 143.11 139.45) (layer "F.SilkS")
+    (effects (font (size 2 2) (thickness 0.3)))
+  )
   (gr_line (start 256.54 142.24) (end 258.92 142.24) (layer "Edge.Cuts") (width 0.05))
   (gr_line (start 256.54 34.29) (end 258.92 34.29) (layer "Edge.Cuts") (width 0.05))
@@
   (gr_line (start 258.92 34.29) (end 258.92 142.24) (layer "Edge.Cuts") (width 0.05))
   (gr_line (start 256.54 34.29) (end 116.84 34.29) (layer "Edge.Cuts") (width 0.05))
+  (via (at 137.25 49.9) (size 0.45) (drill 0.3) (layers "F.Cu" "B.Cu") (net 1))
+  (via (at 135 71.75) (size 0.45) (drill 0.3) (layers "F.Cu" "B.Cu") (net 1))
+  (via (at 150.79 72.09) (size 0.45) (drill 0.3) (layers "F.Cu" "B.Cu") (net 1))
+  (via (at 164.79 73.17) (size 0.45) (drill 0.3) (layers "F.Cu" "B.Cu") (net 1))
+  (via (at 224.31 107.21) (size 0.45) (drill 0.3) (layers "F.Cu" "B.Cu") (net 1))
+  (via (at 220.45 107.44) (size 0.45) (drill 0.3) (layers "F.Cu" "B.Cu") (net 1))
+  (via (at 186.64 106.87) (size 0.45) (drill 0.3) (layers "F.Cu" "B.Cu") (net 1))
+  (via (at 206.1 107.06) (size 0.45) (drill 0.3) (layers "F.Cu" "B.Cu") (net 1))
+  (via (at 167.74 107.18) (size 0.45) (drill 0.3) (layers "F.Cu" "B.Cu") (net 1))
+  (via (at 150.92 107.42) (size 0.45) (drill 0.3) (layers "F.Cu" "B.Cu") (net 1))
+  (via (at 249.78 136.83) (size 0.45) (drill 0.3) (layers "F.Cu" "B.Cu") (net 1))
+  (via (at 255.54 129.6) (size 0.45) (drill 0.3) (layers "F.Cu" "B.Cu") (net 1))
+  (via (at 256.97 106.61) (size 0.45) (drill 0.3) (layers "F.Cu" "B.Cu") (net 1))
+  (via (at 253.94 88.31) (size 0.45) (drill 0.3) (layers "F.Cu" "B.Cu") (net 1))
+  (via (at 255.48 80.03) (size 0.45) (drill 0.3) (layers "F.Cu" "B.Cu") (net 1))
+  (via (at 255.38 64.79) (size 0.45) (drill 0.3) (layers "F.Cu" "B.Cu") (net 1))
+  (via (at 255.36 49.49) (size 0.45) (drill 0.3) (layers "F.Cu" "B.Cu") (net 1))
+  (via (at 255.7 36.56) (size 0.45) (drill 0.3) (layers "F.Cu" "B.Cu") (net 1))
+  (segment (start 249.41 56.94) (end 247.62 55.15) (width 0.2) (layer "F.Cu") (net 1))
+  (segment (start 232.50001 36.09001) (end 227.65999 36.09001) (width 0.2) (layer "F.Cu") (net 1))
+  (segment (start 243.7 51.23) (end 243.7 47.29) (width 0.2) (layer "F.Cu") (net 1))
+  (via (at 227.37 36.46) (size 0.45) (drill 0.3) (layers "F.Cu" "B.Cu") (net 1))
+  (segment (start 227.65999 36.09001) (end 227.37 36.38) (width 0.2) (layer "F.Cu") (net 1))
+  (segment (start 227.37 36.38) (end 227.37 36.46) (width 0.2) (layer "F.Cu") (net 1))
+  (segment (start 243.7 47.29) (end 232.50001 36.09001) (width 0.2) (layer "F.Cu") (net 1))
+  (segment (start 249.41 58.18) (end 249.41 56.94) (width 0.2) (layer "F.Cu") (net 1))
+  (segment (start 247.62 55.15) (end 243.7 51.23) (width 0.2) (layer "F.Cu") (net 1))
+  (segment (start 244.500009 46.944311) (end 232.785698 35.23) (width 0.2) (layer "F.Cu") (net 1))
+  (segment (start 224.71601 35.23) (end 223.56601 36.38) (width 0.2) (layer "F.Cu") (net 1))
+  (segment (start 248.325698 54.72) (end 244.50001 50.894312) (width 0.2) (layer "F.Cu") (net 1))
+  (segment (start 244.50001 50.894312) (end 244.500009 46.944311) (width 0.2) (layer "F.Cu") (net 1))
+  (segment (start 249.62 54.72) (end 248.325698 54.72) (width 0.2) (layer "F.Cu") (net 1))
+  (segment (start 223.56601 36.38) (end 223.56601 37.42399) (width 0.2) (layer "F.Cu") (net 1))
+  (segment (start 232.785698 35.23) (end 224.71601 35.23) (width 0.2) (layer "F.Cu") (net 1))
+  (segment (start 223.56601 37.42399) (end 223.519999 37.470001) (width 0.2) (layer "F.Cu") (net 1))
+  (segment (start 224.084956 35.26) (end 223.52 35.824956) (width 0.25) (layer "F.Cu") (net 0))
+  (via (at 249.88 56.16) (size 0.45) (drill 0.3) (layers "F.Cu" "B.Cu") (net 1))
+  (via (at 242.22 42.16) (size 0.45) (drill 0.3) (layers "F.Cu" "B.Cu") (net 1))
+  (via (at 238.18 43.7) (size 0.45) (drill 0.3) (layers "F.Cu" "B.Cu") (net 1))
+  (via (at 249.62 54.72) (size 0.45) (drill 0.3) (layers "F.Cu" "B.Cu") (net 1))
+  (via (at 249.41 58.18) (size 0.45) (drill 0.3) (layers "F.Cu" "B.Cu") (net 1))
   (segment (start 213.36 66.04) (end 195.0275 66.04) (width 1) (layer "F.Cu") (net 2))
   (segment (start 217.17 69.85) (end 213.36 66.04) (width 1) (layer "F.Cu") (net 2))

Commit message: 0065 | 24h | ADDR & DATA & PLACEHOLDER etc
Routing:
- net (no net): track 0.80 -> 0.00 mm
Other:
- net class Default removed

Commit message: 0066 | 6h | made holes in pcbs
Parts:
- added REF**: MountingHole_4.3mm_M4, MountingHole:MountingHole_4.3mm_M4, F.Cu at (241.4, 103.6)
- added REF**: MountingHole_4.3mm_M4, MountingHole:MountingHole_4.3mm_M4, F.Cu at (122.1, 136.9)
- added REF**: MountingHole_4.3mm_M4, MountingHole:MountingHole_4.3mm_M4, F.Cu at (234.3, 85.0)
- added REF**: MountingHole_4.3mm_M4, MountingHole:MountingHole_4.3mm_M4, F.Cu at (122.2, 39.6)
