File: Hardware/CLUSTERFCK/GFX/GFX/GFX.kicad_sch (KiCad schematic)
At the start: 320 parts

Commit message: 29 | 22h | Layoutet GFX Module
Parts:
- removed U? (x23): 74LS08, symbol 74xx:74LS08
- added J1, J2: Conn_02x20_Counter_Clockwise, Connector_PinSocket_2.54mm:PinSocket_2x20_P2.54mm_Horizontal, symbol Connector_Generic:Conn_02x20_Counter_Clockwise
- added unit 2 of U1
- added unit 3 of U1
- added unit 4 of U1
- added U10, U13, U14, U15: 74LS08, symbol 74xx:74LS08
- C1, C10, C11, C12, C13, C14, C15, C16, C17, C18, C19, C2, C20, C21, C22, C3, C4, C5, C6, C7, C8, C9: renamed from C?; footprint (none) -> Capacitor_SMD:C_0805_2012Metric_Pad1.15x1.40mm_HandSolder
- D1, D10, D100, D101, D102, D103, D104, D105, D106, D107, D108, D109, D11, D110, D111, D112, D113, D114, D115, D116, D117, D118, D119, D12, D120, D121, D122, D123, D124, D125, D126, D127, D128, D13, D14, D15, D16, D17, D18, D19, D2, D20, D21, D22, D23, D24, D25, D26, D27, D28, D29, D3, D30, D31, D32, D33, D34, D35, D36, D37, D38, D39, D4, D40, D41, D42, D43, D44, D45, D46, D47, D48, D49, D5, D50, D51, D52, D53, D54, D55, D56, D57, D58, D59, D6, D60, D61, D62, D63, D64, D65, D66, D67, D68, D69, D7, D70, D71, D72, D73, D74, D75, D76, D77, D78, D79, D8, D80, D81, D82, D83, D84, D85, D86, D87, D88, D89, D9, D90, D91, D92, D93, D94, D95, D96, D97, D98, D99: renamed from D?; footprint (none) -> LED_THT:LED_D5.0mm
- R1, R10, R100, R101, R102, R103, R104, R105, R106, R107, R108, R109, R11, R110, R111, R112, R113, R114, R115, R116, R117, R118, R119, R12, R120, R121, R122, R123, R124, R125, R126, R127, R128, R13, R14, R15, R16, R17, R18, R19, R2, R20, R21, R22, R23, R24, R25, R26, R27, R28, R29, R3, R30, R31, R32, R33, R34, R35, R36, R37, R38, R39, R4, R40, R41, R42, R43, R44, R45, R46, R47, R48, R49, R5, R50, R51, R52, R53, R54, R55, R56, R57, R58, R59, R6, R60, R61, R62, R63, R64, R65, R66, R67, R68, R69, R7, R70, R71, R72, R73, R74, R75, R76, R77, R78, R79, R8, R80, R81, R82, R83, R84, R85, R86, R87, R88, R89, R9, R90, R91, R92, R93, R94, R95, R96, R97, R98, R99: renamed from R?; footprint (none) -> Resistor_SMD:R_0805_2012Metric_Pad1.15x1.40mm_HandSolder
- U1: renamed from U?; footprint (none) -> Package_SO:SOIC-14_3.9x8.7mm_P1.27mm
- U11, U12, U18, U19, U2, U24, U25, U3, U31, U32, U34, U35, U36, U37, U7, U8: renamed from U?; footprint (none) -> Package_SO:SOIC-20W_7.5x12.8mm_P1.27mm
- U21: renamed from U?; footprint (none) -> Package_SO:SOIC-24W_7.5x15.4mm_P1.27mm
Connections:
- net +5V: now also J1.21 (Pin_21), J1.22 (Pin_22), J1.39 (Pin_39), J1.40 (Pin_40), J2.21 (Pin_21), J2.22 (Pin_22), J2.39 (Pin_39), J2.40 (Pin_40), U10.14 (VCC), U13.14 (VCC), U14.14 (VCC), U15.14 (VCC)
- net CLK: now also J1.16 (Pin_16), J2.16 (Pin_16)
- net GFX0: now also J1.11 (Pin_11), J2.11 (Pin_11)
- net GFX1: now also J1.12 (Pin_12), J2.12 (Pin_12)
- net GFX2: now also J1.13 (Pin_13), J2.13 (Pin_13)
- net GFX3: now also J1.14 (Pin_14), J2.14 (Pin_14)
- net GFXC0: now also U10.3
- net GFXC1: now also U10.6
- net GFXC10: now also U14.8
- net GFXC11: now also U14.11
- net GFXC12: now also U15.3
- net GFXC13: now also U15.6
- net GFXC14: now also U15.8
- net GFXC15: now also U15.11
- net GFXC2: now also U10.8
- net GFXC3: now also U10.11
- net GFXC4: now also U13.3
- net GFXC5: now also U13.6
- net GFXC6: now also U13.8
- net GFXC7: now also U13.11
- net GFXC8: now also U14.3
- net GFXC9: now also U14.6
- net GFXCLK: now also U10.1, U10.12, U10.4, U10.9, U13.1, U13.12, U13.4, U13.9, U14.1, U14.12, U14.4, U14.9, U15.1, U15.12, U15.4, U15.9
- net GFXI: now also J1.15 (Pin_15), J2.15 (Pin_15)
- net GND: now also J1.1 (Pin_1), J1.19 (Pin_19), J1.2 (Pin_2), J1.20 (Pin_20), J2.1 (Pin_1), J2.19 (Pin_19), J2.2 (Pin_2), J2.20 (Pin_20), U1.10, U1.12, U1.13, U1.4, U1.5, U1.9, U10.7 (GND), U13.7 (GND), U14.7 (GND), U15.7 (GND)
- net at U21.11 (S0): now also U10.2
- net at U21.9 (S1): now also U10.5
- net at U21.10 (S2): now also U10.10
- net at U21.8 (S3): now also U10.13
- net at U21.7 (S4): now also U13.2
- net at U21.6 (S5): now also U13.5
- net at U21.5 (S6): now also U13.10
- net at U21.4 (S7): now also U13.13
- net D0: now reaches U31.2 (D0)
- net D0: now also U11.2 (D0), U12.2 (D0), U18.2 (D0), U19.2 (D0), U2.2 (D0), U24.2 (D0), U25.2 (D0), U3.2 (D0), U32.2 (D0), U34.2 (D0), U35.2 (D0), U36.2 (D0), U37.2 (D0), U7.2 (D0), U8.2 (D0), J1.3 (Pin_3)
- net D1: now reaches U31.3 (D1)
- net D1: now also U11.3 (D1), U12.3 (D1), U18.3 (D1), U19.3 (D1), U2.3 (D1), U24.3 (D1), U25.3 (D1), U3.3 (D1), U32.3 (D1), U34.3 (D1), U35.3 (D1), U36.3 (D1), U37.3 (D1), U7.3 (D1), U8.3 (D1), J1.4 (Pin_4)
- net D2: now reaches U31.4 (D2)
- net D2: now also U11.4 (D2), U12.4 (D2), U18.4 (D2), U19.4 (D2), U2.4 (D2), U24.4 (D2), U25.4 (D2), U3.4 (D2), U32.4 (D2), U34.4 (D2), U35.4 (D2), U36.4 (D2), U37.4 (D2), U7.4 (D2), U8.4 (D2), J1.5 (Pin_5)
- net D3: now reaches U31.5 (D3)
- net D3: now also U11.5 (D3), U12.5 (D3), U18.5 (D3), U19.5 (D3), U2.5 (D3), U24.5 (D3), U25.5 (D3), U3.5 (D3), U32.5 (D3), U34.5 (D3), U35.5 (D3), U36.5 (D3), U37.5 (D3), U7.5 (D3), U8.5 (D3), J1.6 (Pin_6)
- net D4: now reaches U31.6 (D4)
- net D4: now also U11.6 (D4), U12.6 (D4), U18.6 (D4), U19.6 (D4), U2.6 (D4), U24.6 (D4), U25.6 (D4), U3.6 (D4), U32.6 (D4), U34.6 (D4), U35.6 (D4), U36.6 (D4), U37.6 (D4), U7.6 (D4), U8.6 (D4), J1.7 (Pin_7)
- net D5: now reaches U31.7 (D5)
- net D5: now also U11.7 (D5), U12.7 (D5), U18.7 (D5), U19.7 (D5), U2.7 (D5), U24.7 (D5), U25.7 (D5), U3.7 (D5), U32.7 (D5), U34.7 (D5), U35.7 (D5), U36.7 (D5), U37.7 (D5), U7.7 (D5), U8.7 (D5), J1.8 (Pin_8)
- net D6: now reaches U31.8 (D6)
- net D6: now also U11.8 (D6), U12.8 (D6), U18.8 (D6), U19.8 (D6), U2.8 (D6), U24.8 (D6), U25.8 (D6), U3.8 (D6), U32.8 (D6), U34.8 (D6), U35.8 (D6), U36.8 (D6), U37.8 (D6), U7.8 (D6), U8.8 (D6), J1.9 (Pin_9)
- net D7: now reaches U31.9 (D7)
- net D7: now also U11.9 (D7), U12.9 (D7), U18.9 (D7), U19.9 (D7), U2.9 (D7), U24.9 (D7), U25.9 (D7), U3.9 (D7), U32.9 (D7), U34.9 (D7), U35.9 (D7), U36.9 (D7), U37.9 (D7), U7.9 (D7), U8.9 (D7), J1.10 (Pin_10)
- net at U21.13 (S13): now also U15.5
- net at U21.14 (S12): now also U15.2
- net at U21.15 (S15): now also U15.13
- net at U21.16 (S14): now also U15.10
- net at U21.17 (S9): now also U14.5
- net at U21.18 (S8): now also U14.2
- net at U21.19 (S11): now also U14.13
- net at U21.20 (S10): now also U14.10
- no-connect marks 3 -> 46
Other:
- note added: "To ADDR BUS"
- note added: "To DATA BUS"

Commit message: unstable switching device push
Connections:
- net GFX0: now also J2.10 (Pin_10); no longer J2.11 (Pin_11)
Other:
- moved on the sheet: J2

Commit message: 0060 | 2h | 2nd review GFX
Parts:
- U1, U10, U13, U14, U15: footprint (none) -> Package_SO:SOIC-14_3.9x8.7mm_P1.27mm
