File: Hardware/CLUSTERFCK/PLACEHOLDER_L/PLACEHOLDER_L/PLACEHOLDER_L.kicad_pcb (KiCad board)
At the start: 2 copper layers, 142.1 x 237.9 mm, 2 parts, among them J1 Conn_02x20_Counter_Clockwise, J2 Conn_02x20_Counter_Clockwise

Commit message: 0066 | 6h | made holes in pcbs
Parts:
- added REF**: MountingHole_4.3mm_M4, MountingHole:MountingHole_4.3mm_M4, F.Cu at (5.39, 5.42)
- added REF**: MountingHole_4.3mm_M4, MountingHole:MountingHole_4.3mm_M4, F.Cu at (5.39, 232.9)
- added REF**: MountingHole_4.3mm_M4, MountingHole:MountingHole_4.3mm_M4, F.Cu at (136.7, 231.9)
- added REF**: MountingHole_4.3mm_M4, MountingHole:MountingHole_4.3mm_M4, F.Cu at (136.4, 119.3)
- added REF**: MountingHole_4.3mm_M4, MountingHole:MountingHole_4.3mm_M4, F.Cu at (5.39, 119.2)
- added REF**: MountingHole_4.3mm_M4, MountingHole:MountingHole_4.3mm_M4, F.Cu at (130.1, 4.96)
Changed lines of the file:
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@@
     )
+  )
+  (footprint "MountingHole:MountingHole_4.3mm_M4" (layer "F.Cu")
+    (at 5.39 5.42)
+    (descr "Mounting Hole 4.3mm, no annular, M4")
+    (tags "mounting hole 4.3mm no annular m4")
+    (attr exclude_from_pos_files exclude_from_bom)
+    (fp_text reference "REF**" (at -0.18 -2.99) (layer "F.SilkS")
+      (effects (font (size 1 1) (thickness 0.15)))
+    )
+    (fp_text value "MountingHole_4.3mm_M4" (at 0 5.3) (layer "F.Fab")
+      (effects (font (size 1 1) (thickness 0.15)))
+    )
+    (fp_text user "${REFERENCE}" (at 0.3 0) (layer "F.Fab")
+      (effects (font (size 1 1) (thickness 0.15)))
+    )
+    (fp_circle (center 0 0) (end 4.3 0) (layer "Cmts.User") (width 0.15) (fill none))
+    (fp_circle (center 0 0) (end 4.55 0) (layer "F.CrtYd") (width 0.05) (fill none))
+    (pad "1" np_thru_hole circle (at 0 0) (size 4.3 4.3) (drill 4.3) (layers *.Cu *.Mask))
+  )
+  (footprint "MountingHole:MountingHole_4.3mm_M4" (layer "F.Cu")
+    (at 5.39 232.92)
+    (descr "Mounting Hole 4.3mm, no annular, M4")
+    (tags "mounting hole 4.3mm no annular m4")
+    (attr exclude_from_pos_files exclude_from_bom)
+    (fp_text reference "REF**" (at 0.095 -3.05) (layer "F.SilkS")
+      (effects (font (size 1 1) (thickness 0.15)))
+    )
+    (fp_text value "MountingHole_4.3mm_M4" (at 0 5.3) (layer "F.Fab")
+      (effects (font (size 1 1) (thickness 0.15)))
+    )
+    (fp_text user "${REFERENCE}" (at 0.3 0) (layer "F.Fab")
+      (effects (font (size 1 1) (thickness 0.15)))
+    )
+    (fp_circle (center 0 0) (end 4.3 0) (layer "Cmts.User") (width 0.15) (fill none))
+    (fp_circle (center 0 0) (end 4.55 0) (layer "F.CrtYd") (width 0.05) (fill none))
+    (pad "1" np_thru_hole circle (at 0 0) (size 4.3 4.3) (drill 4.3) (layers *.Cu *.Mask))
   )
   (footprint "Connector_PinHeader_2.54mm:PinHeader_2x20_P2.54mm_Horizontal" (layer "F.Cu")
@@
     )
   )
+  (footprint "MountingHole:MountingHole_4.3mm_M4" (layer "F.Cu")
+    (at 136.74 231.87)
+    (descr "Mounting Hole 4.3mm, no annular, M4")
+    (tags "mounting hole 4.3mm no annular m4")
+    (attr exclude_from_pos_files exclude_from_bom)
+    (fp_text reference "REF**" (at 0.3 -2.94) (layer "F.SilkS")
+      (effects (font (size 1 1) (thickness 0.15)))
+    )
+    (fp_text value "MountingHole_4.3mm_M4" (at 0 5.3) (layer "F.Fab")
+      (effects (font (size 1 1) (thickness 0.15)))
+    )
+    (fp_text user "${REFERENCE}" (at 0.3 0) (layer "F.Fab")
+      (effects (font (size 1 1) (thickness 0.15)))
+    )
+    (fp_circle (center 0 0) (end 4.3 0) (layer "Cmts.User") (width 0.15) (fill none))
+    (fp_circle (center 0 0) (end 4.55 0) (layer "F.CrtYd") (width 0.05) (fill none))
+    (pad "1" np_thru_hole circle (at 0 0) (size 4.3 4.3) (drill 4.3) (layers *.Cu *.Mask))
+  )
+  (footprint "MountingHole:MountingHole_4.3mm_M4" (layer "F.Cu")
+    (at 136.45 119.27)
+    (descr "Mounting Hole 4.3mm, no annular, M4")
+    (tags "mounting hole 4.3mm no annular m4")
+    (attr exclude_from_pos_files exclude_from_bom)
+    (fp_text reference "REF**" (at 0.15 -3.02) (layer "F.SilkS")
+      (effects (font (size 1 1) (thickness 0.15)))
+    )
+    (fp_text value "MountingHole_4.3mm_M4" (at 0 5.3) (layer "F.Fab")
+      (effects (font (size 1 1) (thickness 0.15)))
+    )
+    (fp_text user "${REFERENCE}" (at 0.3 0) (layer "F.Fab")
+      (effects (font (size 1 1) (thickness 0.15)))
+    )
+    (fp_circle (center 0 0) (end 4.3 0) (layer "Cmts.User") (width 0.15) (fill none))
+    (fp_circle (center 0 0) (end 4.55 0) (layer "F.CrtYd") (width 0.05) (fill none))
+    (pad "1" np_thru_hole circle (at 0 0) (size 4.3 4.3) (drill 4.3) (layers *.Cu *.Mask))
+  )
+  (footprint "MountingHole:MountingHole_4.3mm_M4" (layer "F.Cu")
+    (at 5.39 119.17)
+    (descr "Mounting Hole 4.3mm, no annular, M4")
+    (tags "mounting hole 4.3mm no annular m4")
+    (attr exclude_from_pos_files exclude_from_bom)
+    (fp_text reference "REF**" (at -0.14 -3.02) (layer "F.SilkS")
+      (effects (font (size 1 1) (thickness 0.15)))
+    )
+    (fp_text value "MountingHole_4.3mm_M4" (at 0 5.3) (layer "F.Fab")
+      (effects (font (size 1 1) (thickness 0.15)))
+    )
+    (fp_text user "${REFERENCE}" (at 0.3 0) (layer "F.Fab")
+      (effects (font (size 1 1) (thickness 0.15)))
+    )
+    (fp_circle (center 0 0) (end 4.3 0) (layer "Cmts.User") (width 0.15) (fill none))
+    (fp_circle (center 0 0) (end 4.55 0) (layer "F.CrtYd") (width 0.05) (fill none))
+    (pad "1" np_thru_hole circle (at 0 0) (size 4.3 4.3) (drill 4.3) (layers *.Cu *.Mask))
+  )
+  (footprint "MountingHole:MountingHole_4.3mm_M4" (layer "F.Cu")
+    (at 130.11 4.96)
+    (descr "Mounting Hole 4.3mm, no annular, M4")
+    (tags "mounting hole 4.3mm no annular m4")
+    (attr exclude_from_pos_files exclude_from_bom)
+    (fp_text reference "REF**" (at 0.14 -2.91) (layer "F.SilkS")
+      (effects (font (size 1 1) (thickness 0.15)))
+    )
+    (fp_text value "MountingHole_4.3mm_M4" (at 0 5.3) (layer "F.Fab")
+      (effects (font (size 1 1) (thickness 0.15)))
+    )
+    (fp_text user "${REFERENCE}" (at 0.3 0) (layer "F.Fab")
+      (effects (font (size 1 1) (thickness 0.15)))
+    )
+    (fp_circle (center 0 0) (end 4.3 0) (layer "Cmts.User") (width 0.15) (fill none))
+    (fp_circle (center 0 0) (end 4.55 0) (layer "F.CrtYd") (width 0.05) (fill none))
+    (pad "1" np_thru_hole circle (at 0 0) (size 4.3 4.3) (drill 4.3) (layers *.Cu *.Mask))
+  )
   (gr_line (start 0 237.91) (end 142.08 237.91) (layer "Edge.Cuts") (width 0.1))
