File: Hardware/CLUSTERFCK/PLACEHOLDER_R/PLACEHOLDER_R/PLACEHOLDER_R.kicad_pcb (KiCad board)
At the start: 2 copper layers, 119 x 142.1 mm, 1 part, among them J1 Conn_02x20_Counter_Clockwise

Commit message: 0066 | 6h | made holes in pcbs
Parts:
- added REF**: MountingHole_4.3mm_M4, MountingHole:MountingHole_4.3mm_M4, F.Cu at (5.83, 4.96)
- added REF**: MountingHole_4.3mm_M4, MountingHole:MountingHole_4.3mm_M4, F.Cu at (112.4, 136.1)
- added REF**: MountingHole_4.3mm_M4, MountingHole:MountingHole_4.3mm_M4, F.Cu at (5.83, 136.1)
- added REF**: MountingHole_4.3mm_M4, MountingHole:MountingHole_4.3mm_M4, F.Cu at (112.4, 4.96)
Changed lines of the file:
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@@
   (net 39 "no_connect_12")
   (net 40 "no_connect_1")
+  (footprint "MountingHole:MountingHole_4.3mm_M4" (layer "F.Cu")
+    (at 5.83 4.96)
+    (descr "Mounting Hole 4.3mm, no annular, M4")
+    (tags "mounting hole 4.3mm no annular m4")
+    (attr exclude_from_pos_files exclude_from_bom)
+    (fp_text reference "REF**" (at 0.07 -2.92) (layer "F.SilkS")
+      (effects (font (size 1 1) (thickness 0.15)))
+    )
+    (fp_text value "MountingHole_4.3mm_M4" (at 0 5.3) (layer "F.Fab")
+      (effects (font (size 1 1) (thickness 0.15)))
+    )
+    (fp_text user "${REFERENCE}" (at 0.3 0) (layer "F.Fab")
+      (effects (font (size 1 1) (thickness 0.15)))
+    )
+    (fp_circle (center 0 0) (end 4.3 0) (layer "Cmts.User") (width 0.15) (fill none))
+    (fp_circle (center 0 0) (end 4.55 0) (layer "F.CrtYd") (width 0.05) (fill none))
+    (pad "1" np_thru_hole circle (at 0 0) (size 4.3 4.3) (drill 4.3) (layers *.Cu *.Mask))
+  )
+  (footprint "MountingHole:MountingHole_4.3mm_M4" (layer "F.Cu")
+    (at 112.44 136.14)
+    (descr "Mounting Hole 4.3mm, no annular, M4")
+    (tags "mounting hole 4.3mm no annular m4")
+    (attr exclude_from_pos_files exclude_from_bom)
+    (fp_text reference "REF**" (at 0.07 -2.92) (layer "F.SilkS")
+      (effects (font (size 1 1) (thickness 0.15)))
+    )
+    (fp_text value "MountingHole_4.3mm_M4" (at 0 5.3) (layer "F.Fab")
+      (effects (font (size 1 1) (thickness 0.15)))
+    )
+    (fp_text user "${REFERENCE}" (at 0.3 0) (layer "F.Fab")
+      (effects (font (size 1 1) (thickness 0.15)))
+    )
+    (fp_circle (center 0 0) (end 4.3 0) (layer "Cmts.User") (width 0.15) (fill none))
+    (fp_circle (center 0 0) (end 4.55 0) (layer "F.CrtYd") (width 0.05) (fill none))
+    (pad "1" np_thru_hole circle (at 0 0) (size 4.3 4.3) (drill 4.3) (layers *.Cu *.Mask))
+  )
+  (footprint "MountingHole:MountingHole_4.3mm_M4" (layer "F.Cu")
+    (at 5.83 136.14)
+    (descr "Mounting Hole 4.3mm, no annular, M4")
+    (tags "mounting hole 4.3mm no annular m4")
+    (attr exclude_from_pos_files exclude_from_bom)
+    (fp_text reference "REF**" (at 0.07 -2.92) (layer "F.SilkS")
+      (effects (font (size 1 1) (thickness 0.15)))
+    )
+    (fp_text value "MountingHole_4.3mm_M4" (at 0 5.3) (layer "F.Fab")
+      (effects (font (size 1 1) (thickness 0.15)))
+    )
+    (fp_text user "${REFERENCE}" (at 0.3 0) (layer "F.Fab")
+      (effects (font (size 1 1) (thickness 0.15)))
+    )
+    (fp_circle (center 0 0) (end 4.3 0) (layer "Cmts.User") (width 0.15) (fill none))
+    (fp_circle (center 0 0) (end 4.55 0) (layer "F.CrtYd") (width 0.05) (fill none))
+    (pad "1" np_thru_hole circle (at 0 0) (size 4.3 4.3) (drill 4.3) (layers *.Cu *.Mask))
+  )
   (footprint "Connector_PinHeader_2.54mm:PinHeader_2x20_P2.54mm_Horizontal" (layer "F.Cu")
     (at 6.64 95.17 180)
@@
     )
   )
+  (footprint "MountingHole:MountingHole_4.3mm_M4" (layer "F.Cu")
+    (at 112.44 4.96)
+    (descr "Mounting Hole 4.3mm, no annular, M4")
+    (tags "mounting hole 4.3mm no annular m4")
+    (attr exclude_from_pos_files exclude_from_bom)
+    (fp_text reference "REF**" (at 0.07 -2.92) (layer "F.SilkS")
+      (effects (font (size 1 1) (thickness 0.15)))
+    )
+    (fp_text value "MountingHole_4.3mm_M4" (at 0 5.3) (layer "F.Fab")
+      (effects (font (size 1 1) (thickness 0.15)))
+    )
+    (fp_text user "${REFERENCE}" (at 0.3 0) (layer "F.Fab")
+      (effects (font (size 1 1) (thickness 0.15)))
+    )
+    (fp_circle (center 0 0) (end 4.3 0) (layer "Cmts.User") (width 0.15) (fill none))
+    (fp_circle (center 0 0) (end 4.55 0) (layer "F.CrtYd") (width 0.05) (fill none))
+    (pad "1" np_thru_hole circle (at 0 0) (size 4.3 4.3) (drill 4.3) (layers *.Cu *.Mask))
+  )
   (gr_line (start 119 0) (end 119 142.08) (layer "Edge.Cuts") (width 0.1))
