File: Hardware/CLUSTERFCK/ADDR/ADDR/ADDR.kicad_pcb (KiCad board)
At the start: 2 copper layers, 64.3 x 469.5 mm, 38 parts, among them J1 Conn_02x04_Counter_Clockwise, J10 Conn_02x20_Counter_Clockwise, J11 Conn_02x20_Counter_Clockwise, J12 Conn_02x20_Counter_Clockwise, J13 Conn_02x20_Counter_Clockwise, J14 Conn_02x20_Counter_Clockwise, J2 Conn_02x06_Odd_Even, J3 Conn_02x10_Counter_Clockwise, J4 Conn_02x20_Counter_Clockwise, J5 Conn_02x20_Counter_Clockwise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

Commit message: 0066 | 6h | made holes in pcbs
Parts:
- added REF**: MountingHole_4.3mm_M4, MountingHole:MountingHole_4.3mm_M4, F.Cu at (422.6, 212.7)
- added REF**: MountingHole_4.3mm_M4, MountingHole:MountingHole_4.3mm_M4, F.Cu at (199.1, 212.2)
- added REF**: MountingHole_4.3mm_M4, MountingHole:MountingHole_4.3mm_M4, F.Cu at (225.1, 167.7)
- added REF**: MountingHole_4.3mm_M4, MountingHole:MountingHole_4.3mm_M4, F.Cu at (485.9, 168.4)
- added REF**: MountingHole_4.3mm_M4, MountingHole:MountingHole_4.3mm_M4, F.Cu at (141.2, 164.4)
- added REF**: MountingHole_4.3mm_M4, MountingHole:MountingHole_4.3mm_M4, F.Cu at (533.5, 213.3)
- added REF**: MountingHole_4.3mm_M4, MountingHole:MountingHole_4.3mm_M4, F.Cu at (385.0, 168.0)
- added REF**: MountingHole_4.3mm_M4, MountingHole:MountingHole_4.3mm_M4, F.Cu at (149.8, 198.9)
- added REF**: MountingHole_4.3mm_M4, MountingHole:MountingHole_4.3mm_M4, F.Cu at (313.6, 213.7)
- moved J13 512.7 mm to (498.3, 167.4), turned to 90 degrees
- moved J8 503.2 mm to (477.7, 206.4), turned to 90 degrees
- moved J12 465.9 mm to (464.1, 166.3), turned to -90 degrees
- moved J14 317.9 mm to (352.2, 166.3), turned to -90 degrees
- moved J7 310.2 mm to (320.8, 206.4), turned to 90 degrees
- moved J4 248.1 mm to (258.4, 207.2), turned to 90 degrees
- moved J6 246.3 mm to (294.0, 166.6), turned to -90 degrees
- moved J9 210.3 mm to (206.3, 207.2), turned to 90 degrees
- moved J5 208.9 mm to (86.6, 203.8), turned to 90 degrees
- moved R12 195.2 mm to (82.9, 191.1), turned to -90 degrees
- moved J10 194.3 mm to (143.7, 207.2), turned to 90 degrees
- moved R11 190.7 mm to (89.9, 191.1), turned to -90 degrees
- moved D12 186.6 mm to (82.9, 184.1), turned to -90 degrees
- moved R10 186.6 mm to (96.9, 191.1), turned to -90 degrees
- moved R9 182.9 mm to (103.9, 191.1), turned to -90 degrees
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Other:
- board size 64.3 x 469.5 mm -> 469.5 x 64.3 mm
