File: Hardware/CLUSTERFCK/DATA/DATA/DATA.kicad_pcb (KiCad board)
At the start: 2 copper layers, 64.3 x 469.5 mm, 27 parts, among them J1 Conn_02x04_Odd_Even, J10 Conn_02x08_Counter_Clockwise, J11 Conn_02x20_Counter_Clockwise, J2 Conn_02x20_Counter_Clockwise, J3 Conn_02x20_Counter_Clockwise, J4 Conn_02x20_Counter_Clockwise, J5 Conn_02x20_Counter_Clockwise, J6 Conn_02x20_Counter_Clockwise, J7 Conn_02x20_Counter_Clockwise, J8 Conn_02x20_Counter_Clockwise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

Commit message: 0066 | 6h | made holes in pcbs
Parts:
- added REF**: MountingHole_4.3mm_M4, MountingHole:MountingHole_4.3mm_M4, F.Cu at (270.6, 178.7)
- added REF**: MountingHole_4.3mm_M4, MountingHole:MountingHole_4.3mm_M4, F.Cu at (96.3, 228.4)
- added REF**: MountingHole_4.3mm_M4, MountingHole:MountingHole_4.3mm_M4, F.Cu at (399.2, 227.4)
- added REF**: MountingHole_4.3mm_M4, MountingHole:MountingHole_4.3mm_M4, F.Cu at (441.6, 178.6)
- added REF**: MountingHole_4.3mm_M4, MountingHole:MountingHole_4.3mm_M4, F.Cu at (173.5, 223.4)
- added REF**: MountingHole_4.3mm_M4, MountingHole:MountingHole_4.3mm_M4, F.Cu at (528.7, 176.2)
- added REF**: MountingHole_4.3mm_M4, MountingHole:MountingHole_4.3mm_M4, F.Cu at (251.2, 219.6)
- added REF**: MountingHole_4.3mm_M4, MountingHole:MountingHole_4.3mm_M4, F.Cu at (96.1, 174.3)
- moved J6 535.6 mm to (510.2, 220.9), turned to 90 degrees
- moved J11 520.8 mm to (513.6, 181.9), turned to -90 degrees
- moved J5 491.4 mm to (475.4, 222.0), turned to -90 degrees
- moved J9 375.3 mm to (404.0, 180.9), turned to -90 degrees
- moved J4 356.3 mm to (364.2, 222.0), turned to -90 degrees
- moved J3 294.1 mm to (305.9, 221.7), turned to -90 degrees
- moved J10 248.3 mm to (298.7, 181.8), turned to -90 degrees
- moved J2 232.7 mm to (228.4, 222.0), turned to -90 degrees
- moved J1 220.7 mm to (118.0, 220.9), turned to 90 degrees
- moved R8 214.2 mm to (94.9, 206.9), turned to -90 degrees
- moved R7 210.0 mm to (101.8, 206.9), turned to -90 degrees
- moved R6 206.2 mm to (108.8, 206.9), turned to -90 degrees
- moved D8 205.4 mm to (94.9, 199.9), turned to -90 degrees
- moved R5 202.8 mm to (115.8, 206.9), turned to -90 degrees
- moved D7 201.0 mm to (101.8, 199.9), turned to -90 degrees
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Other:
- board size 64.3 x 469.5 mm -> 469.5 x 64.3 mm

Commit message: 0072 | 3h | make silkscreen prettier
Other:
- board text removed: "done"
Changed lines of the file:
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@@
     (property "Schaltplanname" "")
     (attr through_hole)
-    (fp_text reference "J7" (at -5.65 -2.77 -270) (layer "F.SilkS")
+    (fp_text reference "J7" (at -1.5935 50.46 -270) (layer "F.SilkS")
       (effects (font (size 1 1) (thickness 0.15)))
     )
@@
     (property "Schaltplanname" "")
     (attr through_hole)
-    (fp_text reference "J9" (at -5.65 -2.77 -270) (layer "F.SilkS")
+    (fp_text reference "J9" (at -1.1535 50.774 -90) (layer "F.SilkS")
       (effects (font (size 1 1) (thickness 0.15)))
     )
@@
     (property "Schaltplanname" "")
     (attr through_hole)
-    (fp_text reference "J6" (at -5.65 -2.77 90) (layer "F.SilkS")
+    (fp_text reference "J6" (at -1.5965 -2.46 270) (layer "F.SilkS")
       (effects (font (size 1 1) (thickness 0.15)))
     )
@@
     (property "Schaltplanname" "")
     (attr through_hole)
-    (fp_text reference "J11" (at -5.65 -2.77 -270) (layer "F.SilkS")
+    (fp_text reference "J11" (at -1.4235 51.14 -90) (layer "F.SilkS")
       (effects (font (size 1 1) (thickness 0.15)))
     )
@@
     (property "Schaltplanname" "")
     (attr through_hole)
-    (fp_text reference "J2" (at 5.655 -2.27 -270) (layer "F.SilkS")
+    (fp_text reference "J2" (at 1.1765 50.38 -90) (layer "F.SilkS")
       (effects (font (size 1 1) (thickness 0.15)))
     )
@@
     (property "Schaltplanname" "")
     (attr through_hole)
-    (fp_text reference "J4" (at 5.655 -2.27 -270) (layer "F.SilkS")
+    (fp_text reference "J4" (at 1.3965 50.78 -90) (layer "F.SilkS")
       (effects (font (size 1 1) (thickness 0.15)))
     )
@@
     (property "Schaltplanname" "")
     (attr through_hole)
-    (fp_text reference "J10" (at -5.65 -2.77 -270) (layer "F.SilkS")
+    (fp_text reference "J10" (at -1.1435 20.67 -90) (layer "F.SilkS")
       (effects (font (size 1 1) (thickness 0.15)))
     )
@@
     (property "Schaltplanname" "")
     (attr through_hole)
-    (fp_text reference "J3" (at 5.655 -2.27 -270) (layer "F.SilkS")
+    (fp_text reference "J3" (at 1.1065 50.75 -90) (layer "F.SilkS")
       (effects (font (size 1 1) (thickness 0.15)))
     )
@@
     (property "Schaltplanname" "")
     (attr through_hole)
-    (fp_text reference "J8" (at -5.65 -2.77 -270) (layer "F.SilkS")
+    (fp_text reference "J8" (at -1.1735 50.76 -90) (layer "F.SilkS")
       (effects (font (size 1 1) (thickness 0.15)))
     )
@@
     (property "Schaltplanname" "")
     (attr through_hole)
-    (fp_text reference "J1" (at -5.65 -2.77 90) (layer "F.SilkS")
+    (fp_text reference "J1" (at -1.1865 -2.37 270) (layer "F.SilkS")
       (effects (font (size 1 1) (thickness 0.15)))
     )
@@
     (property "Schaltplanname" "")
     (attr through_hole)
-    (fp_text reference "J5" (at 5.655 -2.27 -270) (layer "F.SilkS")
+    (fp_text reference "J5" (at 1.2865 50.72 -90) (layer "F.SilkS")
       (effects (font (size 1 1) (thickness 0.15)))
     )
@@
     (effects (font (size 2 2) (thickness 0.3)))
   )
-  (gr_text "D1" (at 136.77 195.4635 90) (layer "F.SilkS")
+  (gr_text "D1" (at 136.73 195.62 90) (layer "F.SilkS")
     (effects (font (size 2 2) (thickness 0.3)))
   )
@@
     (effects (font (size 2 2) (thickness 0.3)))
   )
-  (gr_text "DATA Bus" (at 553.965 180.8585 90) (layer "F.SilkS")
+  (gr_text "DATA Bus" (at 554.14 181.33 90) (layer "F.SilkS")
     (effects (font (size 3 3) (thickness 0.5)))
   )
@@
     (effects (font (size 2 2) (thickness 0.3)))
   )
-  (gr_text "done" (at 122.165 247.5335 90) (layer "User.1")
-    (effects (font (size 1 1) (thickness 0.15)))
-  )
-  (gr_text "done" (at 126.47 164.8135 90) (layer "User.1")
-    (effects (font (size 1 1) (thickness 0.15)))
-  )
-  (gr_text "done" (at 290.15 162.8135 90) (layer "User.1")
-    (effects (font (size 1 1) (thickness 0.15)))
-  )
-  (gr_text "done" (at 450.51 238.6435 90) (layer "User.1")
-    (effects (font (size 1 1) (thickness 0.15)))
-  )
-  (gr_text "done" (at 282.28 240.9035 90) (layer "User.1")
-    (effects (font (size 1 1) (thickness 0.15)))
-  )
-  (gr_text "done" (at 537.97 238.6135 90) (layer "User.1")
-    (effects (font (size 1 1) (thickness 0.15)))
-  )
-  (gr_text "done" (at 202.75 242.9035 90) (layer "User.1")
-    (effects (font (size 1 1) (thickness 0.15)))
-  )
-  (gr_text "done" (at 203.84 159.9335 90) (layer "User.1")
-    (effects (font (size 1 1) (thickness 0.15)))
-  )
-  (gr_text "done" (at 489.02 162.8235 90) (layer "User.1")
-    (effects (font (size 1 1) (thickness 0.15)))
-  )
-  (gr_text "done" (at 373.65 163.2935 90) (layer "User.1")
-    (effects (font (size 1 1) (thickness 0.15)))
-  )
-  (gr_text "done" (at 337.73 238.5735 90) (layer "User.1")
-    (effects (font (size 1 1) (thickness 0.15)))
-  )
   (segment (start 143.755 205.8685) (end 143.755 202.4485) (width 1) (layer "F.Cu") (net 1))
   (segment (start 214.85 182.6935) (end 214.85 220.148501) (width 0.2) (layer "F.Cu") (net 2))
@@
   (via (at 522.85 191.6535) (size 0.8) (drill 0.4) (layers "F.Cu" "B.Cu") (free) (net 2))
   (via (at 383.785 214.5135) (size 0.8) (drill 0.4) (layers "F.Cu" "B.Cu") (free) (net 2))
-  (via (at 558.41 191.6535) (size 0.8) (drill 0.4) (layers "F.Cu" "B.Cu") (free) (net 2))
+  (via (at 559.03 191.29) (size 0.8) (drill 0.4) (layers "F.Cu" "B.Cu") (free) (net 2))
   (via (at 383.785 199.2735) (size 0.8) (drill 0.4) (layers "F.Cu" "B.Cu") (free) (net 2))
   (via (at 155.185 170.6985) (size 0.8) (drill 0.4) (layers "F.Cu" "B.Cu") (free) (net 2))
@@
   (via (at 533.645 191.6535) (size 0.8) (drill 0.4) (layers "F.Cu" "B.Cu") (free) (net 2))
   (via (at 195.19 199.9085) (size 0.8) (drill 0.4) (layers "F.Cu" "B.Cu") (free) (net 2))
-  (via (at 558.41 214.5135) (size 0.8) (drill 0.4) (layers "F.Cu" "B.Cu") (free) (net 2))
+  (via (at 558.84 214.22) (size 0.8) (drill 0.4) (layers "F.Cu" "B.Cu") (free) (net 2))
   (via (at 241.545 174.5085) (size 0.8) (drill 0.4) (layers "F.Cu" "B.Cu") (free) (net 2))
   (via (at 462.525 191.6535) (size 0.8) (drill 0.4) (layers "F.Cu" "B.Cu") (free) (net 2))
@@
   (via (at 226.94 193.5585) (size 0.8) (drill 0.4) (layers "F.Cu" "B.Cu") (free) (net 2))
   (via (at 438.395 199.2735) (size 0.8) (drill 0.4) (layers "F.Cu" "B.Cu") (free) (net 2))
-  (via (at 128.515 194.1935) (size 0.8) (drill 0.4) (layers "F.Cu" "B.Cu") (free) (net 2))
+  (via (at 128.05 194.21) (size 0.8) (drill 0.4) (layers "F.Cu" "B.Cu") (free) (net 2))
   (via (at 241.545 227.8485) (size 0.8) (drill 0.4) (layers "F.Cu" "B.Cu") (free) (net 2))
   (via (at 273.93 170.6985) (size 0.8) (drill 0.4) (layers "F.Cu" "B.Cu") (free) (net 2))
@@
   (via (at 308.22 174.5085) (size 0.8) (drill 0.4) (layers "F.Cu" "B.Cu") (free) (net 2))
   (via (at 315.84 182.7635) (size 0.8) (drill 0.4) (layers "F.Cu" "B.Cu") (free) (net 2))
-  (via (at 558.41 199.2735) (size 0.8) (drill 0.4) (layers "F.Cu" "B.Cu") (free) (net 2))
+  (via (at 558.99 199.3) (size 0.8) (drill 0.4) (layers "F.Cu" "B.Cu") (free) (net 2))
   (via (at 388.23 182.7635) (size 0.8) (drill 0.4) (layers "F.Cu" "B.Cu") (free) (net 2))
   (via (at 533.645 182.7635) (size 0.8) (drill 0.4) (layers "F.Cu" "B.Cu") (free) (net 2))
