File: Hardware/CLUSTERFCK/PC/PC/PC.kicad_pcb (KiCad board)
At the start: 2 copper layers, 142.1 x 63 mm, 35 parts, among them J1 Conn_02x20_Counter_Clockwise, U1 74LS245, U2 74LS161, U3 74LS245, U4 74LS161, U5 74LS161

Commit message: 0066 | 6h | made holes in pcbs
Parts:
- added REF**: MountingHole_4.3mm_M4, MountingHole:MountingHole_4.3mm_M4, F.Cu at (6.23, 30.5)
- added REF**: MountingHole_4.3mm_M4, MountingHole:MountingHole_4.3mm_M4, F.Cu at (123.5, 9.99)
- added REF**: MountingHole_4.3mm_M4, MountingHole:MountingHole_4.3mm_M4, F.Cu at (125.3, 56.5)
Other:
- net class Default removed

Commit message: 0072 | 3h | make silkscreen prettier
Changed lines of the file:
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@@
     (tags "LED diameter 5.0mm 2 pins")
     (attr through_hole)
-    (fp_text reference "D5" (at 1.27 -3.96 90) (layer "F.SilkS")
+    (fp_text reference "D5" (at 1.27 -3.74 90) (layer "F.SilkS")
       (effects (font (size 1 1) (thickness 0.15)))
     )
@@
     (tags "capacitor handsolder")
     (attr smd)
-    (fp_text reference "C1" (at 0 -1.65 90) (layer "F.SilkS")
+    (fp_text reference "C1" (at -1.09 -1.52 90) (layer "F.SilkS")
       (effects (font (size 1 1) (thickness 0.15)))
     )
@@
     (tags "LED diameter 5.0mm 2 pins")
     (attr through_hole)
-    (fp_text reference "D10" (at 1.27 -3.96 90) (layer "F.SilkS")
+    (fp_text reference "D10" (at 1.27 -3.74 90) (layer "F.SilkS")
       (effects (font (size 1 1) (thickness 0.15)))
     )
@@
     (tags "LED diameter 5.0mm 2 pins")
     (attr through_hole)
-    (fp_text reference "D12" (at 1.27 -3.96 90) (layer "F.SilkS")
+    (fp_text reference "D12" (at 1.27 -3.74 90) (layer "F.SilkS")
       (effects (font (size 1 1) (thickness 0.15)))
     )
@@
     (tags "LED diameter 5.0mm 2 pins")
     (attr through_hole)
-    (fp_text reference "D1" (at 1.27 -3.96 90) (layer "F.SilkS")
+    (fp_text reference "D1" (at 1.27 -3.74 90) (layer "F.SilkS")
       (effects (font (size 1 1) (thickness 0.15)))
     )
@@
     (tags "LED diameter 5.0mm 2 pins")
     (attr through_hole)
-    (fp_text reference "D8" (at 1.27 -3.96 90) (layer "F.SilkS")
+    (fp_text reference "D8" (at 1.27 -3.74 90) (layer "F.SilkS")
       (effects (font (size 1 1) (thickness 0.15)))
     )
@@
     (tags "capacitor handsolder")
     (attr smd)
-    (fp_text reference "C2" (at 0 -1.65 90) (layer "F.SilkS")
+    (fp_text reference "C2" (at 0 -2.055 90) (layer "F.SilkS")
       (effects (font (size 1 1) (thickness 0.15)))
     )
@@
     (tags "capacitor handsolder")
     (attr smd)
-    (fp_text reference "C5" (at 0 -1.65 90) (layer "F.SilkS")
+    (fp_text reference "C5" (at -0.265 -2.165 90) (layer "F.SilkS")
       (effects (font (size 1 1) (thickness 0.15)))
     )
@@
     (tags "LED diameter 5.0mm 2 pins")
     (attr through_hole)
-    (fp_text reference "D3" (at 1.27 -3.96 90) (layer "F.SilkS")
+    (fp_text reference "D3" (at 1.27 -3.74 90) (layer "F.SilkS")
       (effects (font (size 1 1) (thickness 0.15)))
     )
@@
     (tags "LED diameter 5.0mm 2 pins")
     (attr through_hole)
-    (fp_text reference "D4" (at 1.27 -3.96 90) (layer "F.SilkS")
+    (fp_text reference "D4" (at 1.27 -3.74 90) (layer "F.SilkS")
       (effects (font (size 1 1) (thickness 0.15)))
     )
@@
     (tags "LED diameter 5.0mm 2 pins")
     (attr through_hole)
-    (fp_text reference "D2" (at 1.27 -3.96 90) (layer "F.SilkS")
+    (fp_text reference "D2" (at 1.27 -3.74 90) (layer "F.SilkS")
       (effects (font (size 1 1) (thickness 0.15)))
     )
@@
     (tags "LED diameter 5.0mm 2 pins")
     (attr through_hole)
-    (fp_text reference "D9" (at 1.27 -3.96 90) (layer "F.SilkS")
+    (fp_text reference "D9" (at 1.27 -3.74 90) (layer "F.SilkS")
       (effects (font (size 1 1) (thickness 0.15)))
     )
@@
     (tags "SOIC SO")
     (attr smd)
-    (fp_text reference "U4" (at 0 -5.9 90) (layer "F.SilkS")
+    (fp_text reference "U4" (at -2.41 -6.16 90) (layer "F.SilkS")
       (effects (font (size 1 1) (thickness 0.15)))
     )
@@
     (tags "Through hole angled socket strip THT 2x20 2.54mm double row")
     (attr through_hole)
-    (fp_text reference "J1" (at -5.65 -2.77) (layer "F.SilkS")
+    (fp_text reference "J1" (at -1.205 -2.565) (layer "F.SilkS")
       (effects (font (size 1 1) (thickness 0.15)))
     )
@@
     (tags "capacitor handsolder")
     (attr smd)
-    (fp_text reference "C3" (at 0 -1.65 90) (layer "F.SilkS")
+    (fp_text reference "C3" (at -0.93 -1.855 90) (layer "F.SilkS")
       (effects (font (size 1 1) (thickness 0.15)))
     )
@@
     (tags "SOIC SO")
     (attr smd)
-    (fp_text reference "U2" (at 0 -5.9 90) (layer "F.SilkS")
+    (fp_text reference "U2" (at -2.41 -6.055 90) (layer "F.SilkS")
       (effects (font (size 1 1) (thickness 0.15)))
     )
@@
     (tags "LED diameter 5.0mm 2 pins")
     (attr through_hole)
-    (fp_text reference "D7" (at 1.27 -3.96 90) (layer "F.SilkS")
+    (fp_text reference "D7" (at 1.27 -3.74 90) (layer "F.SilkS")
       (effects (font (size 1 1) (thickness 0.15)))
     )
@@
     (tags "LED diameter 5.0mm 2 pins")
     (attr through_hole)
-    (fp_text reference "D6" (at 1.27 -3.96 90) (layer "F.SilkS")
+    (fp_text reference "D6" (at 1.27 -3.74 90) (layer "F.SilkS")
       (effects (font (size 1 1) (thickness 0.15)))
     )
@@
     (tags "LED diameter 5.0mm 2 pins")
     (attr through_hole)
-    (fp_text reference "D11" (at 1.27 -3.96 90) (layer "F.SilkS")
+    (fp_text reference "D11" (at 1.27 -3.74 90) (layer "F.SilkS")
       (effects (font (size 1 1) (thickness 0.15)))
     )
@@
     (tags "SOIC SO")
     (attr smd)
-    (fp_text reference "U5" (at 0 -5.9 90) (layer "F.SilkS")
+    (fp_text reference "U5" (at -0.985 -5.87 90) (layer "F.SilkS")
       (effects (font (size 1 1) (thickness 0.15)))
     )
@@
     (tags "capacitor handsolder")
     (attr smd)
-    (fp_text reference "C4" (at 0 -1.65 90) (layer "F.SilkS")
+    (fp_text reference "C4" (at -0.93 -1.715 90) (layer "F.SilkS")
       (effects (font (size 1 1) (thickness 0.15)))
     )
@@
     (effects (font (size 3 3) (thickness 0.7)))
   )
-  (gr_text "Kevin da Silva Fernandes 2020" (at 102.743 2.921) (layer "F.SilkS")
+  (gr_text "Kevin da Silva Fernandes 2020" (at 102.743 2.775) (layer "F.SilkS")
     (effects (font (size 2 2) (thickness 0.3)))
   )
@@
   (segment (start 85.755 40.885) (end 85.59 40.885) (width 1) (layer "F.Cu") (net 2))
   (segment (start 81.27 12.31) (end 89.23 4.35) (width 1) (layer "F.Cu") (net 2))
+  (segment (start 87.47 24.67) (end 87.47 39.17) (width 1) (layer "F.Cu") (net 2))
   (segment (start 87.47 18.635) (end 87.47 24.67) (width 1) (layer "F.Cu") (net 2))
-  (segment (start 87.47 24.67) (end 87.47 39.17) (width 1) (layer "F.Cu") (net 2))
   (segment (start 81.145 12.31) (end 79.64 12.31) (width 0.5) (layer "F.Cu") (net 2))
   (segment (start 51.935 4.33) (end 53.88 4.33) (width 0.5) (layer "F.Cu") (net 2))
@@
   (via (at 64.005 50.395) (size 0.45) (drill 0.3) (layers "F.Cu" "B.Cu") (net 31))
   (via (at 114.165 50.395) (size 0.45) (drill 0.3) (layers "F.Cu" "B.Cu") (net 31))
+  (segment (start 64.005 50.395) (end 114.165 50.395) (width 0.2) (layer "B.Cu") (net 31))
   (segment (start 46.855 50.395) (end 64.005 50.395) (width 0.2) (layer "B.Cu") (net 31))
-  (segment (start 64.005 50.395) (end 114.165 50.395) (width 0.2) (layer "B.Cu") (net 31))
   (segment (start 106.545 49.865) (end 106.545 52.365) (width 0.2) (layer "F.Cu") (net 32))
   (segment (start 48.125 42.66) (end 48.125 49.865) (width 0.2) (layer "F.Cu") (net 32))
@@
   (via (at 76.07 47.72) (size 0.45) (drill 0.3) (layers "F.Cu" "B.Cu") (net 36))
   (via (at 78.605 47.715) (size 0.45) (drill 0.3) (layers "F.Cu" "B.Cu") (net 36))
+  (segment (start 76.07 47.72) (end 78.6 47.72) (width 0.2) (layer "B.Cu") (net 36))
   (segment (start 53.23 47.72) (end 76.07 47.72) (width 0.2) (layer "B.Cu") (net 36))
-  (segment (start 76.07 47.72) (end 78.6 47.72) (width 0.2) (layer "B.Cu") (net 36))
   (segment (start 78.6 47.72) (end 78.605 47.715) (width 0.2) (layer "B.Cu") (net 36))
   (segment (start 79.875 40.485) (end 79.875 47.175) (width 0.2) (layer "F.Cu") (net 37))
@@
   (via (at 39.857497 46.112503) (size 0.45) (drill 0.3) (layers "F.Cu" "B.Cu") (net 39))
   (segment (start 39.857497 46.112503) (end 52.707497 46.112503) (width 0.2) (layer "B.Cu") (net 39))
+  (segment (start 57.737503 17.242503) (end 55.607497 17.242503) (width 0.2) (layer "B.Cu") (net 39))
   (segment (start 55.607497 17.242503) (end 39.857497 17.242503) (width 0.2) (layer "B.Cu") (net 39))
-  (segment (start 57.737503 17.242503) (end 55.607497 17.242503) (width 0.2) (layer "B.Cu") (net 39))
   (segment (start 57.737503 17.242503) (end 72.897497 17.242503) (width 0.2) (layer "B.Cu") (net 39))
   (segment (start 56.875 14.085) (end 56.875 16.710004) (width 0.2) (layer "F.Cu") (net 40))
@@
   (via (at 37.965 45.045) (size 0.45) (drill 0.3) (layers "F.Cu" "B.Cu") (net 41))
   (segment (start 59.227501 16.192501) (end 75.437499 16.192501) (width 0.2) (layer "B.Cu") (net 41))
+  (segment (start 59.227501 16.192501) (end 58.137499 16.192501) (width 0.2) (layer "B.Cu") (net 41))
   (segment (start 58.137499 16.192501) (end 40.907499 16.192501) (width 0.2) (layer "B.Cu") (net 41))
-  (segment (start 59.227501 16.192501) (end 58.137499 16.192501) (width 0.2) (layer "B.Cu") (net 41))
   (segment (start 37.972501 45.052501) (end 37.965 45.045) (width 0.2) (layer "B.Cu") (net 41))
   (segment (start 40.907499 45.052501) (end 37.972501 45.052501) (width 0.2) (layer "B.Cu") (net 41))
